File: PCB/Rev 02.00/000018 PGKB/leds.kicad_sch (KiCad schematic)
At the start: 5 parts

Commit message: Schematic
Other:
- company: 4D Haptics Oy -> Kallio Designs Oy
- title: Suspension Rig -> Programmable Keyboard
Changed lines of the file:
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@@
   (paper "A4")
   (title_block
-    (title "Suspension Rig")
-    (date "2023-09-25")
+    (title "Programmable Keyboard")
+    (date "2023-10-14")
     (rev "1.0")
-    (company "4D Haptics Oy")
-    (comment 1 "TL, SB")
+    (company "Kallio Designs Oy")
+    (comment 1 "TL, NH")
     (comment 3 "PCB_PN")
   )
