File: PCB/Rev 02.00/000018 PGKB/main.kicad_sch (KiCad schematic)
At the start: 0 parts

Commit message: buttons
Other:
- added sheet Untitled Sheet (buttons.kicad_sch)
- sheet Microcontroller ports: added GPIO0, GPIO1, GPIO2; removed none
Changed lines of the file:
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@@
+    )
+  )
+  (sheet (at 201.93 63.5) (size 34.29 20.32) (fields_autoplaced)
+    (stroke (width 0.1524) (type solid))
+    (fill (color 0 0 0 0.0000))
+    (property "Sheetname" "Untitled Sheet" (at 201.93 62.7884 0)
+      (effects (font (size 1.27 1.27)) (justify left bottom))
+    )
+    (property "Sheetfile" "buttons.kicad_sch" (at 201.93 84.4046 0)
+      (effects (font (size 1.27 1.27)) (justify left top))
+    )
+    (pin "Button1" output (at 201.93 69.85 180)
+      (effects (font (size 1.27 1.27)) (justify left))
+    )
+    (pin "Button4" output (at 201.93 77.47 180)
+      (effects (font (size 1.27 1.27)) (justify left))
+    )
+    (pin "Button0" output (at 201.93 67.31 180)
+      (effects (font (size 1.27 1.27)) (justify left))
+    )
+    (pin "Button3" output (at 201.93 74.93 180)
+      (effects (font (size 1.27 1.27)) (justify left))
+    )
+    (pin "Button5" output (at 201.93 80.01 180)
+      (effects (font (size 1.27 1.27)) (justify left))
+    )
+    (pin "Button2" output (at 201.93 72.39 180)
+      (effects (font (size 1.27 1.27)) (justify left))
+    )
+    (instances
+      (project "000018 PGKB"
+        (path "/e63e39d7-6ac0-4ffd-8aa3-1841a4541b55/2eb44e1a-4042-4ea6-aca2-4836a6ec84e9" (page "10"))
+      )
     )
   )
@@
     )
   )
-  (sheet (at 151.13 85.09) (size 21.59 31.75) (fields_autoplaced)
+  (sheet (at 151.13 63.5) (size 38.1 77.47) (fields_autoplaced)
     (stroke (width 0.1524) (type solid))
     (fill (color 0 0 0 0.0000))
-    (property "Sheetname" "Microcontroller" (at 151.13 84.3784 0)
+    (property "Sheetname" "Microcontroller" (at 151.13 62.7884 0)
       (effects (font (size 1.27 1.27)) (justify left bottom))
     )
-    (property "Sheetfile" "mcu.kicad_sch" (at 151.13 117.4246 0)
+    (property "Sheetfile" "mcu.kicad_sch" (at 151.13 141.5546 0)
       (effects (font (size 1.27 1.27)) (justify left top))
     )
@@
       (effects (font (size 1.27 1.27)) (justify left))
     )
-    (pin "{I2C}" bidirectional (at 172.72 105.41 0)
+    (pin "{I2C}" bidirectional (at 189.23 105.41 0)
       (effects (font (size 1.27 1.27)) (justify right))
     )
+    (pin "GPIO1" bidirectional (at 189.23 69.85 0)
+      (effects (font (size 1.27 1.27)) (justify right))
+    )
+    (pin "GPIO0" bidirectional (at 189.23 67.31 0)
+      (effects (font (size 1.27 1.27)) (justify right))
+    )
+    (pin "GPIO2" bidirectional (at 189.23 72.39 0)
+      (effects (font (size 1.27 1.27)) (justify right))
+    )

Commit message: schematic
Other:
- added sheet Connectors (connectors.kicad_sch)
- sheet Microcontroller ports: added {I2C0}; removed {I2C}
Changed lines of the file:
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@@
     (comment 3 "PCB_PN")
   )
+  (bus_alias "I2C" (members "SDA" "SCL"))
   (wire (pts (xy 81.28 95.25) (xy 151.13 95.25))
     (stroke (width 0) (type default))
@@
   (bus (pts (xy 82.55 107.95) (xy 151.13 107.95))
     (stroke (width 0) (type default))
+  )
+  (sheet (at 201.93 93.98) (size 29.21 12.7) (fields_autoplaced)
+    (stroke (width 0.1524) (type solid))
+    (fill (color 0 0 0 0.0000))
+    (property "Sheetname" "Connectors" (at 201.93 93.2684 0)
+      (effects (font (size 1.27 1.27)) (justify left bottom))
+    )
+    (property "Sheetfile" "connectors.kicad_sch" (at 201.93 107.2646 0)
+      (effects (font (size 1.27 1.27)) (justify left top))
+    )
+    (pin "{I2C}" bidirectional (at 201.93 96.52 180)
+      (effects (font (size 1.27 1.27)) (justify left))
+    )
+    (instances
+      (project "000018 PGKB"
+        (path "/e63e39d7-6ac0-4ffd-8aa3-1841a4541b55/2eb44e1a-4042-4ea6-aca2-4836a6ec84e9" (page "11"))
+      )
+    )
   )
   (sheet (at 57.15 87.63) (size 24.13 10.16) (fields_autoplaced)
@@
       (effects (font (size 1.27 1.27)) (justify left))
     )
-    (pin "{I2C}" bidirectional (at 189.23 105.41 0)
-      (effects (font (size 1.27 1.27)) (justify right))
-    )
     (pin "GPIO1" bidirectional (at 189.23 69.85 0)
       (effects (font (size 1.27 1.27)) (justify right))
@@
       (effects (font (size 1.27 1.27)) (justify right))
     )
+    (pin "{I2C0}" bidirectional (at 189.23 97.79 0)
+      (effects (font (size 1.27 1.27)) (justify right))
+    )

Commit message: Schematic
Other:
- sheet Untitled Sheet renamed Buttons
- title: TITLE -> Programmable Keyboard
Changed lines of the file:
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@@
   (paper "A4")
   (title_block
-    (title "TITLE")
-    (date "2023-05-28")
+    (title "Programmable Keyboard")
+    (date "2023-10-14")
     (rev "1.0")
     (company "Kallio Designs Oy")
-    (comment 1 "Teemu Latonen")
+    (comment 1 "TL, NH")
     (comment 2 "ASSEMBLY_PN")
     (comment 3 "PCB_PN")
@@
     (instances
       (project "000018 PGKB"
-        (path "/e63e39d7-6ac0-4ffd-8aa3-1841a4541b55/2eb44e1a-4042-4ea6-aca2-4836a6ec84e9" (page "11"))
+        (path "/e63e39d7-6ac0-4ffd-8aa3-1841a4541b55/2eb44e1a-4042-4ea6-aca2-4836a6ec84e9" (page "7"))
       )
     )
@@
       (project "000018 PGKB"
         (path "/e63e39d7-6ac0-4ffd-8aa3-1841a4541b55" (page "6"))
-        (path "/e63e39d7-6ac0-4ffd-8aa3-1841a4541b55/2eb44e1a-4042-4ea6-aca2-4836a6ec84e9" (page "6"))
+        (path "/e63e39d7-6ac0-4ffd-8aa3-1841a4541b55/2eb44e1a-4042-4ea6-aca2-4836a6ec84e9" (page "3"))
       )
     )
@@
     (stroke (width 0.1524) (type solid))
     (fill (color 0 0 0 0.0000))
-    (property "Sheetname" "Untitled Sheet" (at 201.93 62.7884 0)
+    (property "Sheetname" "Buttons" (at 201.93 62.7884 0)
       (effects (font (size 1.27 1.27)) (justify left bottom))
     )
@@
     (instances
       (project "000018 PGKB"
-        (path "/e63e39d7-6ac0-4ffd-8aa3-1841a4541b55/2eb44e1a-4042-4ea6-aca2-4836a6ec84e9" (page "10"))
+        (path "/e63e39d7-6ac0-4ffd-8aa3-1841a4541b55/2eb44e1a-4042-4ea6-aca2-4836a6ec84e9" (page "4"))
       )
     )
@@
       (project "000018 PGKB"
         (path "/e63e39d7-6ac0-4ffd-8aa3-1841a4541b55" (page "2"))
-        (path "/e63e39d7-6ac0-4ffd-8aa3-1841a4541b55/2eb44e1a-4042-4ea6-aca2-4836a6ec84e9" (page "2"))
+        (path "/e63e39d7-6ac0-4ffd-8aa3-1841a4541b55/2eb44e1a-4042-4ea6-aca2-4836a6ec84e9" (page "9"))
       )
     )
@@
     (instances
       (project "000018 PGKB"
-        (path "/e63e39d7-6ac0-4ffd-8aa3-1841a4541b55/2eb44e1a-4042-4ea6-aca2-4836a6ec84e9" (page "7"))
+        (path "/e63e39d7-6ac0-4ffd-8aa3-1841a4541b55/2eb44e1a-4042-4ea6-aca2-4836a6ec84e9" (page "5"))
       )
     )
@@
     (instances
       (project "000018 PGKB"
-        (path "/e63e39d7-6ac0-4ffd-8aa3-1841a4541b55/2eb44e1a-4042-4ea6-aca2-4836a6ec84e9" (page "9"))
+        (path "/e63e39d7-6ac0-4ffd-8aa3-1841a4541b55/2eb44e1a-4042-4ea6-aca2-4836a6ec84e9" (page "6"))
       )
     )
