File: PCB/Rev 02.00/000018 PGKB/main.kicad_sch (KiCad schematic)
At the start: 0 parts

Commit message: buttons
Other:
- added sheet Buttons1 (buttons.kicad_sch)
- sheet Microcontroller ports: added ENC_A, ENC_B, GPIO10, GPIO11, GPIO12, GPIO3, GPIO4, GPIO5, GPIO6, GPIO7, GPIO8, GPIO9, NEOPIX_DRIVE, {I2C1}, {SPI}; removed none
Changed lines of the file:
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@@
   )
   (bus_alias "I2C" (members "SDA" "SCL"))
+  (wire (pts (xy 189.23 93.98) (xy 199.39 93.98))
+    (stroke (width 0) (type default))
+  )
+  (wire (pts (xy 189.23 88.9) (xy 199.39 88.9))
+    (stroke (width 0) (type default))
+  )
+  (bus (pts (xy 189.23 129.54) (xy 201.93 129.54))
+    (stroke (width 0) (type default))
+  )
   (wire (pts (xy 81.28 95.25) (xy 151.13 95.25))
     (stroke (width 0) (type default))
@@
     (stroke (width 0) (type default))
   )
+  (wire (pts (xy 189.23 80.01) (xy 199.39 80.01))
+    (stroke (width 0) (type default))
+  )
+  (wire (pts (xy 189.23 99.06) (xy 199.39 99.06))
+    (stroke (width 0) (type default))
+  )
   (wire (pts (xy 87.63 90.17) (xy 87.63 52.07))
     (stroke (width 0) (type default))
   )
+  (wire (pts (xy 189.23 77.47) (xy 199.39 77.47))
+    (stroke (width 0) (type default))
+  )
+  (wire (pts (xy 189.23 96.52) (xy 199.39 96.52))
+    (stroke (width 0) (type default))
+  )
+  (wire (pts (xy 189.23 101.6) (xy 199.39 101.6))
+    (stroke (width 0) (type default))
+  )
+  (wire (pts (xy 189.23 69.85) (xy 199.39 69.85))
+    (stroke (width 0) (type default))
+  )
+  (wire (pts (xy 189.23 67.31) (xy 199.39 67.31))
+    (stroke (width 0) (type default))
+  )
+  (wire (pts (xy 189.23 72.39) (xy 199.39 72.39))
+    (stroke (width 0) (type default))
+  )
+  (wire (pts (xy 189.23 74.93) (xy 199.39 74.93))
+    (stroke (width 0) (type default))
+  )
   (bus (pts (xy 82.55 107.95) (xy 151.13 107.95))
+    (stroke (width 0) (type default))
+  )
+  (wire (pts (xy 189.23 91.44) (xy 199.39 91.44))
     (stroke (width 0) (type default))
   )
@@
     )
   )
-  (sheet (at 201.93 63.5) (size 34.29 55.88) (fields_autoplaced)
-    (stroke (width 0.1524) (type solid))
-    (fill (color 0 0 0 0.0000))
-    (property "Sheetname" "Buttons" (at 201.93 62.7884 0)
-      (effects (font (size 1.27 1.27)) (justify left bottom))
-    )
-    (property "Sheetfile" "buttons.kicad_sch" (at 201.93 119.9646 0)
-      (effects (font (size 1.27 1.27)) (justify left top))
-    )
-    (pin "Button1" output (at 201.93 69.85 180)
-      (effects (font (size 1.27 1.27)) (justify left))
-    )
-    (pin "Button4" output (at 201.93 77.47 180)
-      (effects (font (size 1.27 1.27)) (justify left))
-    )
-    (pin "Button0" output (at 201.93 67.31 180)
-      (effects (font (size 1.27 1.27)) (justify left))
-    )
-    (pin "Button3" output (at 201.93 74.93 180)
-      (effects (font (size 1.27 1.27)) (justify left))
-    )
-    (pin "Button5" output (at 201.93 80.01 180)
-      (effects (font (size 1.27 1.27)) (justify left))
-    )
-    (pin "Button2" output (at 201.93 72.39 180)
+  (sheet (at 199.39 64.77) (size 34.29 17.78) (fields_autoplaced)
+    (stroke (width 0.1524) (type solid))
+    (fill (color 0 0 0 0.0000))
+    (property "Sheetname" "Buttons" (at 199.39 64.0584 0)
+      (effects (font (size 1.27 1.27)) (justify left bottom))
+    )
+    (property "Sheetfile" "buttons.kicad_sch" (at 199.39 83.1346 0)
+      (effects (font (size 1.27 1.27)) (justify left top) hide)
+    )
+    (pin "Button1" output (at 199.39 69.85 180)
+      (effects (font (size 1.27 1.27)) (justify left))
+    )
+    (pin "Button4" output (at 199.39 77.47 180)
+      (effects (font (size 1.27 1.27)) (justify left))
+    )
+    (pin "Button0" output (at 199.39 67.31 180)
+      (effects (font (size 1.27 1.27)) (justify left))
+    )
+    (pin "Button3" output (at 199.39 74.93 180)
+      (effects (font (size 1.27 1.27)) (justify left))
+    )
+    (pin "Button5" output (at 199.39 80.01 180)
+      (effects (font (size 1.27 1.27)) (justify left))
+    )
+    (pin "Button2" output (at 199.39 72.39 180)
       (effects (font (size 1.27 1.27)) (justify left))
     )
@@
       (effects (font (size 1.27 1.27)) (justify right))
     )
-    (pin "{I2C0}" bidirectional (at 189.23 97.79 0)
+    (pin "{I2C0}" bidirectional (at 189.23 111.76 0)
+      (effects (font (size 1.27 1.27)) (justify right))
+    )
+    (pin "{SPI}" bidirectional (at 189.23 116.84 0)
+      (effects (font (size 1.27 1.27)) (justify right))
+    )
+    (pin "GPIO11" bidirectional (at 189.23 101.6 0)
+      (effects (font (size 1.27 1.27)) (justify right))
+    )
+    (pin "GPIO12" bidirectional (at 189.23 134.62 0)
+      (effects (font (size 1.27 1.27)) (justify right))
+    )
+    (pin "GPIO10" bidirectional (at 189.23 99.06 0)
+      (effects (font (size 1.27 1.27)) (justify right))
+    )
+    (pin "NEOPIX_DRIVE" output (at 189.23 107.95 0)
+      (effects (font (size 1.27 1.27)) (justify right))
+    )
+    (pin "GPIO5" bidirectional (at 189.23 80.01 0)
+      (effects (font (size 1.27 1.27)) (justify right))
+    )
+    (pin "GPIO4" bidirectional (at 189.23 77.47 0)
+      (effects (font (size 1.27 1.27)) (justify right))
+    )
+    (pin "GPIO3" bidirectional (at 189.23 74.93 0)
+      (effects (font (size 1.27 1.27)) (justify right))
+    )
+    (pin "GPIO6" bidirectional (at 189.23 88.9 0)
+      (effects (font (size 1.27 1.27)) (justify right))
+    )
+    (pin "GPIO8" bidirectional (at 189.23 93.98 0)
+      (effects (font (size 1.27 1.27)) (justify right))
+    )
+    (pin "GPIO7" bidirectional (at 189.23 91.44 0)
+      (effects (font (size 1.27 1.27)) (justify right))
+    )
+    (pin "ENC_A" input (at 189.23 120.65 0)
+      (effects (font (size 1.27 1.27)) (justify right))
+    )
+    (pin "ENC_B" input (at 189.23 123.19 0)
+      (effects (font (size 1.27 1.27)) (justify right))
+    )
+    (pin "GPIO9" bidirectional (at 189.23 96.52 0)
+      (effects (font (size 1.27 1.27)) (justify right))
+    )
+    (pin "{I2C1}" bidirectional (at 189.23 129.54 0)
       (effects (font (size 1.27 1.27)) (justify right))
     )
@@
       )
     )
+  )
+  (sheet (at 199.39 86.36) (size 34.29 17.78) (fields_autoplaced)
+    (stroke (width 0.1524) (type solid))
+    (fill (color 0 0 0 0.0000))
+    (property "Sheetname" "Buttons1" (at 199.39 85.6484 0)
+      (effects (font (size 1.27 1.27)) (justify left bottom))
+    )
+    (property "Sheetfile" "buttons.kicad_sch" (at 199.39 104.7246 0)
+      (effects (font (size 1.27 1.27)) (justify left top) hide)
+    )
+    (pin "Button1" output (at 199.39 91.44 180)
+      (effects (font (size 1.27 1.27)) (justify left))
+    )
+    (pin "Button4" output (at 199.39 99.06 180)
+      (effects (font (size 1.27 1.27)) (justify left))
+    )
+    (pin "Button0" output (at 199.39 88.9 180)
+      (effects (font (size 1.27 1.27)) (justify left))
+    )
+    (pin "Button3" output (at 199.39 96.52 180)
+      (effects (font (size 1.27 1.27)) (justify left))
+    )
+    (pin "Button5" output (at 199.39 101.6 180)
+      (effects (font (size 1.27 1.27)) (justify left))
+    )
+    (pin "Button2" output (at 199.39 93.98 180)
+      (effects (font (size 1.27 1.27)) (justify left))
+    )
+    (instances
+      (project "000018 PGKB"
+        (path "/e63e39d7-6ac0-4ffd-8aa3-1841a4541b55/2eb44e1a-4042-4ea6-aca2-4836a6ec84e9" (page "12"))
+      )
+    )

Commit message: ledit
Other:
- removed sheet Buttons1
- added sheet Neopixel LEDs (LEDS_Neopixel.kicad_sch)
- added sheet Other Controls (controls.kicad_sch)
- sheet Buttons ports: added Button6, Button7, Button8; removed none
- sheet Microcontroller ports: added none; removed GPIO10, GPIO11, GPIO9

Commit message: updates
Other:
- sheet Buttons ports: added Button9; removed none
- sheet Microcontroller ports: added GPIO9; removed none
- sheet Neopixel LEDs ports: added NEOPIXEL_VDD; removed none
Changed lines of the file:
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@@
   )
   (bus_alias "I2C" (members "SDA" "SCL"))
+  (junction (at 87.63 78.74) (diameter 0) (color 0 0 0 0)
+  )
+  (wire (pts (xy 143.51 78.74) (xy 151.13 78.74))
+    (stroke (width 0) (type default))
+  )
   (wire (pts (xy 189.23 87.63) (xy 199.39 87.63))
     (stroke (width 0) (type default))
@@
     (stroke (width 0) (type default))
   )
-  (wire (pts (xy 189.23 99.06) (xy 199.39 99.06))
+  (wire (pts (xy 189.23 107.95) (xy 199.39 107.95))
+    (stroke (width 0) (type default))
+  )
+  (wire (pts (xy 189.23 90.17) (xy 199.39 90.17))
     (stroke (width 0) (type default))
   )
@@
     (stroke (width 0) (type default))
   )
-  (wire (pts (xy 87.63 90.17) (xy 87.63 52.07))
+  (wire (pts (xy 87.63 90.17) (xy 87.63 78.74))
     (stroke (width 0) (type default))
   )
@@
     (stroke (width 0) (type default))
   )
-  (wire (pts (xy 189.23 96.52) (xy 199.39 96.52))
+  (wire (pts (xy 87.63 78.74) (xy 105.41 78.74))
+    (stroke (width 0) (type default))
+  )
+  (wire (pts (xy 87.63 78.74) (xy 87.63 52.07))
+    (stroke (width 0) (type default))
+  )
+  (wire (pts (xy 189.23 105.41) (xy 199.39 105.41))
     (stroke (width 0) (type default))
   )
@@
     (stroke (width 0) (type default))
   )
-  (wire (pts (xy 189.23 102.87) (xy 199.39 102.87))
+  (wire (pts (xy 189.23 111.76) (xy 199.39 111.76))
     (stroke (width 0) (type default))
   )
@@
     )
   )
-  (sheet (at 109.22 76.2) (size 34.29 11.43) (fields_autoplaced)
-    (stroke (width 0.1524) (type solid))
-    (fill (color 0 0 0 0.0000))
-    (property "Sheetname" "Neopixel LEDs" (at 109.22 75.4884 0)
-      (effects (font (size 1.27 1.27)) (justify left bottom))
-    )
-    (property "Sheetfile" "LEDS_Neopixel.kicad_sch" (at 109.22 88.2146 0)
+  (sheet (at 105.41 76.2) (size 38.1 11.43) (fields_autoplaced)
+    (stroke (width 0.1524) (type solid))
+    (fill (color 0 0 0 0.0000))
+    (property "Sheetname" "Neopixel LEDs" (at 105.41 75.4884 0)
+      (effects (font (size 1.27 1.27)) (justify left bottom))
+    )
+    (property "Sheetfile" "LEDS_Neopixel.kicad_sch" (at 105.41 88.2146 0)
       (effects (font (size 1.27 1.27)) (justify left top) hide)
     )
@@
       (effects (font (size 1.27 1.27)) (justify right))
     )
-    (instances
-      (project "000018 PGKB"
-        (path "/e63e39d7-6ac0-4ffd-8aa3-1841a4541b55/2eb44e1a-4042-4ea6-aca2-4836a6ec84e9" (page "13"))
+    (pin "NEOPIXEL_VDD" input (at 105.41 78.74 180)
+      (effects (font (size 1.27 1.27)) (justify left))
+    )
+    (instances
+      (project "000018 PGKB"
+        (path "/e63e39d7-6ac0-4ffd-8aa3-1841a4541b55/2eb44e1a-4042-4ea6-aca2-4836a6ec84e9" (page "5"))
       )
     )
@@
     )
   )
-  (sheet (at 199.39 64.77) (size 34.29 25.4) (fields_autoplaced)
+  (sheet (at 199.39 64.77) (size 34.29 27.94) (fields_autoplaced)
     (stroke (width 0.1524) (type solid))
     (fill (color 0 0 0 0.0000))
@@
       (effects (font (size 1.27 1.27)) (justify left bottom))
     )
-    (property "Sheetfile" "buttons.kicad_sch" (at 199.39 90.7546 0)
+    (property "Sheetfile" "buttons.kicad_sch" (at 199.39 93.2946 0)
       (effects (font (size 1.27 1.27)) (justify left top) hide)
     )
@@
     )
     (pin "Button8" output (at 199.39 87.63 180)
+      (effects (font (size 1.27 1.27)) (justify left))
+    )
+    (pin "Button9" output (at 199.39 90.17 180)
       (effects (font (size 1.27 1.27)) (justify left))
     )
@@
     )
   )
-  (sheet (at 199.39 93.98) (size 34.29 11.43) (fields_autoplaced)
-    (stroke (width 0.1524) (type solid))
-    (fill (color 0 0 0 0.0000))
-    (property "Sheetname" "Other Controls" (at 199.39 93.2684 0)
-      (effects (font (size 1.27 1.27)) (justify left bottom))
-    )
-    (property "Sheetfile" "controls.kicad_sch" (at 199.39 105.9946 0)
-      (effects (font (size 1.27 1.27)) (justify left top) hide)
-    )
-    (pin "ENC_B" output (at 199.39 99.06 180)
-      (effects (font (size 1.27 1.27)) (justify left))
-    )
-    (pin "SWITCH" output (at 199.39 102.87 180)
-      (effects (font (size 1.27 1.27)) (justify left))
-    )
-    (pin "ENC_A" output (at 199.39 96.52 180)
+  (sheet (at 199.39 102.87) (size 34.29 11.43) (fields_autoplaced)
+    (stroke (width 0.1524) (type solid))
+    (fill (color 0 0 0 0.0000))
+    (property "Sheetname" "Other Controls" (at 199.39 102.1584 0)
+      (effects (font (size 1.27 1.27)) (justify left bottom))
+    )
+    (property "Sheetfile" "controls.kicad_sch" (at 199.39 114.8846 0)
+      (effects (font (size 1.27 1.27)) (justify left top) hide)
+    )
+    (pin "ENC_B" output (at 199.39 107.95 180)
+      (effects (font (size 1.27 1.27)) (justify left))
+    )
+    (pin "SWITCH" output (at 199.39 111.76 180)
+      (effects (font (size 1.27 1.27)) (justify left))
+    )
+    (pin "ENC_A" output (at 199.39 105.41 180)
       (effects (font (size 1.27 1.27)) (justify left))
     )
@@
       (effects (font (size 1.27 1.27)) (justify left))
     )
-    (pin "GPIO12" bidirectional (at 189.23 102.87 0)
+    (pin "GPIO12" bidirectional (at 189.23 111.76 0)
       (effects (font (size 1.27 1.27)) (justify right))
     )
@@
       (effects (font (size 1.27 1.27)) (justify right))
     )
-    (pin "ENC_A" input (at 189.23 96.52 0)
-      (effects (font (size 1.27 1.27)) (justify right))
-    )
-    (pin "ENC_B" input (at 189.23 99.06 0)
+    (pin "ENC_A" input (at 189.23 105.41 0)
+      (effects (font (size 1.27 1.27)) (justify right))
+    )
+    (pin "ENC_B" input (at 189.23 107.95 0)
       (effects (font (size 1.27 1.27)) (justify right))
     )
@@
       (effects (font (size 1.27 1.27)) (justify right))
     )
+    (pin "GPIO9" bidirectional (at 189.23 90.17 0)
+      (effects (font (size 1.27 1.27)) (justify right))
+    )

Commit message: Leiskaa
Other:
- sheet Buttons ports: added Button10, Button11; removed none
- sheet Connectors ports: added {I2C1}; removed {I2C}
- sheet Microcontroller ports: added GPIO10, GPIO11; removed none
Changed lines of the file:
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@@
+    (stroke (width 0) (type default))
+  )
+  (wire (pts (xy 189.23 92.71) (xy 199.39 92.71))
     (stroke (width 0) (type default))
   )
@@
     (stroke (width 0) (type default))
   )
+  (wire (pts (xy 189.23 95.25) (xy 199.39 95.25))
+    (stroke (width 0) (type default))
+  )
   (wire (pts (xy 189.23 85.09) (xy 199.39 85.09))
     (stroke (width 0) (type default))
@@
     (stroke (width 0) (type default))
   )
+  (wire (pts (xy 87.63 78.74) (xy 105.41 78.74))
+    (stroke (width 0) (type default))
+  )
+  (wire (pts (xy 87.63 78.74) (xy 87.63 52.07))
+    (stroke (width 0) (type default))
+  )
+  (wire (pts (xy 189.23 105.41) (xy 199.39 105.41))
+    (stroke (width 0) (type default))
+  )
+  (wire (pts (xy 189.23 77.47) (xy 199.39 77.47))
+    (stroke (width 0) (type default))
+  )
   (bus (pts (xy 189.23 130.81) (xy 199.39 130.81))
-    (stroke (width 0) (type default))
-  )
-  (wire (pts (xy 87.63 78.74) (xy 105.41 78.74))
-    (stroke (width 0) (type default))
-  )
-  (wire (pts (xy 87.63 78.74) (xy 87.63 52.07))
-    (stroke (width 0) (type default))
-  )
-  (wire (pts (xy 189.23 105.41) (xy 199.39 105.41))
-    (stroke (width 0) (type default))
-  )
-  (wire (pts (xy 189.23 77.47) (xy 199.39 77.47))
     (stroke (width 0) (type default))
   )
@@
       (effects (font (size 1.27 1.27)) (justify left top) hide)
     )
-    (pin "{I2C}" bidirectional (at 199.39 130.81 180)
+    (pin "{I2C1}" bidirectional (at 199.39 130.81 180)
       (effects (font (size 1.27 1.27)) (justify left))
     )
@@
     )
   )
-  (sheet (at 199.39 64.77) (size 34.29 27.94) (fields_autoplaced)
+  (sheet (at 199.39 64.77) (size 34.29 34.29) (fields_autoplaced)
     (stroke (width 0.1524) (type solid))
     (fill (color 0 0 0 0.0000))
@@
       (effects (font (size 1.27 1.27)) (justify left bottom))
     )
-    (property "Sheetfile" "buttons.kicad_sch" (at 199.39 93.2946 0)
+    (property "Sheetfile" "buttons.kicad_sch" (at 199.39 99.6446 0)
       (effects (font (size 1.27 1.27)) (justify left top) hide)
     )
@@
     )
     (pin "Button9" output (at 199.39 90.17 180)
+      (effects (font (size 1.27 1.27)) (justify left))
+    )
+    (pin "Button11" output (at 199.39 95.25 180)
+      (effects (font (size 1.27 1.27)) (justify left))
+    )
+    (pin "Button10" output (at 199.39 92.71 180)
       (effects (font (size 1.27 1.27)) (justify left))
     )
@@
       (effects (font (size 1.27 1.27)) (justify right))
     )
+    (pin "GPIO11" bidirectional (at 189.23 95.25 0)
+      (effects (font (size 1.27 1.27)) (justify right))
+    )
+    (pin "GPIO10" bidirectional (at 189.23 92.71 0)
+      (effects (font (size 1.27 1.27)) (justify right))
+    )

Commit message: error fixing
Connections:
- no-connect marks 0 -> 3
Other:
- sheet Buttons ports: added none; removed Button0
Changed lines of the file:
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@@
   (title_block
     (title "Programmable Keyboard")
-    (date "2023-10-14")
+    (date "2023-10-19")
     (rev "1.0")
     (company "Kallio Designs Oy")
@@
   (junction (at 87.63 78.74) (diameter 0) (color 0 0 0 0)
   )
+  (no_connect (at 189.23 67.31))
+  (no_connect (at 151.13 125.73))
+  (no_connect (at 151.13 120.65))
   (wire (pts (xy 143.51 78.74) (xy 151.13 78.74))
     (stroke (width 0) (type default))
@@
   )
   (wire (pts (xy 189.23 69.85) (xy 199.39 69.85))
-    (stroke (width 0) (type default))
-  )
-  (wire (pts (xy 189.23 67.31) (xy 199.39 67.31))
     (stroke (width 0) (type default))
   )
@@
     )
   )
-  (sheet (at 199.39 64.77) (size 34.29 34.29) (fields_autoplaced)
+  (sheet (at 199.39 66.04) (size 34.29 33.02) (fields_autoplaced)
     (stroke (width 0.1524) (type solid))
     (fill (color 0 0 0 0.0000))
-    (property "Sheetname" "Buttons" (at 199.39 64.0584 0)
+    (property "Sheetname" "Buttons" (at 199.39 65.3284 0)
       (effects (font (size 1.27 1.27)) (justify left bottom))
     )
@@
       (effects (font (size 1.27 1.27)) (justify left))
     )
-    (pin "Button0" output (at 199.39 67.31 180)
-      (effects (font (size 1.27 1.27)) (justify left))
-    )
