File: PCB/Rev 02.00/000018 PGKB/mcu.kicad_sch (KiCad schematic)
At the start: 15 parts, among them U3 RP2040, Y1 8 MHz

Commit message: buttons
Connections:
- net GPIO0: now reaches U3.2 (GPIO0)
- net GPIO1: now reaches U3.3 (GPIO1)
- net GPIO2: now reaches U3.4 (GPIO2)
Changed lines of the file:
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@@
     (comment 3 "PCB_PN")
   )
+  (bus_alias "SPI" (members "CLK" "MISO" "MOSI" "~{CS}_SDCARD"))
   (bus_alias "QSPI" (members "DATA0" "DATA1" "DATA2" "DATA3" "~{CS}_MEMORY" "CLK"))
   (bus_alias "I2C" (members "SDA" "SCL"))
-  (bus_alias "SPI" (members "CLK" "MISO" "MOSI" "~{CS}_SDCARD"))
   (junction (at 63.5 121.92) (diameter 0) (color 0 0 0 0)
   )
@@
     (stroke (width 0) (type default))
   )
+  (wire (pts (xy 177.8 69.85) (xy 162.56 69.85))
+    (stroke (width 0) (type default))
+  )
+  (wire (pts (xy 177.8 67.31) (xy 162.56 67.31))
+    (stroke (width 0) (type default))
+  )
   (wire (pts (xy 137.16 152.4) (xy 137.16 151.13))
     (stroke (width 0) (type default))
@@
   )
   (wire (pts (xy 63.5 127) (xy 66.04 127))
+    (stroke (width 0) (type default))
+  )
+  (wire (pts (xy 177.8 72.39) (xy 162.56 72.39))
     (stroke (width 0) (type default))
   )
@@
     (effects (font (size 1.27 1.27)) (justify left bottom))
   )
-  (label "DATA0" (at 111.76 90.17 180)
+  (label "DATA0" (at 111.76 90.17 180) (fields_autoplaced)
     (effects (font (size 1.27 1.27)) (justify right bottom))
   )
@@
     (effects (font (size 1.27 1.27)) (justify right))
   )
+  (hierarchical_label "GPIO2" (shape bidirectional) (at 177.8 72.39 0) (fields_autoplaced)
+    (effects (font (size 1.27 1.27)) (justify left))
+  )
+  (hierarchical_label "GPIO1" (shape bidirectional) (at 177.8 69.85 0) (fields_autoplaced)
+    (effects (font (size 1.27 1.27)) (justify left))
+  )
+  (hierarchical_label "GPIO0" (shape bidirectional) (at 177.8 67.31 0) (fields_autoplaced)
+    (effects (font (size 1.27 1.27)) (justify left))
+  )
   (symbol (lib_id "power:GND") (at 71.12 39.37 0) (mirror y) (unit 1)

Commit message: schematic
Parts:
- removed C1: 100n, KD_Capacitor:CAPC1608X90N, symbol KD_Capacitor:C_0603_100n_X7R_50V
- removed Y1: 8 MHz, KD_Oscillator:OSCCC320X250X70_M, symbol KD_Oscillator:XO_8M_Jauch_O_8_0-JO32-B-1V3-1-T1-LF
- added C12, C7: 27p, KD_Capacitor:CAPC1608X90N, symbol KD_Capacitor:C_0603_27p_NP0_5%_50V
- added C2 (x7): 100n, KD_Capacitor:CAPC1608X90N, symbol KD_Capacitor:C_0603_100n_X7R_50V
- added C4 (x2): 1u, KD_Capacitor:CAPC2012X135N, symbol KD_Capacitor:C_0805_1u_X7R_25V
- added D5: Schottky_30V_200mA_DCo_BAT54WS, KD_Diode:D_SOD-323, symbol KD_Diode:Schottky_30V_200mA_DCo_BAT54WS
- added R12, R13: 1k, KD_Resistor:RESC1608X55N, symbol KD_Resistor:R_0603_1k_1%
- added TP7, TP8, TP9: TP D2.5 mm H0.9mm, KD_Connector_Pads:TestPoint_Pad_D2.5mm_H0.9mm, symbol KD_Connector_Pads:TestPoint_2.5mm_H0.9
- added Y1: 12 MHz, KD_Oscillator:OSCCC320X250X70_M, symbol KD_Oscillator:Crystal_12M_RH100-12.000-18-2020-EXT-TR
- R5: footprint KD_Resistor:RESC1608X55N -> KD_Resistor:RESC1608X55N_DNP; symbol KD_Resistor:R_0603_22k_1% -> KD_Resistor:R_0603_DNP; Code 22k -> DNP; DNP F -> T; MFG_PartNo 311-22.0KHRCT-ND -> DNP; Manufacturer YAGEO -> DNP; Price 0.01 -> 0.00; Supplier Digi-Key -> DNP; Supplier_PartNo 311-22.0KHRCT-ND -> DNP
Connections:
- net BOOT is gone; now on net USBBOOT: S2.3
- net +3V3: now also FB3.1
- net GND: now also U3.19 (TESTEN), C12.2, C2.2, C2.2, C2.2, C2.2, C2.2, C2.2, C2.2, C4.2, C4.2, C7.2, Y1.2 (GND), Y1.4 (GND)
- net SCL: now also R38.2, TP5.1, U3.37 (GPIO25); no longer R37.2, TP6.1
- net SDA: now also R37.2, TP6.1, U3.36 (GPIO24); no longer R38.2, TP5.1
- net ~{CS}_MEMORY: now also D5.2 (A)
- net ~{RESET}: now also TP9.1
- net at U3.1 (IOVDD), U3.10 (IOVDD), U3.22 (IOVDD)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: now also C2.1, C4.1, FB3.2, U3.43 (ADC_AVDD), U3.44 (VREG_IN), U3.48 (USB_VDD), C2.1, C2.1, C2.1, C2.1, C2.1, C4.1
- net at U3.20 (XIN): now also C7.1, Y1.1
- net at U3.21 (XOUT): now also R12.2
- net 1V2: now reaches U3.23 (DVDD), U3.50 (DVDD)
- net 1V2: now also U3.45 (VREG_VOUT), C2.1, C2.1, C4.1, TP7.1
- net UART_TX: now reaches U3.30 (GPIO19)
- net USBBOOT: now reaches U3.32 (GPIO21)
- net USBBOOT: now also R13.2, TP8.1
- net I2C1_SDA: now reaches U3.34 (GPIO22)
- net I2C1_SCL: now reaches U3.35 (GPIO23)
- net SPI_MOSI: now reaches U3.5 (GPIO3)
- net SPI_MISO: now reaches U3.6 (GPIO4)
- net UART_RX: now reaches U3.7 (GPIO5)
- net SPI_CLK: now reaches U3.8 (GPIO6)
- new net: C12.1, R12.1, Y1.3
- new net: D5.1 (K), R13.1
Other:
- note removed: "MINKÄ TAAJUNEN OSKILLAATTORI PITÄS OLLA?"
- moved on the sheet: C2, C4, FB3, R37, R38, S2, TP5, TP6

Commit message: Schematic
Connections:
- net DEBUG_LED_BLUE: now also U3.15 (GPIO12)
- net DEBUG_LED_GREEN: now also U3.13 (GPIO10)
- net DEBUG_LED_RED: now also U3.14 (GPIO11)
- net GPIO4: now reaches U3.11 (GPIO8)
- net GPIO5: now reaches U3.12 (GPIO9)
- net GPIO6: now reaches U3.16 (GPIO13)
- net GPIO7: now reaches U3.17 (GPIO14)
- net GPIO8: now reaches U3.18 (GPIO15)
- net GPIO9: now reaches U3.27 (GPIO16)
- net ENC_A: now reaches U3.28 (GPIO17)
- net ENC_B: now reaches U3.29 (GPIO18)
- net GPIO10: now reaches U3.39 (GPIO27_ADC1)
- net GPIO11: now reaches U3.40 (GPIO28_ADC2)
- net GPIO12: now reaches U3.41 (GPIO29_ADC3)
- net GPIO3: now reaches U3.9 (GPIO7)
Other:
- company: 4D Haptics Oy -> Kallio Designs Oy
- title: Suspension Rig -> Programmable Keyboard
Changed lines of the file:
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@@
   (paper "A4")
   (title_block
-    (title "Suspension Rig")
-    (date "2023-09-25")
+    (title "Programmable Keyboard")
+    (date "2023-10-14")
     (rev "1.0")
-    (company "4D Haptics Oy")
-    (comment 1 "TL, SB")
+    (company "Kallio Designs Oy")
+    (comment 1 "TL, NH")
     (comment 3 "PCB_PN")
   )
+  (bus_alias "I2C0" (members "SDA" "SCL"))
+  (bus_alias "I2C1" (members "I2C1_SDA" "I2C1_SCL"))
   (bus_alias "QSPI" (members "DATA0" "DATA1" "DATA2" "DATA3" "~{CS}_MEMORY" "CLK"))
-  (bus_alias "I2C1" (members "I2C1_SDA" "I2C1_SCL"))
-  (bus_alias "I2C0" (members "SDA" "SCL"))
   (bus_alias "SPI" (members "SPI_CLK" "SPI_MISO" "SPI_MOSI" "SPI_CS0"))
   (junction (at 142.24 57.15) (diameter 0) (color 0 0 0 0)
@@
     (stroke (width 0) (type default))
   )
-  (wire (pts (xy 177.8 69.85) (xy 162.56 69.85))
-    (stroke (width 0) (type default))
-  )
-  (wire (pts (xy 177.8 67.31) (xy 162.56 67.31))
+  (wire (pts (xy 187.96 69.85) (xy 162.56 69.85))
+    (stroke (width 0) (type default))
+  )
+  (wire (pts (xy 187.96 67.31) (xy 162.56 67.31))
     (stroke (width 0) (type default))
   )
@@
     (stroke (width 0) (type default))
   )
+  (wire (pts (xy 187.96 138.43) (xy 162.56 138.43))
+    (stroke (width 0) (type default))
+  )
   (bus (pts (xy 39.37 87.63) (xy 39.37 92.71))
     (stroke (width 0) (type default))
   )
+  (wire (pts (xy 162.56 113.03) (xy 185.42 113.03))
+    (stroke (width 0) (type default))
+  )
   (wire (pts (xy 162.56 74.93) (xy 248.92 74.93))
     (stroke (width 0) (type default))
@@
     (stroke (width 0) (type default))
   )
+  (wire (pts (xy 187.96 87.63) (xy 162.56 87.63))
+    (stroke (width 0) (type default))
+  )
   (wire (pts (xy 142.24 57.15) (xy 139.7 57.15))
     (stroke (width 0) (type default))
@@
     (stroke (width 0) (type default))
   )
+  (wire (pts (xy 187.96 143.51) (xy 162.56 143.51))
+    (stroke (width 0) (type default))
+  )
   (wire (pts (xy 109.22 64.77) (xy 109.22 67.31))
     (stroke (width 0) (type default))
@@
     (stroke (width 0) (type default))
   )
+  (wire (pts (xy 187.96 107.95) (xy 162.56 107.95))
+    (stroke (width 0) (type default))
+  )
   (wire (pts (xy 229.87 130.81) (xy 248.92 130.81))
     (stroke (width 0) (type default))
@@
     (stroke (width 0) (type default))
   )
+  (wire (pts (xy 163.83 92.71) (xy 162.56 92.71))
+    (stroke (width 0) (type default))
+  )
   (wire (pts (xy 83.82 67.31) (xy 88.9 67.31))
     (stroke (width 0) (type default))
@@
     (stroke (width 0) (type default))
   )
+  (wire (pts (xy 187.96 90.17) (xy 162.56 90.17))
+    (stroke (width 0) (type default))
+  )
   (bus (pts (xy 39.37 97.79) (xy 39.37 100.33))
     (stroke (width 0) (type default))
@@
     (stroke (width 0) (type default))
   )
+  (wire (pts (xy 163.83 95.25) (xy 162.56 95.25))
+    (stroke (width 0) (type default))
+  )
   (bus (pts (xy 251.46 130.81) (xy 251.46 133.35))
     (stroke (width 0) (type default))
@@
     (stroke (width 0) (type default))
   )
+  (wire (pts (xy 163.83 97.79) (xy 162.56 97.79))
+    (stroke (width 0) (type default))
+  )
   (wire (pts (xy 138.43 26.67) (xy 138.43 25.4))
     (stroke (width 0) (type default))
@@
     (stroke (width 0) (type default))
   )
+  (wire (pts (xy 162.56 110.49) (xy 185.42 110.49))
+    (stroke (width 0) (type default))
+  )
   (wire (pts (xy 147.32 25.4) (xy 147.32 57.15))
     (stroke (width 0) (type default))
@@
     (stroke (width 0) (type default))
   )
+  (wire (pts (xy 187.96 105.41) (xy 162.56 105.41))
+    (stroke (width 0) (type default))
+  )
   (wire (pts (xy 134.62 59.69) (xy 134.62 57.15))
     (stroke (width 0) (type default))
@@
     (stroke (width 0) (type default))
   )
+  (wire (pts (xy 187.96 100.33) (xy 162.56 100.33))
+    (stroke (width 0) (type default))
+  )
   (wire (pts (xy 168.91 21.59) (xy 168.91 20.32))
     (stroke (width 0) (type default))
@@
     (stroke (width 0) (type default))
   )
-  (wire (pts (xy 177.8 72.39) (xy 162.56 72.39))
+  (wire (pts (xy 187.96 72.39) (xy 162.56 72.39))
     (stroke (width 0) (type default))
   )
@@
     (stroke (width 0) (type default))
   )
+  (wire (pts (xy 187.96 140.97) (xy 162.56 140.97))
+    (stroke (width 0) (type default))
+  )
   (bus (pts (xy 254 134.62) (xy 251.46 134.62))
     (stroke (width 0) (type default))
   )
+  (wire (pts (xy 187.96 102.87) (xy 162.56 102.87))
+    (stroke (width 0) (type default))
+  )
   (wire (pts (xy 92.71 25.4) (xy 104.14 25.4))
     (stroke (width 0) (type default))
@@
   )
   (wire (pts (xy 39.37 149.86) (xy 38.1 149.86))
+    (stroke (width 0) (type default))
+  )
+  (wire (pts (xy 187.96 85.09) (xy 162.56 85.09))
     (stroke (width 0) (type default))
   )
@@
     (effects (font (size 1.27 1.27)) (justify left bottom))
   )
-  (label "DEBUG_LED_GREEN" (at 177.8 100.33 0) (fields_autoplaced)
+  (label "DEBUG_LED_GREEN" (at 163.83 92.71 0) (fields_autoplaced)
     (effects (font (size 1.27 1.27)) (justify left bottom))
   )
@@
     (effects (font (size 1.27 1.27)) (justify left bottom))
   )
-  (label "TP1" (at 177.8 95.25 0) (fields_autoplaced)
-    (effects (font (size 1.27 1.27)) (justify left bottom))
-  )
   (label "DEBUG_LED_BLUE" (at 231.14 27.94 0) (fields_autoplaced)
     (effects (font (size 1.27 1.27)) (justify left bottom))
   )
-  (label "TP10" (at 177.8 92.71 0) (fields_autoplaced)
-    (effects (font (size 1.27 1.27)) (justify left bottom))
-  )
   (label "~{CS}_MEMORY" (at 34.29 170.18 0) (fields_autoplaced)
     (effects (font (size 1.27 1.27)) (justify left bottom))
@@
     (effects (font (size 1.27 1.27)) (justify left bottom))
   )
-  (label "DEBUG_LED_BLUE" (at 177.8 102.87 0) (fields_autoplaced)
+  (label "DEBUG_LED_BLUE" (at 163.83 97.79 0) (fields_autoplaced)
     (effects (font (size 1.27 1.27)) (justify left bottom))
   )
@@
     (effects (font (size 1.27 1.27)) (justify left bottom))
   )
-  (label "DEBUG_LED_RED" (at 177.8 97.79 0) (fields_autoplaced)
+  (label "DEBUG_LED_RED" (at 163.83 95.25 0) (fields_autoplaced)
     (effects (font (size 1.27 1.27)) (justify left bottom))
   )
@@
   (label "~{RESET}" (at 57.15 149.86 180) (fields_autoplaced)
     (effects (font (size 1.27 1.27)) (justify right bottom))
+  )
+  (hierarchical_label "GPIO9" (shape bidirectional) (at 187.96 107.95 0) (fields_autoplaced)
+    (effects (font (size 1.27 1.27)) (justify left))
+  )
+  (hierarchical_label "GPIO11" (shape bidirectional) (at 187.96 140.97 0) (fields_autoplaced)
+    (effects (font (size 1.27 1.27)) (justify left))
   )
   (hierarchical_label "{I2C0}" (shape bidirectional) (at 254 134.62 0) (fields_autoplaced)
@@
     (effects (font (size 1.27 1.27)) (justify right))
   )
+  (hierarchical_label "GPIO12" (shape bidirectional) (at 187.96 143.51 0) (fields_autoplaced)
+    (effects (font (size 1.27 1.27)) (justify left))
+  )
+  (hierarchical_label "GPIO5" (shape bidirectional) (at 187.96 90.17 0) (fields_autoplaced)
+    (effects (font (size 1.27 1.27)) (justify left))
+  )
+  (hierarchical_label "GPIO6" (shape bidirectional) (at 187.96 100.33 0) (fields_autoplaced)
+    (effects (font (size 1.27 1.27)) (justify left))
+  )
+  (hierarchical_label "GPIO8" (shape bidirectional) (at 187.96 105.41 0) (fields_autoplaced)
+    (effects (font (size 1.27 1.27)) (justify left))
+  )
   (hierarchical_label "{I2C1}" (shape bidirectional) (at 190.5 125.73 0) (fields_autoplaced)
     (effects (font (size 1.27 1.27)) (justify left))
@@
     (effects (font (size 1.27 1.27)) (justify right))
   )
-  (hierarchical_label "GPIO2" (shape bidirectional) (at 177.8 72.39 0) (fields_autoplaced)
+  (hierarchical_label "GPIO2" (shape bidirectional) (at 187.96 72.39 0) (fields_autoplaced)
+    (effects (font (size 1.27 1.27)) (justify left))
+  )
+  (hierarchical_label "ENC_B" (shape input) (at 185.42 113.03 0) (fields_autoplaced)
     (effects (font (size 1.27 1.27)) (justify left))
   )
@@
     (effects (font (size 1.27 1.27)) (justify left))
   )
-  (hierarchical_label "GPIO1" (shape bidirectional) (at 177.8 69.85 0) (fields_autoplaced)
-    (effects (font (size 1.27 1.27)) (justify left))
-  )
-  (hierarchical_label "GPIO0" (shape bidirectional) (at 177.8 67.31 0) (fields_autoplaced)
-    (effects (font (size 1.27 1.27)) (justify left))
-  )
+  (hierarchical_label "GPIO1" (shape bidirectional) (at 187.96 69.85 0) (fields_autoplaced)
+    (effects (font (size 1.27 1.27)) (justify left))
+  )
+  (hierarchical_label "GPIO7" (shape bidirectional) (at 187.96 102.87 0) (fields_autoplaced)
+    (effects (font (size 1.27 1.27)) (justify left))
+  )
+  (hierarchical_label "GPIO4" (shape bidirectional) (at 187.96 87.63 0) (fields_autoplaced)
+    (effects (font (size 1.27 1.27)) (justify left))
+  )
+  (hierarchical_label "ENC_A" (shape input) (at 185.42 110.49 0) (fields_autoplaced)
+    (effects (font (size 1.27 1.27)) (justify left))
+  )
+  (hierarchical_label "GPIO10" (shape bidirectional) (at 187.96 138.43 0) (fields_autoplaced)
+    (effects (font (size 1.27 1.27)) (justify left))
+  )
+  (hierarchical_label "GPIO0" (shape bidirectional) (at 187.96 67.31 0) (fields_autoplaced)
+    (effects (font (size 1.27 1.27)) (justify left))
+  )
+  (hierarchical_label "GPIO3" (shape bidirectional) (at 187.96 85.09 0) (fields_autoplaced)
+    (effects (font (size 1.27 1.27)) (justify left))
+  )
