File: PCB/Rev 02.00/000018 PGKB/mcu.kicad_sch (KiCad schematic)
At the start: 31 parts, among them U3 RP2040, Y1 12 MHz

Commit message: updates
Parts:
- removed TP4: TestPoint_1.5mm_Round, KD_Connector_Pads:TestPoint_Pad_D1.5mm, symbol KD_Connector_Pads:TestPoint_1.5mm_Round
- renumbered C7 to C27, C12 to C30, D5 to D3, FB3 to FB2, R13 to R23, R5 to R24, R12 to R25, S2 to S12, S1 to S13, TP5 to TP11, TP6 to TP12, TP7 to TP6, TP8 to TP7, TP9 to TP8, TP3 to TP9, U3 to U5
Connections:
- net TP10: now also U5.31 (GPIO20)
- net DEBUG_LED_BLUE: no longer names the net of U5.15 (GPIO12)
- net DEBUG_LED_GREEN: no longer names the net of U5.13 (GPIO10)
- net DEBUG_LED_RED: no longer names the net of U5.14 (GPIO11)
- no-connect marks 4 -> 9
Other:
- removed sheet LEDs
