File: PCB/Rev 02.00/000018 PGKB/mcu.kicad_sch (KiCad schematic)
At the start: 30 parts, among them U5 RP2040, Y1 12 MHz

Commit message: Layout
Parts:
- renumbered D3 to D13
Changed lines of the file:
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@@
   (symbol (lib_id "KD_Diode:Schottky_30V_200mA_DCo_BAT54WS") (at 50.8 170.18 180) (unit 1)
     (in_bom yes) (on_board yes) (dnp no) (fields_autoplaced)
-    (property "Reference" "D3" (at 51.1175 163.83 0)
+    (property "Reference" "D13" (at 51.1175 163.83 0)
       (effects (font (size 1.27 1.27)))
     )
@@
       (project "000018 PGKB"
         (path "/e63e39d7-6ac0-4ffd-8aa3-1841a4541b55/2eb44e1a-4042-4ea6-aca2-4836a6ec84e9/a467c90b-3665-441c-9913-5c8fd91b3b4b"
-          (reference "D3") (unit 1)
+          (reference "D13") (unit 1)
         )
       )

Commit message: step
Parts:
- R37, R38: value R_0805_4700_5% -> 4k7; footprint KD_Resistor:RESC2012X50N -> KD_Resistor:RESC1005X40N; symbol KD_Resistor:R_0805_4700_5% -> KD_Resistor:R_0402_4700_1%; MFG_PartNo RMCF0805JT4K70 -> CR0402-FX-4701GLF; Manufacturer Stackpole Electronics Inc -> Bourns Inc.; Supplier_PartNo RMCF0805JT4K70CT-ND -> CR0402-FX-4701GLFCT-ND
Changed lines of the file:
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@@
     (comment 3 "PCB_PN")
   )
+  (bus_alias "QSPI" (members "DATA0" "DATA1" "DATA2" "DATA3" "~{CS}_MEMORY" "CLK"))
   (bus_alias "I2C0" (members "SDA" "SCL"))
   (bus_alias "SPI" (members "SPI_CLK" "SPI_MISO" "SPI_MOSI" "SPI_CS0"))
-  (bus_alias "QSPI" (members "DATA0" "DATA1" "DATA2" "DATA3" "~{CS}_MEMORY" "CLK"))
   (bus_alias "I2C1" (members "I2C1_SDA" "I2C1_SCL"))
   (junction (at 142.24 57.15) (diameter 0) (color 0 0 0 0)
@@
     )
   )
-  (symbol (lib_id "KD_Resistor:R_0805_4700_5%") (at 209.55 116.84 0) (unit 1)
+  (symbol (lib_id "KD_Resistor:R_0402_4700_1%") (at 209.55 116.84 0) (unit 1)
     (in_bom yes) (on_board yes) (dnp no) (fields_autoplaced)
     (property "Reference" "R37" (at 212.09 115.57 0)
       (effects (font (size 1.27 1.27)) (justify left))
     )
-    (property "Value" "R_0805_4700_5%" (at 196.85 85.09 0)
-      (effects (font (size 1.27 1.27)) (justify left) hide)
-    )
-    (property "Footprint" "KD_Resistor:RESC2012X50N" (at 196.85 102.87 0)
-      (effects (font (size 1.27 1.27)) (justify left) hide)
-    )
-    (property "Datasheet" "https://www.seielect.com/catalog/sei-rmcf_rmcp.pdf" (at 196.85 105.41 0)
+    (property "Value" "4k7" (at 196.85 85.09 0)
+      (effects (font (size 1.27 1.27)) (justify left) hide)
+    )
+    (property "Footprint" "KD_Resistor:RESC1005X40N" (at 196.85 102.87 0)
+      (effects (font (size 1.27 1.27)) (justify left) hide)
+    )
+    (property "Datasheet" "https://www.te.com/commerce/DocumentDelivery/DDEController?Action=srchrtrv&DocNm=1773204-3&DocType=DS&DocLang=English" (at 196.85 105.41 0)
       (effects (font (size 1.27 1.27)) (justify left) hide)
     )
@@
       (effects (font (size 1.27 1.27)) (justify left))
     )
-    (property "Manufacturer" "Stackpole Electronics Inc" (at 196.85 87.63 0)
-      (effects (font (size 1.27 1.27)) (justify left) hide)
-    )
-    (property "MFG_PartNo" "RMCF0805JT4K70" (at 196.85 90.17 0)
+    (property "Manufacturer" "Bourns Inc." (at 196.85 87.63 0)
+      (effects (font (size 1.27 1.27)) (justify left) hide)
+    )
+    (property "MFG_PartNo" "CR0402-FX-4701GLF" (at 196.85 90.17 0)
       (effects (font (size 1.27 1.27)) (justify left) hide)
     )
@@
       (effects (font (size 1.27 1.27)) (justify left) hide)
     )
-    (property "Supplier_PartNo" "RMCF0805JT4K70CT-ND" (at 196.85 95.25 0)
+    (property "Supplier_PartNo" "CR0402-FX-4701GLFCT-ND" (at 196.85 95.25 0)
       (effects (font (size 1.27 1.27)) (justify left) hide)
     )
@@
     )
   )
-  (symbol (lib_id "KD_Resistor:R_0805_4700_5%") (at 218.44 116.84 0) (unit 1)
+  (symbol (lib_id "KD_Resistor:R_0402_4700_1%") (at 218.44 116.84 0) (unit 1)
     (in_bom yes) (on_board yes) (dnp no) (fields_autoplaced)
     (property "Reference" "R38" (at 220.98 115.57 0)
       (effects (font (size 1.27 1.27)) (justify left))
     )
-    (property "Value" "R_0805_4700_5%" (at 205.74 85.09 0)
-      (effects (font (size 1.27 1.27)) (justify left) hide)
-    )
-    (property "Footprint" "KD_Resistor:RESC2012X50N" (at 205.74 102.87 0)
-      (effects (font (size 1.27 1.27)) (justify left) hide)
-    )
-    (property "Datasheet" "https://www.seielect.com/catalog/sei-rmcf_rmcp.pdf" (at 205.74 105.41 0)
+    (property "Value" "4k7" (at 205.74 85.09 0)
+      (effects (font (size 1.27 1.27)) (justify left) hide)
+    )
+    (property "Footprint" "KD_Resistor:RESC1005X40N" (at 205.74 102.87 0)
+      (effects (font (size 1.27 1.27)) (justify left) hide)
+    )
+    (property "Datasheet" "https://www.te.com/commerce/DocumentDelivery/DDEController?Action=srchrtrv&DocNm=1773204-3&DocType=DS&DocLang=English" (at 205.74 105.41 0)
       (effects (font (size 1.27 1.27)) (justify left) hide)
     )
@@
       (effects (font (size 1.27 1.27)) (justify left))
     )
-    (property "Manufacturer" "Stackpole Electronics Inc" (at 205.74 87.63 0)
-      (effects (font (size 1.27 1.27)) (justify left) hide)
-    )
-    (property "MFG_PartNo" "RMCF0805JT4K70" (at 205.74 90.17 0)
+    (property "Manufacturer" "Bourns Inc." (at 205.74 87.63 0)
+      (effects (font (size 1.27 1.27)) (justify left) hide)
+    )
+    (property "MFG_PartNo" "CR0402-FX-4701GLF" (at 205.74 90.17 0)
       (effects (font (size 1.27 1.27)) (justify left) hide)
     )
@@
       (effects (font (size 1.27 1.27)) (justify left) hide)
     )
-    (property "Supplier_PartNo" "RMCF0805JT4K70CT-ND" (at 205.74 95.25 0)
-      (effects (font (size 1.27 1.27)) (justify left) hide)
-    )
+    (property "Supplier_PartNo" "CR0402-FX-4701GLFCT-ND" (at 205.74 95.25 0)
+      (effects (font (size 1.27 1.27)) (justify left) hide)
+    )

Commit message: Leiskaa
Parts:
- added C3: 10n, KD_Capacitor:CAPC1608X90N, symbol KD_Capacitor:C_0603_10n_X7R_100V
- added R29: 10k, KD_Resistor:RESC1608X55N, symbol KD_Resistor:R_0603_10k_1%
- FB2: value Ferrite_300mA_Abracon_ACML-0805-102-T -> Ferrite_500mA_TDK_MMZ2012Y152BT000; symbol KD_Inductor:Ferrite_300mA_Abracon_ACML-0805-102-T -> KD_Inductor:Ferrite_500mA_TDK_MMZ2012Y152BT000; Code ACML-0805-102-T -> MMZ2012Y152BT000; MFG_PartNo ACML-0805-102-T -> MMZ2012Y152BT000; Supplier_PartNo 535-ACML-0805-102-TCT-ND -> 445-MMZ2012Y152BT000CT-ND
- R24: value R_0603_22k_1% -> R_0603_DNP
- R37, R38: value 4k7 -> R_0603_5100_1%; footprint KD_Resistor:RESC1005X40N -> KD_Resistor:RESC1608X55N; symbol KD_Resistor:R_0402_4700_1% -> KD_Resistor:R_0603_5100_1%; Code 4k7 -> 5k1; MFG_PartNo CR0402-FX-4701GLF -> RMCF0603JT5K10; Manufacturer Bourns Inc. -> Stackpole Electronics Inc; Supplier_PartNo CR0402-FX-4701GLFCT-ND -> RMCF0603JT5K10CT-ND
Connections:
- net GND: now also C3.1
- net I2C1_SCL: now also R38.2, TP12.1
- net I2C1_SDA: now also R37.2, TP11.1
- net SCL: no longer R38.2, TP11.1
- net SDA: no longer R37.2, TP12.1
- net ~{RESET}: now also C3.2, R29.2
- net 3V3_MCU: now reaches C2.1, C2.1, C2.1, C2.1, C2.1, C2.1, C4.1, C4.1, FB2.2, U5.1 (IOVDD), U5.10 (IOVDD), U5.22 (IOVDD), U5.33 (IOVDD), U5.42 (IOVDD), U5.43 (ADC_AVDD), U5.44 (VREG_IN), U5.48 (USB_VDD), U5.49 (IOVDD)
- new net PERIP_~{RESET}: R29.1
Other:
- moved on the sheet: C2, C4, FB2, R37, R38, TP11, TP12, TP6, TP8

Commit message: error fixing
Parts:
- S12, S13: value Button_tactile_45x38_430181038816 -> 430181038816; Code 430181038816 -> (none)
Changed lines of the file:
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@@
   (title_block
     (title "Programmable Keyboard")
-    (date "2023-10-14")
+    (date "2023-10-19")
     (rev "1.0")
     (company "Kallio Designs Oy")
@@
   )
   (bus_alias "I2C0" (members "SDA" "SCL"))
-  (bus_alias "QSPI" (members "DATA0" "DATA1" "DATA2" "DATA3" "~{CS}_MEMORY" "CLK"))
   (bus_alias "I2C1" (members "I2C1_SDA" "I2C1_SCL"))
   (bus_alias "SPI" (members "SPI_CLK" "SPI_MISO" "SPI_MOSI" "SPI_CS0"))
+  (bus_alias "QSPI" (members "DATA0" "DATA1" "DATA2" "DATA3" "~{CS}_MEMORY" "CLK"))
   (junction (at 142.24 57.15) (diameter 0) (color 0 0 0 0)
   )
@@
       (effects (font (size 1.27 1.27)))
     )
-    (property "Value" "Button_tactile_45x38_430181038816" (at 29.21 148.59 0)
-      (effects (font (size 1.27 1.27)) (justify left) hide)
+    (property "Value" "430181038816" (at 41.91 175.26 0)
+      (effects (font (size 1.27 1.27)))
     )
     (property "Footprint" "KD_Switch:SW_Push_1P1T_NO_Wurth_430181038816" (at 29.21 166.37 0)
@@
     (property "Datasheet" "https://www.mouser.fi/datasheet/2/445/430181038816-1717160.pdf" (at 29.21 168.91 0)
       (effects (font (size 1.27 1.27)) (justify left) hide)
-    )
-    (property "Code" "430181038816" (at 41.91 175.26 0)
-      (effects (font (size 1.27 1.27)))
     )
     (property "Manufacturer" "Wurth Elektronik" (at 29.21 151.13 0)
@@
       (effects (font (size 1.27 1.27)))
     )
-    (property "Value" "Button_tactile_45x38_430181038816" (at 31.75 115.57 0)
-      (effects (font (size 1.27 1.27)) (justify left) hide)
+    (property "Value" "430181038816" (at 44.45 142.24 0)
+      (effects (font (size 1.27 1.27)))
     )
     (property "Footprint" "KD_Switch:SW_Push_1P1T_NO_Wurth_430181038816" (at 31.75 133.35 0)
@@
       (effects (font (size 1.27 1.27)) (justify left) hide)
     )
-    (property "Code" "430181038816" (at 44.45 142.24 0)
-      (effects (font (size 1.27 1.27)))
-    )
     (property "Manufacturer" "Wurth Elektronik" (at 31.75 118.11 0)
