File: PCB/Rev 02.00/000018 PGKB/USBcon.kicad_sch (KiCad schematic)
At the start: 8 parts, among them J1 USB_B_V_Adam_USB-B-S-VT

Commit message: schematic
Parts:
- removed J1: USB_B_V_Adam_USB-B-S-VT, KD_Connector_USB_HDMI_Etc:USB_B_Vertical_Adam_USB-B-S-VT, symbol KD_Connector_USB_HDMI_Etc:USB_B_V_Adam_USB-B-S-VT
- added D6: Schottky_30V_1A_PMEG3010ER_115, KD_Diode:DIOC360X180X150_SOD123, symbol KD_Diode:Schottky_30V_1A_PMEG3010ER_115
- added J1: USB Mini B, KD_Connector_USB_HDMI_Etc:USB_C_Receptacle_GCT_USB4085, symbol KD_Connector_USB_HDMI_Etc:USB_C_V_GCT_USB4085-GF-A
- added R14, R15: R_0603_5100_1%, KD_Resistor:RESC1608X55N, symbol KD_Resistor:R_0603_5100_1%
Connections:
- net GND: now also J1.A1 (GND), J1.A12 (GND), J1.B1 (GND), J1.B12 (GND), J1.S1 (SHIELD), R14.2, R15.2
- net USB_D_N: now also J1.A6 (D+), J1.B6 (D+)
- net USB_D_P: now also J1.A7 (D-), J1.B7 (D-)
- net at D3.5 (V+): now also D6.2 (A), J1.A4 (VBUS), J1.A9 (VBUS), J1.B4 (VBUS), J1.B9 (VBUS); no longer FB2.1
- new net: D6.1 (K), FB2.1
- new net CC1: J1.A5 (CC1), R15.1
- new net CC2: J1.B5 (CC2), R14.1
- no-connect marks 2 -> 12
Other:
- moved on the sheet: C4, C5, C6, D3, FB2, R3, R4

Commit message: Schematic
Other:
- company: 4D Haptics Oy -> Kallio Designs Oy
- title: Suspension Rig -> Programmable Keyboard
Changed lines of the file:
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@@
   (paper "A4")
   (title_block
-    (title "Suspension Rig")
-    (date "2023-09-25")
+    (title "Programmable Keyboard")
+    (date "2023-10-14")
     (rev "1.0")
-    (company "4D Haptics Oy")
-    (comment 1 "TL, SB")
+    (company "Kallio Designs Oy")
+    (comment 1 "TL, NH")
     (comment 3 "PCB_PN")
   )

Commit message: updates
Parts:
- renumbered C4 to C1, C5 to C2, C6 to C3, D3 to D1, D6 to D2, FB2 to FB1, R14 to R1, R15 to R2
Connections:
- no-connect marks 12 -> 4
Changed lines of the file:
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@@
   (junction (at 135.89 92.71) (diameter 0) (color 0 0 0 0)
   )
-  (no_connect (at 99.06 118.11))
-  (no_connect (at 99.06 102.87))
   (no_connect (at 99.06 130.81))
-  (no_connect (at 99.06 110.49))
-  (no_connect (at 99.06 125.73))
   (no_connect (at 152.4 118.11))
   (no_connect (at 99.06 133.35))
-  (no_connect (at 99.06 115.57))
-  (no_connect (at 99.06 100.33))
-  (no_connect (at 99.06 123.19))
   (no_connect (at 137.16 118.11))
-  (no_connect (at 99.06 107.95))
   (wire (pts (xy 121.92 50.8) (xy 121.92 54.61))
     (stroke (width 0) (type default))
@@
   (symbol (lib_id "KD_Resistor:R_0603_5100_1%") (at 113.03 58.42 0) (unit 1)
     (in_bom yes) (on_board yes) (dnp no) (fields_autoplaced)
-    (property "Reference" "R14" (at 115.57 57.15 0)
+    (property "Reference" "R1" (at 115.57 57.15 0)
       (effects (font (size 1.27 1.27)) (justify left))
     )
@@
       (project "000018 PGKB"
         (path "/e63e39d7-6ac0-4ffd-8aa3-1841a4541b55/2eb44e1a-4042-4ea6-aca2-4836a6ec84e9/7f81d4f7-3bdd-46dd-b342-c371ad5913dc"
-          (reference "R14") (unit 1)
+          (reference "R1") (unit 1)
         )
       )
@@
   (symbol (lib_id "KD_Capacitor:C_1206_10u_X5R_50V_automotive") (at 184.15 55.88 0) (unit 1)
     (in_bom yes) (on_board yes) (dnp no) (fields_autoplaced)
-    (property "Reference" "C4" (at 187.96 54.61 0)
+    (property "Reference" "C1" (at 187.96 54.61 0)
       (effects (font (size 1.27 1.27)) (justify left))
     )
@@
       (project "000018 PGKB"
         (path "/e63e39d7-6ac0-4ffd-8aa3-1841a4541b55/2eb44e1a-4042-4ea6-aca2-4836a6ec84e9/7f81d4f7-3bdd-46dd-b342-c371ad5913dc"
-          (reference "C4") (unit 1)
+          (reference "C1") (unit 1)
         )
       )
@@
   (symbol (lib_id "KD_Capacitor:C_AE_4.7uF_16V_EEE-1CA4R7NR") (at 210.82 55.88 0) (unit 1)
     (in_bom yes) (on_board yes) (dnp no) (fields_autoplaced)
-    (property "Reference" "C6" (at 214.63 53.721 0)
+    (property "Reference" "C3" (at 214.63 53.721 0)
       (effects (font (size 1.27 1.27)) (justify left))
     )
@@
       (project "000018 PGKB"
         (path "/e63e39d7-6ac0-4ffd-8aa3-1841a4541b55/2eb44e1a-4042-4ea6-aca2-4836a6ec84e9/7f81d4f7-3bdd-46dd-b342-c371ad5913dc"
-          (reference "C6") (unit 1)
+          (reference "C3") (unit 1)
         )
       )
@@
   (symbol (lib_id "power:GND") (at 113.03 64.77 0) (unit 1)
     (in_bom yes) (on_board yes) (dnp no)
-    (property "Reference" "#PWR06" (at 113.03 71.12 0)
+    (property "Reference" "#PWR03" (at 113.03 71.12 0)
       (effects (font (size 1.27 1.27)) hide)
     )
@@
       (project "000018 PGKB"
         (path "/e63e39d7-6ac0-4ffd-8aa3-1841a4541b55/2eb44e1a-4042-4ea6-aca2-4836a6ec84e9/7f81d4f7-3bdd-46dd-b342-c371ad5913dc"
-          (reference "#PWR06") (unit 1)
+          (reference "#PWR03") (unit 1)
         )
       )
@@
   (symbol (lib_id "KD_Diode:TVS_5V5_DRTR5V0U4S-7-M") (at 144.78 110.49 0) (unit 1)
     (in_bom yes) (on_board yes) (dnp no) (fields_autoplaced)
-    (property "Reference" "D3" (at 144.78 96.52 0)
+    (property "Reference" "D1" (at 144.78 96.52 0)
       (effects (font (size 1.27 1.27)))
     )
@@
       (project "000018 PGKB"
         (path "/e63e39d7-6ac0-4ffd-8aa3-1841a4541b55/2eb44e1a-4042-4ea6-aca2-4836a6ec84e9/7f81d4f7-3bdd-46dd-b342-c371ad5913dc"
-          (reference "D3") (unit 1)
+          (reference "D1") (unit 1)
         )
       )
@@
   (symbol (lib_id "power:GND") (at 83.82 143.51 0) (unit 1)
     (in_bom yes) (on_board yes) (dnp no)
-    (property "Reference" "#PWR07" (at 83.82 149.86 0)
+    (property "Reference" "#PWR02" (at 83.82 149.86 0)
       (effects (font (size 1.27 1.27)) hide)
     )
@@
       (project "000018 PGKB"
         (path "/e63e39d7-6ac0-4ffd-8aa3-1841a4541b55/2eb44e1a-4042-4ea6-aca2-4836a6ec84e9/7f81d4f7-3bdd-46dd-b342-c371ad5913dc"
-          (reference "#PWR07") (unit 1)
+          (reference "#PWR02") (unit 1)
         )
       )
@@
   (symbol (lib_id "power:GND") (at 76.2 143.51 0) (unit 1)
     (in_bom yes) (on_board yes) (dnp no)
-    (property "Reference" "#PWR012" (at 76.2 149.86 0)
+    (property "Reference" "#PWR01" (at 76.2 149.86 0)
       (effects (font (size 1.27 1.27)) hide)
     )
@@
       (project "000018 PGKB"
         (path "/e63e39d7-6ac0-4ffd-8aa3-1841a4541b55/2eb44e1a-4042-4ea6-aca2-4836a6ec84e9/7f81d4f7-3bdd-46dd-b342-c371ad5913dc"
-          (reference "#PWR012") (unit 1)
+          (reference "#PWR01") (unit 1)
         )
       )
@@
   (symbol (lib_id "power:GND") (at 154.94 111.76 0) (unit 1)
     (in_bom yes) (on_board yes) (dnp no)
-    (property "Reference" "#PWR09" (at 154.94 118.11 0)
+    (property "Reference" "#PWR04" (at 154.94 118.11 0)
       (effects (font (size 1.27 1.27)) hide)
     )
@@
       (project "000018 PGKB"
         (path "/e63e39d7-6ac0-4ffd-8aa3-1841a4541b55/2eb44e1a-4042-4ea6-aca2-4836a6ec84e9/7f81d4f7-3bdd-46dd-b342-c371ad5913dc"
-          (reference "#PWR09") (unit 1)
+          (reference "#PWR04") (unit 1)
         )
       )
@@
   (symbol (lib_id "KD_Inductor:Ferrite_500mA_TDK_MMZ2012Y152BT000") (at 176.53 50.8 90) (unit 1)
     (in_bom yes) (on_board yes) (dnp no) (fields_autoplaced)
-    (property "Reference" "FB2" (at 176.53 44.45 90)
+    (property "Reference" "FB1" (at 176.53 44.45 90)
       (effects (font (size 1.27 1.27)))
     )
@@
       (project "000018 PGKB"
         (path "/e63e39d7-6ac0-4ffd-8aa3-1841a4541b55/2eb44e1a-4042-4ea6-aca2-4836a6ec84e9/7f81d4f7-3bdd-46dd-b342-c371ad5913dc"
-          (reference "FB2") (unit 1)
+          (reference "FB1") (unit 1)
         )
       )
@@
   (symbol (lib_id "KD_Diode:Schottky_30V_1A_PMEG3010ER_115") (at 153.67 50.8 180) (unit 1)
     (in_bom yes) (on_board yes) (dnp no) (fields_autoplaced)
-    (property "Reference" "D6" (at 153.9875 44.45 0)
+    (property "Reference" "D2" (at 153.9875 44.45 0)
       (effects (font (size 1.27 1.27)))
     )
@@
       (project "000018 PGKB"
         (path "/e63e39d7-6ac0-4ffd-8aa3-1841a4541b55/2eb44e1a-4042-4ea6-aca2-4836a6ec84e9/7f81d4f7-3bdd-46dd-b342-c371ad5913dc"
-          (reference "D6") (unit 1)
+          (reference "D2") (unit 1)
         )
       )
@@
   (symbol (lib_id "KD_Capacitor:C_0603_100n_X7R_50V") (at 196.85 55.88 0) (unit 1)
     (in_bom yes) (on_board yes) (dnp no) (fields_autoplaced)
-    (property "Reference" "C5" (at 200.66 54.61 0)
+    (property "Reference" "C2" (at 200.66 54.61 0)
       (effects (font (size 1.27 1.27)) (justify left))
     )
@@
       (project "000018 PGKB"
         (path "/e63e39d7-6ac0-4ffd-8aa3-1841a4541b55/2eb44e1a-4042-4ea6-aca2-4836a6ec84e9/7f81d4f7-3bdd-46dd-b342-c371ad5913dc"
-          (reference "C5") (unit 1)
+          (reference "C2") (unit 1)
         )
       )
@@
   (symbol (lib_id "power:GND") (at 196.85 60.96 0) (unit 1)
     (in_bom yes) (on_board yes) (dnp no)
-    (property "Reference" "#PWR010" (at 196.85 67.31 0)
+    (property "Reference" "#PWR06" (at 196.85 67.31 0)
       (effects (font (size 1.27 1.27)) hide)
     )
@@
       (project "000018 PGKB"
         (path "/e63e39d7-6ac0-4ffd-8aa3-1841a4541b55/2eb44e1a-4042-4ea6-aca2-4836a6ec84e9/7f81d4f7-3bdd-46dd-b342-c371ad5913dc"
-          (reference "#PWR010") (unit 1)
+          (reference "#PWR06") (unit 1)
         )
       )
@@
   (symbol (lib_id "power:GND") (at 210.82 60.96 0) (unit 1)
     (in_bom yes) (on_board yes) (dnp no)
-    (property "Reference" "#PWR011" (at 210.82 67.31 0)
+    (property "Reference" "#PWR07" (at 210.82 67.31 0)
       (effects (font (size 1.27 1.27)) hide)
     )
@@
       (project "000018 PGKB"
         (path "/e63e39d7-6ac0-4ffd-8aa3-1841a4541b55/2eb44e1a-4042-4ea6-aca2-4836a6ec84e9/7f81d4f7-3bdd-46dd-b342-c371ad5913dc"
-          (reference "#PWR011") (unit 1)
+          (reference "#PWR07") (unit 1)
         )
       )
@@
   (symbol (lib_id "KD_Resistor:R_0603_5100_1%") (at 121.92 58.42 0) (unit 1)
     (in_bom yes) (on_board yes) (dnp no) (fields_autoplaced)
-    (property "Reference" "R15" (at 124.46 57.15 0)
+    (property "Reference" "R2" (at 124.46 57.15 0)
       (effects (font (size 1.27 1.27)) (justify left))
     )
@@
       (project "000018 PGKB"
         (path "/e63e39d7-6ac0-4ffd-8aa3-1841a4541b55/2eb44e1a-4042-4ea6-aca2-4836a6ec84e9/7f81d4f7-3bdd-46dd-b342-c371ad5913dc"
-          (reference "R15") (unit 1)
+          (reference "R2") (unit 1)
         )
       )
@@
   (symbol (lib_id "power:GND") (at 184.15 60.96 0) (unit 1)
     (in_bom yes) (on_board yes) (dnp no)
-    (property "Reference" "#PWR08" (at 184.15 67.31 0)
+    (property "Reference" "#PWR05" (at 184.15 67.31 0)
       (effects (font (size 1.27 1.27)) hide)
     )
@@
       (project "000018 PGKB"
         (path "/e63e39d7-6ac0-4ffd-8aa3-1841a4541b55/2eb44e1a-4042-4ea6-aca2-4836a6ec84e9/7f81d4f7-3bdd-46dd-b342-c371ad5913dc"
-          (reference "#PWR08") (unit 1)
+          (reference "#PWR05") (unit 1)
         )
       )
@@
     )
     (pin "A1")
-    (pin "A10")
-    (pin "A11")
     (pin "A12")
-    (pin "A2")
-    (pin "A3")
     (pin "A4")
     (pin "A5")
@@
     (pin "A9")
     (pin "B1")
-    (pin "B10")
-    (pin "B11")
     (pin "B12")
-    (pin "B2")
-    (pin "B3")
     (pin "B4")
     (pin "B5")
