File: PCB/Rev 02.00/000018 PGKB/USBcon.kicad_sch (KiCad schematic)
At the start: 11 parts, among them J1 USB Mini B

Commit message: Layout
Parts:
- renumbered D1 to D11, D2 to D12
Changed lines of the file:
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@@
   (symbol (lib_id "KD_Diode:TVS_5V5_DRTR5V0U4S-7-M") (at 144.78 110.49 0) (unit 1)
     (in_bom yes) (on_board yes) (dnp no) (fields_autoplaced)
-    (property "Reference" "D1" (at 144.78 96.52 0)
+    (property "Reference" "D11" (at 144.78 96.52 0)
       (effects (font (size 1.27 1.27)))
     )
@@
       (project "000018 PGKB"
         (path "/e63e39d7-6ac0-4ffd-8aa3-1841a4541b55/2eb44e1a-4042-4ea6-aca2-4836a6ec84e9/7f81d4f7-3bdd-46dd-b342-c371ad5913dc"
-          (reference "D1") (unit 1)
+          (reference "D11") (unit 1)
         )
       )
@@
   (symbol (lib_id "KD_Diode:Schottky_30V_1A_PMEG3010ER_115") (at 146.05 50.8 180) (unit 1)
     (in_bom yes) (on_board yes) (dnp no) (fields_autoplaced)
-    (property "Reference" "D2" (at 146.3675 44.45 0)
+    (property "Reference" "D12" (at 146.3675 44.45 0)
       (effects (font (size 1.27 1.27)))
     )
@@
       (project "000018 PGKB"
         (path "/e63e39d7-6ac0-4ffd-8aa3-1841a4541b55/2eb44e1a-4042-4ea6-aca2-4836a6ec84e9/7f81d4f7-3bdd-46dd-b342-c371ad5913dc"
-          (reference "D2") (unit 1)
-        )
-      )
+          (reference "D12") (unit 1)
+        )
+      )

Commit message: sitte vaan routaus
Parts:
- removed C3: 4u7, KD_Capacitor:CAPAE400x540N, symbol KD_Capacitor:C_AE_4.7uF_16V_EEE-1CA4R7NR
Changed lines of the file:
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@@
   (junction (at 214.63 50.8) (diameter 0) (color 0 0 0 0)
-  )
-  (junction (at 228.6 50.8) (diameter 0) (color 0 0 0 0)
   )
   (junction (at 113.03 63.5) (diameter 0) (color 0 0 0 0)
@@
     (stroke (width 0) (type default))
   )
-  (wire (pts (xy 228.6 60.96) (xy 228.6 59.69))
-    (stroke (width 0) (type default))
-  )
   (wire (pts (xy 127 110.49) (xy 127 74.93))
     (stroke (width 0) (type default))
@@
     (stroke (width 0) (type default))
   )
-  (wire (pts (xy 228.6 50.8) (xy 228.6 52.07))
-    (stroke (width 0) (type default))
-  )
   (wire (pts (xy 135.89 92.71) (xy 158.75 92.71))
     (stroke (width 0) (type default))
@@
     (stroke (width 0) (type default))
   )
-  (wire (pts (xy 214.63 50.8) (xy 228.6 50.8))
+  (wire (pts (xy 214.63 50.8) (xy 238.76 50.8))
     (stroke (width 0) (type default))
   )
@@
   )
   (wire (pts (xy 214.63 52.07) (xy 214.63 50.8))
-    (stroke (width 0) (type default))
-  )
-  (wire (pts (xy 228.6 50.8) (xy 238.76 50.8))
     (stroke (width 0) (type default))
   )
@@
         (path "/e63e39d7-6ac0-4ffd-8aa3-1841a4541b55/2eb44e1a-4042-4ea6-aca2-4836a6ec84e9/7f81d4f7-3bdd-46dd-b342-c371ad5913dc"
           (reference "C1") (unit 1)
-        )
-      )
-    )
-  )
-  (symbol (lib_id "KD_Capacitor:C_AE_4.7uF_16V_EEE-1CA4R7NR") (at 228.6 55.88 0) (unit 1)
-    (in_bom yes) (on_board yes) (dnp no) (fields_autoplaced)
-    (property "Reference" "C3" (at 232.41 53.721 0)
-      (effects (font (size 1.27 1.27)) (justify left))
-    )
-    (property "Value" "4u7" (at 232.41 56.261 0)
-      (effects (font (size 1.27 1.27)) (justify left))
-    )
-    (property "Footprint" "KD_Capacitor:CAPAE400x540N" (at 215.9 41.91 0)
-      (effects (font (size 1.27 1.27)) (justify left) hide)
-    )
-    (property "Datasheet" "https://mm.digikey.com/Volume0/opasdata/d220001/medias/docus/2172/S_Series,Type_V_Rev2018.pdf" (at 215.9 44.45 0)
-      (effects (font (size 1.27 1.27)) (justify left) hide)
-    )
-    (property "Manufacturer" "Panasonic Electronic Components" (at 215.9 26.67 0)
-      (effects (font (size 1.27 1.27)) (justify left) hide)
-    )
-    (property "MFG_PartNo" "EEE-1CA4R7NR" (at 215.9 29.21 0)
-      (effects (font (size 1.27 1.27)) (justify left) hide)
-    )
-    (property "Supplier" "Digi-Key" (at 215.9 31.75 0)
-      (effects (font (size 1.27 1.27)) (justify left) hide)
-    )
-    (property "Supplier_PartNo" "PCE4290CT-ND" (at 215.9 34.29 0)
-      (effects (font (size 1.27 1.27)) (justify left) hide)
-    )
-    (property "DNP" "F" (at 215.9 36.83 0)
-      (effects (font (size 1.27 1.27)) (justify left) hide)
-    )
-    (property "Price" "0.3" (at 215.9 39.37 0)
-      (effects (font (size 1.27 1.27)) (justify left) hide)
-    )
-    (pin "1")
-    (pin "2")
-    (instances
-      (project "000018 PGKB"
-        (path "/e63e39d7-6ac0-4ffd-8aa3-1841a4541b55/2eb44e1a-4042-4ea6-aca2-4836a6ec84e9/7f81d4f7-3bdd-46dd-b342-c371ad5913dc"
-          (reference "C3") (unit 1)
         )
       )
@@
         )
       )
-    )
-  )
-  (symbol (lib_id "power:GND") (at 228.6 60.96 0) (unit 1)
-    (in_bom yes) (on_board yes) (dnp no)
-    (property "Reference" "#PWR07" (at 228.6 67.31 0)
-      (effects (font (size 1.27 1.27)) hide)
-    )
-    (property "Value" "GND" (at 228.6 64.77 0)
-      (effects (font (size 1.27 1.27)))
-    )
-    (property "Footprint" "" (at 228.6 60.96 0)
-      (effects (font (size 1.27 1.27)) hide)
-    )
-    (property "Datasheet" "" (at 228.6 60.96 0)
-      (effects (font (size 1.27 1.27)) hide)
-    )
-    (pin "1")
-    (instances
-      (project "000018 PGKB"
-        (path "/e63e39d7-6ac0-4ffd-8aa3-1841a4541b55/2eb44e1a-4042-4ea6-aca2-4836a6ec84e9/7f81d4f7-3bdd-46dd-b342-c371ad5913dc"
-          (reference "#PWR07") (unit 1)
-        )
-      )

Commit message: MODIFICATIONS To Rev 2
Parts:
- J1: value USB Mini B -> USB C; MFG_PartNo USB-B-S-VT -> USB4085-GF-A; Manufacturer Adam Tech -> GCT; Price 1 -> 0.85; Supplier_PartNo 2057-USB-B-S-VT-ND -> 2073-USB4085-GF-ACT-ND
Changed lines of the file:
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@@
   (title_block
     (title "Programmable Keyboard")
-    (date "2023-10-19")
+    (date "2024-01-24")
     (rev "1.0")
     (company "Kallio Designs Oy")
@@
       (effects (font (size 1.27 1.27)) (justify left))
     )
-    (property "Value" "USB Mini B" (at 73.66 71.12 0) (do_not_autoplace)
+    (property "Value" "USB C" (at 73.66 71.12 0) (do_not_autoplace)
       (effects (font (size 1.27 1.27)) (justify left))
     )
@@
       (effects (font (size 1.27 1.27)) (justify left) hide)
     )
-    (property "Datasheet" "https://app.adam-tech.com/products/download/data_sheet/195855/usb-b-s-vt-data-sheet.pdf" (at 91.44 59.69 0)
-      (effects (font (size 1.27 1.27)) (justify left) hide)
-    )
-    (property "Manufacturer" "Adam Tech" (at 91.44 41.91 0)
-      (effects (font (size 1.27 1.27)) (justify left) hide)
-    )
-    (property "MFG_PartNo" "USB-B-S-VT" (at 91.44 44.45 0)
+    (property "Datasheet" "https://gct.co/files/drawings/usb4085.pdf" (at 91.44 59.69 0)
+      (effects (font (size 1.27 1.27)) (justify left) hide)
+    )
+    (property "Manufacturer" "GCT" (at 91.44 41.91 0)
+      (effects (font (size 1.27 1.27)) (justify left) hide)
+    )
+    (property "MFG_PartNo" "USB4085-GF-A" (at 91.44 44.45 0)
       (effects (font (size 1.27 1.27)) (justify left) hide)
     )
@@
       (effects (font (size 1.27 1.27)) (justify left) hide)
     )
-    (property "Supplier_PartNo" "2057-USB-B-S-VT-ND" (at 91.44 49.53 0)
+    (property "Supplier_PartNo" "2073-USB4085-GF-ACT-ND" (at 91.44 49.53 0)
       (effects (font (size 1.27 1.27)) (justify left) hide)
     )
@@
       (effects (font (size 1.27 1.27)) (justify left) hide)
     )
-    (property "Price" "1" (at 91.44 54.61 0)
-      (effects (font (size 1.27 1.27)) (justify left) hide)
-    )
+    (property "Price" "0.85" (at 91.44 54.61 0)
+      (effects (font (size 1.27 1.27)) (justify left) hide)
+    )
