File: PCB/Rev 02.00/000018 PGKB/buttons.kicad_sch (KiCad schematic)
At the start: 18 parts, among them U12 SN74HCS365PWR

Commit message: Schematic
Other:
- company: 4D Haptics Oy -> Kallio Designs Oy
- title: Suspension Rig -> Programmable Keyboard
Changed lines of the file:
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@@
   (paper "A4")
   (title_block
-    (title "Suspension Rig")
-    (date "2023-09-25")
+    (title "Programmable Keyboard")
+    (date "2023-10-14")
     (rev "1.0")
-    (company "4D Haptics Oy")
-    (comment 1 "TL, SB")
+    (company "Kallio Designs Oy")
+    (comment 1 "TL, NH")
     (comment 3 "PCB_PN")
   )

Commit message: buttons
Parts:
- removed S3, S4, S5: Button_tactile_45x38_430181038816, KD_Switch:SW_Push_1P1T_NO_Wurth_430181038816, symbol KD_Switch:Button_tactile_45x38_430181038816
- added S3, S4, S5, S6, S7, S8: 5124, KD_Switch:SWITCH_BUTTON_Kailh_mx, symbol KD_Switch:Button_keyboard_Adafruit_5124
- added TP10: TP D2.5 mm H0.9mm, KD_Connector_Pads:TestPoint_Pad_D2.5mm_H0.9mm, symbol KD_Connector_Pads:TestPoint_2.5mm_H0.9
Connections:
- net +3.3V: now also S3.2, S4.2, S5.2, S6.2, S7.2, S8.2
- net Button5: now also TP10.1
- net at R53.1: now also S6.3
- net at R50.1: now also S3.3
- net at R55.1: now also S8.3
- net at R54.1: now also S7.3
- net at R51.1: now also S4.3
- net at R52.1: now also S5.3
- no-connect marks 6 -> 0

Commit message: ledit
Parts:
- added C25, C26, C27: 10n, KD_Capacitor:CAPC1608X90N, symbol KD_Capacitor:C_0603_10n_X7R_100V
- added C28: 100n, KD_Capacitor:CAPC1608X90N, symbol KD_Capacitor:C_0603_100n_X7R_50V
- added R17, R18, R19: 1k, KD_Resistor:RESC1608X55N, symbol KD_Resistor:R_0603_1k_1%
- added S10, S11, S9: 5124, KD_Switch:SWITCH_BUTTON_Kailh_mx, symbol KD_Switch:Button_keyboard_Adafruit_5124
- added U5: SN74HCS365PWR, KD_Package_SO:SOP65P600X150-16N, symbol KD_IC_Buffer_Driver_Interface:Schmitt_6CH_SN74HCS365PWR
Connections:
- net +3.3V: now also C28.1, S10.2, S11.2, S9.2, U5.16 (VCC)
- net GND: now also C25.2, C26.2, C27.2, C28.2, U5.1 (E1), U5.15 (E2), U5.8 (GND)
- net at C52.1, R50.2, U12.2 (I1): no longer TP12.1
- new net: R17.1, S9.3
- new net: C25.1, R17.2, U5.2 (I1)
- new net: C26.1, R18.2, U5.4 (I2)
- new net: C27.1, R19.2, U5.6 (I3)
- new net: R18.1, S10.3
- new net: R19.1, S11.3
- new net Button6: U5.3 (O1)
- new net Button7: U5.5 (O2)
- new net Button8: U5.7 (O3)
Other:
- moved on the sheet: C19, C52, C53, C54, C55, C56, C57, R50, R51, R52, R53, R54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

Commit message: updates
Parts:
- added C13: 10n, KD_Capacitor:CAPC1608X90N, symbol KD_Capacitor:C_0603_10n_X7R_100V
- added R14: 1k, KD_Resistor:RESC1608X55N, symbol KD_Resistor:R_0603_1k_1%
- added S10: 5124, KD_Switch:SWITCH_BUTTON_Kailh_mx, symbol KD_Switch:Button_keyboard_Adafruit_5124
- renumbered C25 to C10, C26 to C11, C27 to C12, C19 to C14, C28 to C15, C52 to C4, C53 to C5, C54 to C6, C55 to C7, C56 to C8, C57 to C9, R55 to R10, R17 to R11, R18 to R12, R19 to R13, R50 to R5, R51 to R6, R52 to R7, R53 to R8, R54 to R9, S3 to S1, S4 to S2, S5 to S3, S6 to S4, S7 to S5, S8 to S6, S9 to S7, S10 to S8, S11 to S9, TP12 to TP1, TP10 to TP2, U12 to U1, U5 to U2
Connections:
- net +3.3V: now also S1.1, S2.1, S3.1, S4.1, S5.1, S6.1, S7.1, S8.1, S9.1, S10.1; no longer S1.2, S2.2, S3.2, S4.2, S5.2, S6.2, S7.2, S8.2, S9.2
- net GND: now also U2.12 (I5), U2.14 (I6), C13.2
- net at R11.1: now also S7.2; no longer S7.3
- net at R8.1: now also S4.2; no longer S4.3
- net at R5.1: now also S1.2; no longer S1.3
- net at C4.1, R5.2, U1.2 (I1): now also TP1.1
- net at R7.1: now also S3.2; no longer S3.3
- net at R10.1: now also S6.2; no longer S6.3
- net at R9.1: now also S5.2; no longer S5.3
- net at R6.1: now also S2.2; no longer S2.3
- net at R12.1: now also S8.2; no longer S8.3
- net at R13.1: now also S9.2; no longer S9.3
- net at U2.10 (I4): now also C13.1, R14.2
- net Button9: now reaches U2.9 (O4)
- new net: R14.1, S10.2
- no-connect marks 0 -> 2
Other:
- moved on the sheet: C10, C11, C12, R11, R12, R13, S7, S8, S9, TP1
