File: PCB/Rev 02.00/000018 PGKB/buttons.kicad_sch (KiCad schematic)
At the start: 36 parts, among them U1 SN74HCS365PWR, U2 SN74HCS365PWR

Commit message: Layout
Parts:
- added C41: 10n, KD_Capacitor:CAPC1608X90N, symbol KD_Capacitor:C_0603_10n_X7R_100V
- added R28: 1k, KD_Resistor:RESC1608X55N, symbol KD_Resistor:R_0603_1k_1%
- added S11: 4954, KD_Switch:SWITCH_BUTTON_Kailh_mx_socket, symbol KD_Switch:Button_keyboard_socket_Adafruit_4958
- S1, S10, S2, S3, S4, S5, S6, S7, S8, S9: value 5124 -> 4954; footprint KD_Switch:SWITCH_BUTTON_Kailh_mx -> KD_Switch:SWITCH_BUTTON_Kailh_mx_socket; symbol KD_Switch:Button_keyboard_Adafruit_5124 -> KD_Switch:Button_keyboard_socket_Adafruit_4958; MFG_PartNo 5124 -> 4954; Supplier_PartNo 1528-5124-ND -> 1528-4954-ND
Connections:
- net Button0 is gone; now on net Button6: U1.13 (O6)
- net +3.3V: now also S11.1
- net Button1: now also TP2.1, U1.3 (O1); no longer U1.11 (O5)
- net Button2: now also U1.5 (O2); no longer U1.9 (O4)
- net Button4: now also U1.9 (O4); no longer U1.5 (O2)
- net Button5: now also U1.11 (O5); no longer TP2.1, U1.3 (O1)
- net Button6: no longer U2.3 (O1)
- net Button7: now also U2.3 (O1); no longer U2.5 (O2)
- net Button8: now also U2.5 (O2); no longer U2.7 (O3)
- net Button9: now also U2.7 (O3); no longer U2.9 (O4)
- net GND: now also C41.2; no longer U2.12 (I5)
- net Button11: now reaches U2.11 (O5)
- new net: R28.1, S11.2
- new net: C41.1, R28.2, U2.12 (I5)
- new net Button10: U2.9 (O4)
- no-connect marks 2 -> 1
Other:
- moved on the sheet: C10, C11, C12, C13, C14, C15, R11, R12, R13, R14, TP2, U1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

Commit message: sitte vaan routaus
Connections:
- net Button1: now also U2.3 (O1); no longer U1.3 (O1)
- net Button10: now also U1.5 (O2); no longer U2.9 (O4)
- net Button11: now also U1.7 (O3); no longer U2.11 (O5)
- net Button2: now also U2.5 (O2); no longer U1.5 (O2)
- net Button3: now also U2.7 (O3); no longer U1.7 (O3)
- net Button4: now also U2.9 (O4); no longer U1.9 (O4)
- net Button5: now also U1.9 (O4); no longer U1.11 (O5)
- net Button6: now also U1.11 (O5); no longer U1.13 (O6)
- net Button7: now also U2.11 (O5); no longer U2.3 (O1)
- net Button8: now also U2.13 (O6); no longer U2.5 (O2)
- net Button9: now also U1.3 (O1); no longer U2.7 (O3)
- net GND: now also U1.14 (I6); no longer U2.14 (I6)
- net at C7.1, R8.2: now also U2.10 (I4); no longer U1.10 (I4)
- net at C41.1, R28.2: now also U1.6 (I3); no longer U2.12 (I5)
- net at C13.1, R14.2: now also U1.4 (I2); no longer U2.10 (I4)
- net at C6.1, R7.2: now also U2.6 (I3); no longer U1.6 (I3)
- net at C8.1, R9.2: now also U1.10 (I4); no longer U1.12 (I5)
- net at C4.1, R5.2, TP1.1: now also U2.2 (I1); no longer U1.2 (I1)
- net at C9.1, R10.2: now also U1.12 (I5); no longer U1.14 (I6)
- net at C5.1, R6.2: now also U2.4 (I2); no longer U1.4 (I2)
- net at C10.1, R11.2: now also U2.12 (I5); no longer U2.2 (I1)
- net at C11.1, R12.2: now also U2.14 (I6); no longer U2.4 (I2)
- net at C12.1, R13.2: now also U1.2 (I1); no longer U2.6 (I3)
Other:
- moved on the sheet: C10, C11, C12, C13, C14, C15, C41, R11, R12, R13, R14, R28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

Commit message: Leiskaa
Connections:
- net +3.3V renamed +3V3
Changed lines of the file:
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@@
     )
   )
-  (symbol (lib_id "power:+3.3V") (at 31.75 22.86 0) (unit 1)
+  (symbol (lib_id "power:+3V3") (at 31.75 22.86 0) (unit 1)
     (in_bom yes) (on_board yes) (dnp no)
     (property "Reference" "#PWR060" (at 31.75 26.67 0)
       (effects (font (size 1.27 1.27)) hide)
     )
-    (property "Value" "+3.3V" (at 31.75 19.304 0)
+    (property "Value" "+3V3" (at 31.75 19.304 0)
       (effects (font (size 1.27 1.27)))
     )
@@
     )
   )
-  (symbol (lib_id "power:+3.3V") (at 127 57.15 0) (unit 1)
+  (symbol (lib_id "power:+3V3") (at 127 57.15 0) (unit 1)
     (in_bom yes) (on_board yes) (dnp no)
     (property "Reference" "#PWR060" (at 127 60.96 0)
       (effects (font (size 1.27 1.27)) hide)
     )
-    (property "Value" "+3.3V" (at 127 53.594 0)
+    (property "Value" "+3V3" (at 127 53.594 0)
       (effects (font (size 1.27 1.27)))
     )
@@
     )
   )
-  (symbol (lib_id "power:+3.3V") (at 201.93 21.59 0) (unit 1)
+  (symbol (lib_id "power:+3V3") (at 201.93 21.59 0) (unit 1)
     (in_bom yes) (on_board yes) (dnp no) (fields_autoplaced)
     (property "Reference" "#PWR060" (at 201.93 25.4 0)
       (effects (font (size 1.27 1.27)) hide)
     )
-    (property "Value" "+3.3V" (at 201.93 18.034 0)
+    (property "Value" "+3V3" (at 201.93 18.034 0)
       (effects (font (size 1.27 1.27)))
     )
@@
     )
   )
-  (symbol (lib_id "power:+3.3V") (at 201.93 118.11 0) (unit 1)
+  (symbol (lib_id "power:+3V3") (at 201.93 118.11 0) (unit 1)
     (in_bom yes) (on_board yes) (dnp no) (fields_autoplaced)
     (property "Reference" "#PWR060" (at 201.93 121.92 0)
       (effects (font (size 1.27 1.27)) hide)
     )
-    (property "Value" "+3.3V" (at 201.93 114.554 0)
-      (effects (font (size 1.27 1.27)))
-    )
+    (property "Value" "+3V3" (at 201.93 114.554 0)
+      (effects (font (size 1.27 1.27)))
+    )

Commit message: päivityksiä
Parts:
- added R30, R31, R34, R35, R36, R37, R38, R39, R40, R41, R42: 100k, KD_Resistor:RESC1608X55N, symbol KD_Resistor:R_0603_100k_1%
Connections:
- net GND: now also R30.2, R31.2, R34.2, R35.2, R36.2, R37.2, R38.2, R39.2, R40.2, R41.2, R42.2
- net at C7.1, R8.2, U2.10 (I4): now also R35.1
- net at C41.1, R28.2, U1.6 (I3): now also R42.1
- net at C13.1, R14.2, U1.4 (I2): now also R41.1
- net at C6.1, R7.2, U2.6 (I3): now also R34.1
- net at C8.1, R9.2, U1.10 (I4): now also R36.1
- net at C4.1, R5.2, TP1.1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: now also R30.1
- net at C9.1, R10.2, U1.12 (I5): now also R37.1
- net at C12.1, R13.2, U1.2 (I1): now also R40.1
- net at C5.1, R6.2, U2.4 (I2): now also R31.1
- net at C10.1, R11.2, U2.12 (I5): now also R38.1
- net at C11.1, R12.2, U2.14 (I6): now also R39.1
Other:
- moved on the sheet: C10, C11, C12, C13, C41, R11, R12, R13, R14, R28

Commit message: mfg files
Parts:
- added S99: 4954, KD_Switch:SWITCH_BUTTON_Kailh_mx_socket, symbol KD_Switch:Button_keyboard_no_footprint_Adafruit_4958
Changed lines of the file:
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@@
+    )
+  )
+  (symbol (lib_id "KD_Switch:Button_keyboard_no_footprint_Adafruit_4958") (at 121.92 29.21 0) (unit 1)
+    (in_bom yes) (on_board yes) (dnp no) (fields_autoplaced)
+    (property "Reference" "S99" (at 127 27.559 0)
+      (effects (font (size 1.27 1.27)) (justify left))
+    )
+    (property "Value" "4954" (at 127 30.099 0)
+      (effects (font (size 1.27 1.27)) (justify left))
+    )
+    (property "Footprint" "KD_Switch:SWITCH_BUTTON_Kailh_mx_socket" (at 109.22 15.24 0)
+      (effects (font (size 1.27 1.27)) (justify left) hide)
+    )
+    (property "Datasheet" "https://cdn-shop.adafruit.com/product-files/4954/4954_CPG1511F01S03-BOX_Brown.pdf" (at 109.22 17.78 0)
+      (effects (font (size 1.27 1.27)) (justify left) hide)
+    )
+    (property "Manufacturer" "Adafruit" (at 109.22 0 0)
+      (effects (font (size 1.27 1.27)) (justify left) hide)
+    )
+    (property "MFG_PartNo" "4954" (at 109.22 2.54 0)
+      (effects (font (size 1.27 1.27)) (justify left) hide)
+    )
+    (property "Supplier" "Digi-Key" (at 109.22 5.08 0)
+      (effects (font (size 1.27 1.27)) (justify left) hide)
+    )
+    (property "Supplier_PartNo" "1528-4954-ND" (at 109.22 7.62 0)
+      (effects (font (size 1.27 1.27)) (justify left) hide)
+    )
+    (property "DNP" "F" (at 109.22 10.16 0)
+      (effects (font (size 1.27 1.27)) (justify left) hide)
+    )
+    (property "Price" "0.5" (at 109.22 12.7 0)
+      (effects (font (size 1.27 1.27)) (justify left) hide)
+    )
+    (instances
+      (project "000018 PGKB"
+        (path "/e63e39d7-6ac0-4ffd-8aa3-1841a4541b55/2eb44e1a-4042-4ea6-aca2-4836a6ec84e9/86c42f5f-8308-4480-a779-2edf7f31bcc2"
+          (reference "S99") (unit 1)
+        )
+      )
     )
   )

Commit message: MODIFICATIONS Updates
Parts:
- removed S99: 4954, KD_Switch:SWITCH_BUTTON_Kailh_mx_socket, symbol KD_Switch:Button_keyboard_no_footprint_Adafruit_4958
Changed lines of the file:
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@@
-    )
-  )
-  (symbol (lib_id "KD_Switch:Button_keyboard_no_footprint_Adafruit_4958") (at 121.92 29.21 0) (unit 1)
-    (in_bom yes) (on_board yes) (dnp no) (fields_autoplaced)
-    (property "Reference" "S99" (at 127 27.559 0)
-      (effects (font (size 1.27 1.27)) (justify left))
-    )
-    (property "Value" "4954" (at 127 30.099 0)
-      (effects (font (size 1.27 1.27)) (justify left))
-    )
-    (property "Footprint" "KD_Switch:SWITCH_BUTTON_Kailh_mx_socket" (at 109.22 15.24 0)
-      (effects (font (size 1.27 1.27)) (justify left) hide)
-    )
-    (property "Datasheet" "https://cdn-shop.adafruit.com/product-files/4954/4954_CPG1511F01S03-BOX_Brown.pdf" (at 109.22 17.78 0)
-      (effects (font (size 1.27 1.27)) (justify left) hide)
-    )
-    (property "Manufacturer" "Adafruit" (at 109.22 0 0)
-      (effects (font (size 1.27 1.27)) (justify left) hide)
-    )
-    (property "MFG_PartNo" "4954" (at 109.22 2.54 0)
-      (effects (font (size 1.27 1.27)) (justify left) hide)
-    )
-    (property "Supplier" "Digi-Key" (at 109.22 5.08 0)
-      (effects (font (size 1.27 1.27)) (justify left) hide)
-    )
-    (property "Supplier_PartNo" "1528-4954-ND" (at 109.22 7.62 0)
-      (effects (font (size 1.27 1.27)) (justify left) hide)
-    )
-    (property "DNP" "F" (at 109.22 10.16 0)
-      (effects (font (size 1.27 1.27)) (justify left) hide)
-    )
-    (property "Price" "0.5" (at 109.22 12.7 0)
-      (effects (font (size 1.27 1.27)) (justify left) hide)
-    )
-    (instances
-      (project "000018 PGKB"
-        (path "/e63e39d7-6ac0-4ffd-8aa3-1841a4541b55/2eb44e1a-4042-4ea6-aca2-4836a6ec84e9/86c42f5f-8308-4480-a779-2edf7f31bcc2"
-          (reference "S99") (unit 1)
-        )
-      )
     )
   )
