File: PCB/Rev 02.00/000018 PGKB/psu.kicad_sch (KiCad schematic)
At the start: 12 parts, among them U25 CAT811TTBI-GT3, U27 MCP1825T-3302E/DC

Commit message: buttons
Parts:
- renumbered D3 to D1, D12 to D2, R95 to R1, R96 to R2, TP12 to TP1, TP12 to TP2, U27 to U1, U25 to U2
Changed lines of the file:
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@@
   (symbol (lib_id "KD_Resistor:R_0603_360_1%") (at 219.71 118.11 180) (unit 1)
     (in_bom yes) (on_board yes) (dnp no) (fields_autoplaced)
-    (property "Reference" "R96" (at 222.25 116.84 0)
+    (property "Reference" "R2" (at 222.25 116.84 0)
       (effects (font (size 1.27 1.27)) (justify right))
     )
@@
   (symbol (lib_id "KD_Resistor:R_0603_360_1%") (at 123.19 133.35 90) (unit 1)
     (in_bom yes) (on_board yes) (dnp no) (fields_autoplaced)
-    (property "Reference" "R95" (at 123.19 127 90)
+    (property "Reference" "R1" (at 123.19 127 90)
       (effects (font (size 1.27 1.27)))
     )
@@
   (symbol (lib_id "KD_IC_Regulator_DC_Converter:Regulator_3v3_500mA_0.5%_MCP1825T-3302E/DC") (at 93.98 128.27 0) (unit 1)
     (in_bom yes) (on_board yes) (dnp no) (fields_autoplaced)
-    (property "Reference" "U27" (at 93.98 121.92 0) (do_not_autoplace)
+    (property "Reference" "U1" (at 93.98 121.92 0) (do_not_autoplace)
       (effects (font (size 1.27 1.27)))
     )
@@
   (symbol (lib_id "KD_Led:0603_Green_Diff_B1911NG--20D000214U1930") (at 219.71 128.27 90) (unit 1)
     (in_bom yes) (on_board yes) (dnp no) (fields_autoplaced)
-    (property "Reference" "D12" (at 223.52 128.5875 90)
+    (property "Reference" "D2" (at 223.52 128.5875 90)
       (effects (font (size 1.27 1.27)) (justify right))
     )
@@
   (symbol (lib_id "KD_Connector_Pads:TestPoint_2.5mm_H0.9") (at 214.63 107.95 0) (unit 1)
     (in_bom yes) (on_board yes) (dnp no)
-    (property "Reference" "TP12" (at 214.63 102.87 0) (do_not_autoplace)
+    (property "Reference" "TP2" (at 214.63 102.87 0) (do_not_autoplace)
       (effects (font (size 1.27 1.27)))
     )
@@
   (symbol (lib_id "KD_Led:0603_Red_Diff_B1911USD-20D000114U1930") (at 114.3 133.35 0) (unit 1)
     (in_bom yes) (on_board yes) (dnp no) (fields_autoplaced)
-    (property "Reference" "D3" (at 112.7125 127 0)
+    (property "Reference" "D1" (at 112.7125 127 0)
       (effects (font (size 1.27 1.27)))
     )
@@
   (symbol (lib_id "KD_Connector_Pads:TestPoint_2.5mm_H0.9") (at 132.08 110.49 0) (unit 1)
     (in_bom yes) (on_board yes) (dnp no)
-    (property "Reference" "TP12" (at 132.08 105.41 0) (do_not_autoplace)
+    (property "Reference" "TP1" (at 132.08 105.41 0) (do_not_autoplace)
       (effects (font (size 1.27 1.27)))
     )
@@
   (symbol (lib_id "power:GND") (at 209.55 119.38 0) (unit 1)
     (in_bom yes) (on_board yes) (dnp no) (fields_autoplaced)
-    (property "Reference" "#PWR041" (at 209.55 125.73 0)
+    (property "Reference" "#PWR04" (at 209.55 125.73 0)
       (effects (font (size 1.27 1.27)) hide)
     )
@@
   (symbol (lib_id "KD_IC_Other:Supervisor_CAT811TTBI-GT3") (at 184.15 111.76 0) (unit 1)
     (in_bom yes) (on_board yes) (dnp no) (fields_autoplaced)
-    (property "Reference" "U25" (at 186.69 105.664 0) (do_not_autoplace)
+    (property "Reference" "U2" (at 186.69 105.664 0) (do_not_autoplace)
       (effects (font (size 1.27 1.27)) (justify left))
     )

Commit message: Schematic
Other:
- title: TITLE -> Programmable Keyboard
Changed lines of the file:
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@@
   (paper "A4")
   (title_block
-    (title "TITLE")
-    (date "2023-05-28")
+    (title "Programmable Keyboard")
+    (date "2023-10-14")
     (rev "1.0")
     (company "Kallio Designs Oy")
-    (comment 1 "Teemu Latonen")
+    (comment 1 "TL, NH")
     (comment 2 "ASSEMBLY_PN")
     (comment 3 "PCB_PN")

Commit message: updates
Parts:
- renumbered D1 to D5, D2 to D6, R1 to R32, R2 to R33, TP1 to TP13, TP2 to TP14, U1 to U6, U2 to U7
Changed lines of the file:
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@@
   (symbol (lib_id "KD_Resistor:R_0603_360_1%") (at 219.71 118.11 180) (unit 1)
     (in_bom yes) (on_board yes) (dnp no) (fields_autoplaced)
-    (property "Reference" "R2" (at 222.25 116.84 0)
+    (property "Reference" "R33" (at 222.25 116.84 0)
       (effects (font (size 1.27 1.27)) (justify right))
     )
@@
       (project "000018 PGKB"
         (path "/e63e39d7-6ac0-4ffd-8aa3-1841a4541b55/2eb44e1a-4042-4ea6-aca2-4836a6ec84e9/91422aee-53cf-4c28-8efa-7ede5a87a80b"
-          (reference "R2") (unit 1)
+          (reference "R33") (unit 1)
         )
       )
@@
       (project "000018 PGKB"
         (path "/e63e39d7-6ac0-4ffd-8aa3-1841a4541b55/2eb44e1a-4042-4ea6-aca2-4836a6ec84e9/91422aee-53cf-4c28-8efa-7ede5a87a80b"
-          (reference "#PWR05") (unit 1)
+          (reference "#PWR037") (unit 1)
         )
       )
@@
   (symbol (lib_id "KD_Resistor:R_0603_360_1%") (at 123.19 133.35 90) (unit 1)
     (in_bom yes) (on_board yes) (dnp no) (fields_autoplaced)
-    (property "Reference" "R1" (at 123.19 127 90)
+    (property "Reference" "R32" (at 123.19 127 90)
       (effects (font (size 1.27 1.27)))
     )
@@
       (project "000018 PGKB"
         (path "/e63e39d7-6ac0-4ffd-8aa3-1841a4541b55/2eb44e1a-4042-4ea6-aca2-4836a6ec84e9/91422aee-53cf-4c28-8efa-7ede5a87a80b"
-          (reference "R1") (unit 1)
+          (reference "R32") (unit 1)
         )
       )
@@
       (project "000018 PGKB"
         (path "/e63e39d7-6ac0-4ffd-8aa3-1841a4541b55/2eb44e1a-4042-4ea6-aca2-4836a6ec84e9/91422aee-53cf-4c28-8efa-7ede5a87a80b"
-          (reference "#+3V01") (unit 1)
+          (reference "#+3V08") (unit 1)
         )
       )
@@
       (project "000018 PGKB"
         (path "/e63e39d7-6ac0-4ffd-8aa3-1841a4541b55/2eb44e1a-4042-4ea6-aca2-4836a6ec84e9/91422aee-53cf-4c28-8efa-7ede5a87a80b"
-          (reference "#PWR03") (unit 1)
+          (reference "#PWR035") (unit 1)
         )
       )
@@
       (project "000018 PGKB"
         (path "/e63e39d7-6ac0-4ffd-8aa3-1841a4541b55/2eb44e1a-4042-4ea6-aca2-4836a6ec84e9/91422aee-53cf-4c28-8efa-7ede5a87a80b"
-          (reference "C1") (unit 1)
+          (reference "C36") (unit 1)
         )
       )
@@
       (project "000018 PGKB"
         (path "/e63e39d7-6ac0-4ffd-8aa3-1841a4541b55/2eb44e1a-4042-4ea6-aca2-4836a6ec84e9/91422aee-53cf-4c28-8efa-7ede5a87a80b"
-          (reference "#PWR01") (unit 1)
+          (reference "#PWR033") (unit 1)
         )
       )
@@
   (symbol (lib_id "KD_IC_Regulator_DC_Converter:Regulator_3v3_500mA_0.5%_MCP1825T-3302E/DC") (at 93.98 128.27 0) (unit 1)
     (in_bom yes) (on_board yes) (dnp no) (fields_autoplaced)
-    (property "Reference" "U1" (at 93.98 121.92 0) (do_not_autoplace)
+    (property "Reference" "U6" (at 93.98 121.92 0) (do_not_autoplace)
       (effects (font (size 1.27 1.27)))
     )
@@
       (project "000018 PGKB"
         (path "/e63e39d7-6ac0-4ffd-8aa3-1841a4541b55/2eb44e1a-4042-4ea6-aca2-4836a6ec84e9/91422aee-53cf-4c28-8efa-7ede5a87a80b"
-          (reference "U1") (unit 1)
+          (reference "U6") (unit 1)
         )
       )
@@
   (symbol (lib_id "KD_Led:0603_Green_Diff_B1911NG--20D000214U1930") (at 219.71 128.27 90) (unit 1)
     (in_bom yes) (on_board yes) (dnp no) (fields_autoplaced)
-    (property "Reference" "D2" (at 223.52 128.5875 90)
+    (property "Reference" "D6" (at 223.52 128.5875 90)
       (effects (font (size 1.27 1.27)) (justify right))
     )
@@
       (project "000018 PGKB"
         (path "/e63e39d7-6ac0-4ffd-8aa3-1841a4541b55/2eb44e1a-4042-4ea6-aca2-4836a6ec84e9/91422aee-53cf-4c28-8efa-7ede5a87a80b"
-          (reference "D2") (unit 1)
+          (reference "D6") (unit 1)
         )
       )
@@
       (project "000018 PGKB"
         (path "/e63e39d7-6ac0-4ffd-8aa3-1841a4541b55/2eb44e1a-4042-4ea6-aca2-4836a6ec84e9/91422aee-53cf-4c28-8efa-7ede5a87a80b"
-          (reference "C2") (unit 1)
+          (reference "C37") (unit 1)
         )
       )
@@
   (symbol (lib_id "KD_Connector_Pads:TestPoint_2.5mm_H0.9") (at 214.63 107.95 0) (unit 1)
     (in_bom yes) (on_board yes) (dnp no)
-    (property "Reference" "TP2" (at 214.63 102.87 0) (do_not_autoplace)
+    (property "Reference" "TP14" (at 214.63 102.87 0) (do_not_autoplace)
       (effects (font (size 1.27 1.27)))
     )
@@
       (project "000018 PGKB"
         (path "/e63e39d7-6ac0-4ffd-8aa3-1841a4541b55/2eb44e1a-4042-4ea6-aca2-4836a6ec84e9/91422aee-53cf-4c28-8efa-7ede5a87a80b"
-          (reference "TP2") (unit 1)
+          (reference "TP14") (unit 1)
         )
       )
@@
       (project "000018 PGKB"
         (path "/e63e39d7-6ac0-4ffd-8aa3-1841a4541b55/2eb44e1a-4042-4ea6-aca2-4836a6ec84e9/91422aee-53cf-4c28-8efa-7ede5a87a80b"
-          (reference "FB1") (unit 1)
+          (reference "FB3") (unit 1)
         )
       )
@@
   (symbol (lib_id "KD_Led:0603_Red_Diff_B1911USD-20D000114U1930") (at 114.3 133.35 0) (unit 1)
     (in_bom yes) (on_board yes) (dnp no) (fields_autoplaced)
-    (property "Reference" "D1" (at 112.7125 127 0)
+    (property "Reference" "D5" (at 112.7125 127 0)
       (effects (font (size 1.27 1.27)))
     )
@@
       (project "000018 PGKB"
         (path "/e63e39d7-6ac0-4ffd-8aa3-1841a4541b55/2eb44e1a-4042-4ea6-aca2-4836a6ec84e9/91422aee-53cf-4c28-8efa-7ede5a87a80b"
-          (reference "D1") (unit 1)
+          (reference "D5") (unit 1)
         )
       )
@@
       (project "000018 PGKB"
         (path "/e63e39d7-6ac0-4ffd-8aa3-1841a4541b55/2eb44e1a-4042-4ea6-aca2-4836a6ec84e9/91422aee-53cf-4c28-8efa-7ede5a87a80b"
-          (reference "C3") (unit 1)
+          (reference "C38") (unit 1)
         )
       )
@@
       (project "000018 PGKB"
         (path "/e63e39d7-6ac0-4ffd-8aa3-1841a4541b55/2eb44e1a-4042-4ea6-aca2-4836a6ec84e9/91422aee-53cf-4c28-8efa-7ede5a87a80b"
-          (reference "#+3V02") (unit 1)
+          (reference "#+3V09") (unit 1)
         )
       )
@@
       (project "000018 PGKB"
         (path "/e63e39d7-6ac0-4ffd-8aa3-1841a4541b55/2eb44e1a-4042-4ea6-aca2-4836a6ec84e9/91422aee-53cf-4c28-8efa-7ede5a87a80b"
-          (reference "#PWR02") (unit 1)
+          (reference "#PWR034") (unit 1)
         )
       )
@@
   (symbol (lib_id "KD_Connector_Pads:TestPoint_2.5mm_H0.9") (at 132.08 110.49 0) (unit 1)
     (in_bom yes) (on_board yes) (dnp no)
-    (property "Reference" "TP1" (at 132.08 105.41 0) (do_not_autoplace)
+    (property "Reference" "TP13" (at 132.08 105.41 0) (do_not_autoplace)
       (effects (font (size 1.27 1.27)))
     )
@@
       (project "000018 PGKB"
         (path "/e63e39d7-6ac0-4ffd-8aa3-1841a4541b55/2eb44e1a-4042-4ea6-aca2-4836a6ec84e9/91422aee-53cf-4c28-8efa-7ede5a87a80b"
-          (reference "TP1") (unit 1)
+          (reference "TP13") (unit 1)
         )
       )
@@
   (symbol (lib_id "power:GND") (at 209.55 119.38 0) (unit 1)
     (in_bom yes) (on_board yes) (dnp no) (fields_autoplaced)
-    (property "Reference" "#PWR04" (at 209.55 125.73 0)
+    (property "Reference" "#PWR036" (at 209.55 125.73 0)
       (effects (font (size 1.27 1.27)) hide)
     )
@@
       (project "000018 PGKB"
         (path "/e63e39d7-6ac0-4ffd-8aa3-1841a4541b55/2eb44e1a-4042-4ea6-aca2-4836a6ec84e9/91422aee-53cf-4c28-8efa-7ede5a87a80b"
-          (reference "#PWR04") (unit 1)
+          (reference "#PWR036") (unit 1)
         )
       )
@@
       (project "000018 PGKB"
         (path "/e63e39d7-6ac0-4ffd-8aa3-1841a4541b55/2eb44e1a-4042-4ea6-aca2-4836a6ec84e9/91422aee-53cf-4c28-8efa-7ede5a87a80b"
-          (reference "#+3V03") (unit 1)
+          (reference "#+3V010") (unit 1)
         )
       )
@@
   (symbol (lib_id "KD_IC_Other:Supervisor_CAT811TTBI-GT3") (at 184.15 111.76 0) (unit 1)
     (in_bom yes) (on_board yes) (dnp no) (fields_autoplaced)
-    (property "Reference" "U2" (at 186.69 105.664 0) (do_not_autoplace)
+    (property "Reference" "U7" (at 186.69 105.664 0) (do_not_autoplace)
       (effects (font (size 1.27 1.27)) (justify left))
     )
@@
       (project "000018 PGKB"
         (path "/e63e39d7-6ac0-4ffd-8aa3-1841a4541b55/2eb44e1a-4042-4ea6-aca2-4836a6ec84e9/91422aee-53cf-4c28-8efa-7ede5a87a80b"
-          (reference "U2") (unit 1)
-        )
-      )
+          (reference "U7") (unit 1)
+        )
+      )
