File: PCB/Rev 02.00/000018 PGKB/000018 PGKB.kicad_pcb (KiCad board)
At the start: 2 copper layers, 64.9 x 50.6 mm, 49 parts, among them J1 USB_B_V_Adam_USB-B-S-VT, U1 MCP1825T-3302E/DC, U2 CAT811TTBI-GT3, U3 RP2040, Y1 8 MHz

Commit message: schematic
Parts:
- added C12: 27p, KD_Capacitor:CAPC1608X90N, F.Cu at (170.4, 103.4)
- added C13: 100n, KD_Capacitor:CAPC1608X90N, F.Cu at (170.4, 106.0)
- added C14: 100n, KD_Capacitor:CAPC1608X90N, F.Cu at (170.4, 108.5)
- added C15: 100n, KD_Capacitor:CAPC1608X90N, F.Cu at (174.4, 88.4)
- added C16: 100n, KD_Capacitor:CAPC1608X90N, F.Cu at (174.4, 90.9)
- added C17: 100n, KD_Capacitor:CAPC1608X90N, F.Cu at (174.4, 93.4)
- added C18: 1u, KD_Capacitor:CAPC2012X135N, F.Cu at (186.8, 117.2)
- added C19: 100n, KD_Capacitor:CAPC1608X90N, F.Cu at (174.4, 95.9)
- added C20: 1u, KD_Capacitor:CAPC2012X135N, F.Cu at (186.8, 120.2)
- added C21: 100n, KD_Capacitor:CAPC1608X90N, F.Cu at (174.4, 98.4)
- added C22: 100n, KD_Capacitor:CAPC1608X90N, F.Cu at (174.4, 100.9)
- added C23: 1u, KD_Capacitor:CAPC2012X135N, F.Cu at (186.8, 123.3)
- added C24: 100n, KD_Capacitor:CAPC1608X90N, F.Cu at (174.4, 103.4)
- added C52: 10n, KD_Capacitor:CAPC1608X90N, F.Cu at (174.4, 106.0)
- added C53: 10n, KD_Capacitor:CAPC1608X90N, F.Cu at (174.4, 108.5)
- added C54: 10n, KD_Capacitor:CAPC1608X90N, F.Cu at (178.4, 88.4)
- added C55: 10n, KD_Capacitor:CAPC1608X90N, F.Cu at (178.4, 90.9)
- added C56: 10n, KD_Capacitor:CAPC1608X90N, F.Cu at (178.4, 93.4)
- added C57: 10n, KD_Capacitor:CAPC1608X90N, F.Cu at (178.4, 95.9)
- added D5: Schottky_30V_200mA_DCo_BAT54WS, KD_Diode:D_SOD-323, F.Cu at (165.9, 126.7)
- added D6: Schottky_30V_1A_PMEG3010ER_115, KD_Diode:DIOC360X180X150_SOD123, F.Cu at (171.3, 128.9)
- added J2: BM04B-SRSS-TB, KD_Connector_Rectangular:JST_SH_BM04B-SRSS-TB_1x04-1MP_P1.00mm_Vertical, F.Cu at (192.9, 90.2)
- added R12: 1k, KD_Resistor:RESC1608X55N, F.Cu at (182.4, 98.4)
- added R13: 1k, KD_Resistor:RESC1608X55N, F.Cu at (182.4, 100.9)
- added R14: R_0603_5100_1%, KD_Resistor:RESC1608X55N, F.Cu at (182.4, 103.4)
- added R15: R_0603_5100_1%, KD_Resistor:RESC1608X55N, F.Cu at (182.4, 106.0)
- added R16: 10k, KD_Resistor:RESC1608X55N, F.Cu at (182.4, 108.5)
- added R50: 1k, KD_Resistor:RESC1608X55N, F.Cu at (186.4, 88.4)
- added R51: 1k, KD_Resistor:RESC1608X55N, F.Cu at (186.4, 90.9)
- added R52: 1k, KD_Resistor:RESC1608X55N, F.Cu at (186.4, 93.4)
- added R53: 1k, KD_Resistor:RESC1608X55N, F.Cu at (186.4, 95.9)
- added R54: 1k, KD_Resistor:RESC1608X55N, F.Cu at (186.4, 98.4)
- added R55: 1k, KD_Resistor:RESC1608X55N, F.Cu at (186.4, 100.9)
- added S3: Button_tactile_45x38_430181038816, KD_Switch:SW_Push_1P1T_NO_Wurth_430181038816, F.Cu at (163.8, 104.2)
- added S4: Button_tactile_45x38_430181038816, KD_Switch:SW_Push_1P1T_NO_Wurth_430181038816, F.Cu at (163.8, 111.1)
- added S5: Button_tactile_45x38_430181038816, KD_Switch:SW_Push_1P1T_NO_Wurth_430181038816, F.Cu at (163.8, 118.0)
- added TP12: TP D2.5 mm H0.9mm, KD_Connector_Pads:TestPoint_Pad_D2.5mm_H0.9mm, F.Cu at (182.6, 115.8)
- added TP7: TP D2.5 mm H0.9mm, KD_Connector_Pads:TestPoint_Pad_D2.5mm_H0.9mm, F.Cu at (178.5, 111.7)
- added TP8: TP D2.5 mm H0.9mm, KD_Connector_Pads:TestPoint_Pad_D2.5mm_H0.9mm, F.Cu at (178.5, 115.8)
- added TP9: TP D2.5 mm H0.9mm, KD_Connector_Pads:TestPoint_Pad_D2.5mm_H0.9mm, F.Cu at (182.6, 111.7)
- added U12: SN74HCS365PWR, KD_Package_SO:SOP65P600X150-16N, F.Cu at (192.2, 97.7)
- C7: value 100n -> 27p
- J1: value USB_B_V_Adam_USB-B-S-VT -> USB Mini B; footprint KD_Connector_USB_HDMI_Etc:USB_B_Vertical_Adam_USB-B-S-VT -> KD_Connector_USB_HDMI_Etc:USB_C_Receptacle_GCT_USB4085
- R5: footprint KD_Resistor:RESC1608X55N -> KD_Resistor:RESC1608X55N_DNP
- Y1: value 8 MHz -> 12 MHz
- moved FB2 54.4 mm to (197.9, 97.5)
- moved C6 51.9 mm to (192.3, 105.0)
- moved C4 51.2 mm to (199.0, 107.0)
- moved U1 49.6 mm to (194.1, 125.4)
- moved R6 47.5 mm to (179.9, 124.7)
- moved R7 47.5 mm to (179.9, 127.6)
- moved TP3 46.2 mm to (198.8, 88.7)
- moved TP4 46.2 mm to (198.8, 91.7)
- moved U3 45.1 mm to (173.0, 122.5)
- moved FB3 41.3 mm to (197.9, 100.2)
- moved Y1 40.3 mm to (180.7, 120.2)
- moved D1 40.3 mm to (186.8, 126.1)
- moved D2 40.3 mm to (186.8, 128.7)
- moved R5 39.7 mm to (178.4, 108.5)
- moved U2 37.0 mm to (161.4, 123.9)
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Connections:
- C7 pad 1: GND -> Net-(U3-XIN)
- C7 pad 2: +3V3 -> GND
- C8 pad 1: Net-(C8-Pad1) -> Net-(U3-ADC_AVDD)
- C9 pad 1: Net-(C8-Pad1) -> Net-(U3-ADC_AVDD)
- FB2 pad 1: Net-(D3-V+) -> Net-(D6-K)
- FB3 pad 1: unconnected-(FB3-Pad1) -> +3V3
- FB3 pad 2: unconnected-(FB3-Pad2) -> Net-(U3-ADC_AVDD)
- R6 pad 2: /Main/Microcontroller/SCL -> /Main/Microcontroller/SDA
- R7 pad 2: /Main/Microcontroller/SDA -> /Main/Microcontroller/SCL
- S2 pad 3: /Main/Microcontroller/BOOT -> /Main/Microcontroller/USBBOOT
- TP5 pad 1: /Main/Microcontroller/SDA -> /Main/Microcontroller/SCL
- TP6 pad 1: /Main/Microcontroller/SCL -> /Main/Microcontroller/SDA
- U3 pad 1: Net-(U3-IOVDD-Pad1) -> Net-(U3-ADC_AVDD)
- U3 pad 10: Net-(U3-IOVDD-Pad1) -> Net-(U3-ADC_AVDD)
- U3 pad 19: unconnected-(U3-TESTEN-Pad19) -> GND
- U3 pad 2: unconnected-(U3-GPIO0-Pad2) -> /Main/Microcontroller/GPIO0
- U3 pad 21: unconnected-(U3-XOUT-Pad21) -> Net-(U3-XOUT)
- U3 pad 22: Net-(U3-IOVDD-Pad1) -> Net-(U3-ADC_AVDD)
- U3 pad 23: Net-(U3-DVDD-Pad23) -> /Main/Microcontroller/1V2
- U3 pad 3: unconnected-(U3-GPIO1-Pad3) -> /Main/Microcontroller/GPIO1
- U3 pad 30: unconnected-(U3-GPIO19-Pad30) -> /Main/Microcontroller/UART_TX
- U3 pad 32: unconnected-(U3-GPIO21-Pad32) -> /Main/Microcontroller/USBBOOT
- U3 pad 33: Net-(U3-IOVDD-Pad1) -> Net-(U3-ADC_AVDD)
- U3 pad 34: unconnected-(U3-GPIO22-Pad34) -> /Main/Microcontroller/I2C1_SDA
- U3 pad 35: unconnected-(U3-GPIO23-Pad35) -> /Main/Microcontroller/I2C1_SCL
- U3 pad 36: unconnected-(U3-GPIO24-Pad36) -> /Main/Microcontroller/SDA
- U3 pad 37: unconnected-(U3-GPIO25-Pad37) -> /Main/Microcontroller/SCL
- U3 pad 4: unconnected-(U3-GPIO2-Pad4) -> /Main/Microcontroller/GPIO2
- U3 pad 42: Net-(U3-IOVDD-Pad1) -> Net-(U3-ADC_AVDD)
- U3 pad 43: unconnected-(U3-ADC_AVDD-Pad43) -> Net-(U3-ADC_AVDD)
- U3 pad 44: unconnected-(U3-VREG_IN-Pad44) -> Net-(U3-ADC_AVDD)
- U3 pad 45: unconnected-(U3-VREG_VOUT-Pad45) -> /Main/Microcontroller/1V2
- U3 pad 48: unconnected-(U3-USB_VDD-Pad48) -> Net-(U3-ADC_AVDD)
- U3 pad 49: Net-(U3-IOVDD-Pad1) -> Net-(U3-ADC_AVDD)
- U3 pad 5: unconnected-(U3-GPIO3-Pad5) -> /Main/Microcontroller/SPI_MOSI
- U3 pad 50: Net-(U3-DVDD-Pad23) -> /Main/Microcontroller/1V2
- U3 pad 6: unconnected-(U3-GPIO4-Pad6) -> /Main/Microcontroller/SPI_MISO
- U3 pad 7: unconnected-(U3-GPIO5-Pad7) -> /Main/Microcontroller/UART_RX
- U3 pad 8: unconnected-(U3-GPIO6-Pad8) -> /Main/Microcontroller/SPI_CLK
- Y1 pad 1: +3V3 -> Net-(U3-XIN)
- Y1 pad 3: Net-(U3-XIN) -> Net-(C12-Pad1)
- Y1 pad 4: +3V3 -> GND

Commit message: buttons
Parts:
- added C25: 10n, KD_Capacitor:CAPC1608X90N, F.Cu at (224.0, 128.0)
- added C26: 10n, KD_Capacitor:CAPC1608X90N, F.Cu at (224.0, 125.5)
- added C27: 10n, KD_Capacitor:CAPC1608X90N, F.Cu at (224.0, 123.0)
- added C28: 10n, KD_Capacitor:CAPC1608X90N, F.Cu at (224.0, 120.5)
- added C29: 10n, KD_Capacitor:CAPC1608X90N, F.Cu at (224.0, 118.0)
- added C30: 10n, KD_Capacitor:CAPC1608X90N, F.Cu at (224.0, 115.5)
- added C31: 100n, KD_Capacitor:CAPC1608X90N, F.Cu at (228.0, 140.6)
- added R17: 1k, KD_Resistor:RESC1608X55N, F.Cu at (232.0, 115.5)
- added R18: 1k, KD_Resistor:RESC1608X55N, F.Cu at (236.0, 140.6)
- added R19: 1k, KD_Resistor:RESC1608X55N, F.Cu at (236.0, 138.1)
- added R20: 1k, KD_Resistor:RESC1608X55N, F.Cu at (236.0, 135.6)
- added R21: 1k, KD_Resistor:RESC1608X55N, F.Cu at (236.0, 133.1)
- added R22: 1k, KD_Resistor:RESC1608X55N, F.Cu at (236.0, 130.6)
- added S10: 5124, KD_Switch:SWITCH_BUTTON_Kailh_mx, F.Cu at (195.4, 100.1)
- added S11: 5124, KD_Switch:SWITCH_BUTTON_Kailh_mx, F.Cu at (210.4, 100.1)
- added S12: 5124, KD_Switch:SWITCH_BUTTON_Kailh_mx, F.Cu at (180.3, 83.5)
- added S13: 5124, KD_Switch:SWITCH_BUTTON_Kailh_mx, F.Cu at (195.4, 83.5)
- added S14: 5124, KD_Switch:SWITCH_BUTTON_Kailh_mx, F.Cu at (210.4, 83.5)
- added S6: 5124, KD_Switch:SWITCH_BUTTON_Kailh_mx, F.Cu at (180.3, 116.8)
- added S7: 5124, KD_Switch:SWITCH_BUTTON_Kailh_mx, F.Cu at (195.4, 116.8)
- added S8: 5124, KD_Switch:SWITCH_BUTTON_Kailh_mx, F.Cu at (210.4, 116.8)
- added S9: 5124, KD_Switch:SWITCH_BUTTON_Kailh_mx, F.Cu at (180.3, 100.1)
- added TP10: TP D2.5 mm H0.9mm, KD_Connector_Pads:TestPoint_Pad_D2.5mm_H0.9mm, F.Cu at (232.2, 94.5)
- added TP11: TP D2.5 mm H0.9mm, KD_Connector_Pads:TestPoint_Pad_D2.5mm_H0.9mm, F.Cu at (220.0, 90.4)
- added TP13: TP D2.5 mm H0.9mm, KD_Connector_Pads:TestPoint_Pad_D2.5mm_H0.9mm, F.Cu at (228.1, 90.4)
- added U4: W25Q80DVSSIG, KD_Package_SO:SOIC127P790X195-8N, F.Cu at (232.4, 110.6)
- added U5: SN74HCS365PWR, KD_Package_SO:SOP65P600X150-16N, F.Cu at (230.7, 84.1)
- S3, S4, S5: value Button_tactile_45x38_430181038816 -> 5124; footprint KD_Switch:SW_Push_1P1T_NO_Wurth_430181038816 -> KD_Switch:SWITCH_BUTTON_Kailh_mx
- moved U2 78.9 mm to (240.2, 124.3), turned to 180 degrees
- moved C1 72.0 mm to (220.0, 140.6), turned to 180 degrees
- moved R8 70.2 mm to (232.0, 138.1), turned to 180 degrees
- moved C17 68.4 mm to (224.0, 140.6), turned to 180 degrees
- moved C3 68.4 mm to (220.0, 138.1), turned to 180 degrees
- moved C54 66.7 mm to (228.0, 133.1), turned to 180 degrees
- moved R9 66.7 mm to (232.0, 135.6), turned to 180 degrees
- moved U1 65.7 mm to (236.8, 75.6), turned to 180 degrees
- moved C19 65.1 mm to (224.0, 138.1), turned to 180 degrees
- moved C5 65.1 mm to (220.0, 135.6), turned to 180 degrees
- moved D4 64.6 mm to (196.2, 73.6), turned to 180 degrees
- moved C55 63.5 mm to (228.0, 130.6), turned to 180 degrees
- moved R10 63.5 mm to (232.0, 133.1), turned to 180 degrees
- moved R50 63.5 mm to (236.0, 128.0), turned to 180 degrees
- moved U3 62.9 mm to (222.6, 83.7), turned to 180 degrees
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Connections:
- R53 pad 1: unconnected-(R53-Pad1) -> Net-(R53-Pad1)
- R54 pad 1: unconnected-(R54-Pad1) -> Net-(R54-Pad1)
- R55 pad 1: unconnected-(R55-Pad1) -> Net-(R55-Pad1)
- S3 pad 1: unconnected-(S3-Pad1) -> (no net)
- S4 pad 1: unconnected-(S4-Pad1) -> (no net)
- S5 pad 1: unconnected-(S5-Pad1) -> (no net)
- U12 pad 11: /Main/Untitled Sheet/Button1 -> /Main/Buttons/Button1
- U12 pad 13: /Main/Untitled Sheet/Button0 -> /Main/Buttons/Button0
- U12 pad 3: /Main/Untitled Sheet/Button5 -> /Main/Buttons/Button5
- U12 pad 5: /Main/Untitled Sheet/Button4 -> /Main/Buttons/Button4
- U12 pad 7: /Main/Untitled Sheet/Button3 -> /Main/Buttons/Button3
- U12 pad 9: /Main/Untitled Sheet/Button2 -> /Main/Buttons/Button2
- U3 pad 11: unconnected-(U3-GPIO8-Pad11) -> /Main/Buttons/Button4
- U3 pad 12: unconnected-(U3-GPIO9-Pad12) -> /Main/Buttons/Button5
- U3 pad 13: unconnected-(U3-GPIO10-Pad13) -> /Main/Microcontroller/DEBUG_LED_GREEN
- U3 pad 14: unconnected-(U3-GPIO11-Pad14) -> /Main/Microcontroller/DEBUG_LED_RED
- U3 pad 15: unconnected-(U3-GPIO12-Pad15) -> /Main/Microcontroller/DEBUG_LED_BLUE
- U3 pad 16: unconnected-(U3-GPIO13-Pad16) -> /Main/Buttons1/Button0
- U3 pad 17: unconnected-(U3-GPIO14-Pad17) -> /Main/Buttons1/Button1
- U3 pad 18: unconnected-(U3-GPIO15-Pad18) -> /Main/Buttons1/Button2
- U3 pad 2: /Main/Microcontroller/GPIO0 -> /Main/Buttons/Button0
- U3 pad 27: unconnected-(U3-GPIO16-Pad27) -> /Main/Buttons1/Button3
- U3 pad 28: unconnected-(U3-GPIO17-Pad28) -> /Main/Microcontroller/ENC_A
- U3 pad 29: unconnected-(U3-GPIO18-Pad29) -> /Main/Microcontroller/ENC_B
- U3 pad 3: /Main/Microcontroller/GPIO1 -> /Main/Buttons/Button1
- U3 pad 38: unconnected-(U3-GPIO26_ADC0-Pad38) -> /Main/Microcontroller/NEOPIX_DRIVE
- U3 pad 39: unconnected-(U3-GPIO27_ADC1-Pad39) -> /Main/Buttons1/Button4
- U3 pad 4: /Main/Microcontroller/GPIO2 -> /Main/Buttons/Button2
- U3 pad 40: unconnected-(U3-GPIO28_ADC2-Pad40) -> /Main/Buttons1/Button5
- U3 pad 41: unconnected-(U3-GPIO29_ADC3-Pad41) -> /Main/Microcontroller/GPIO12
- U3 pad 9: unconnected-(U3-GPIO7-Pad9) -> /Main/Buttons/Button3
Other:
- board size 64.9 x 50.6 mm -> 112 x 73.3 mm

Commit message: updates
Parts:
- removed C52, C53, C54, C55, C56, C57: 10n, KD_Capacitor:CAPC1608X90N
- removed D4: RGB_Clear_APTF1616SEEZGQBDC, KD_Diode:LEDM1616X80-4N_B
- removed R50, R51, R52, R53, R54, R55: 1k, KD_Resistor:RESC1608X55N
- removed S14: 5124, KD_Switch:SWITCH_BUTTON_Kailh_mx
- removed TP10: TP D2.5 mm H0.9mm, KD_Connector_Pads:TestPoint_Pad_D2.5mm_H0.9mm
- removed U12: SN74HCS365PWR, KD_Package_SO:SOP65P600X150-16N
- added C32: 100n, KD_Capacitor:CAPC1608X90N, F.Cu at (221.7, 120.0)
- added C33: 100n, KD_Capacitor:CAPC1608X90N, F.Cu at (204.1, 124.0)
- added C34: 100n, KD_Capacitor:CAPC1608X90N, F.Cu at (206.6, 124.0)
- added C35: 100n, KD_Capacitor:CAPC1608X90N, F.Cu at (241.5, 89.2)
- added C36: 100n, KD_Capacitor:CAPC1608X90N, F.Cu at (241.5, 91.7)
- added C37: 10u, KD_Capacitor:CAPC3216X150N, F.Cu at (237.0, 107.9)
- added C38: 100n, KD_Capacitor:CAPC1608X90N, F.Cu at (241.5, 94.2)
- added C39: 1u, KD_Capacitor:CAPC2012X135N, F.Cu at (246.0, 121.2)
- added C40: 100n, KD_Capacitor:CAPC1608X90N, F.Cu at (241.5, 96.7)
- added D10: Neopixel Reverse, KD_Diode:LEDM_NEO3535_REVERSE_SK6812-E, F.Cu at (190.0, 105.9)
- added D11: Neopixel Reverse, KD_Diode:LEDM_NEO3535_REVERSE_SK6812-E, F.Cu at (194.8, 105.9)
- added D12: Neopixel Reverse, KD_Diode:LEDM_NEO3535_REVERSE_SK6812-E, F.Cu at (199.6, 105.9)
- added D13: Neopixel Reverse, KD_Diode:LEDM_NEO3535_REVERSE_SK6812-E, F.Cu at (204.5, 105.9)
- added D14: Neopixel Reverse, KD_Diode:LEDM_NEO3535_REVERSE_SK6812-E, F.Cu at (209.3, 105.9)
- added D15: Neopixel Reverse, KD_Diode:LEDM_NEO3535_REVERSE_SK6812-E, F.Cu at (214.1, 105.9)
- added D16: Neopixel Reverse, KD_Diode:LEDM_NEO3535_REVERSE_SK6812-E, F.Cu at (219.0, 105.9)
- added D7: Neopixel Reverse, KD_Diode:LEDM_NEO3535_REVERSE_SK6812-E, F.Cu at (175.4, 105.9)
- added D8: Neopixel Reverse, KD_Diode:LEDM_NEO3535_REVERSE_SK6812-E, F.Cu at (180.3, 105.9)
- added D9: Neopixel Reverse, KD_Diode:LEDM_NEO3535_REVERSE_SK6812-E, F.Cu at (185.1, 105.9)
- added R23: 1k, KD_Resistor:RESC1608X55N, F.Cu at (216.7, 132.1)
- added R24: R_0603_22k_1%, KD_Resistor:RESC1608X55N_DNP, F.Cu at (219.2, 132.1)
- added R25: 1k, KD_Resistor:RESC1608X55N, F.Cu at (221.7, 132.1)
- added R26: R_0805_4700_5%, KD_Resistor:RESC2012X50N, F.Cu at (235.7, 104.0)
- added R27: R_0805_4700_5%, KD_Resistor:RESC2012X50N, F.Cu at (238.6, 104.0)
- added R32: R_0603_360_1%, KD_Resistor:RESC1608X55N, F.Cu at (245.5, 94.2)
- added R33: R_0603_360_1%, KD_Resistor:RESC1608X55N, F.Cu at (245.5, 96.7)
- added TP14: TP D2.5 mm H0.9mm, KD_Connector_Pads:TestPoint_Pad_D2.5mm_H0.9mm, F.Cu at (241.7, 116.1)
- added TP15: TP D2.5 mm H0.9mm, KD_Connector_Pads:TestPoint_Pad_D2.5mm_H0.9mm, F.Cu at (241.7, 120.1)
- added TP16: TP D2.5 mm H0.9mm, KD_Connector_Pads:TestPoint_Pad_D2.5mm_H0.9mm, F.Cu at (241.7, 124.2)
- added U6: MCP1825T-3302E/DC, KD_Package_TO_SOT_SMD:SOT127P700X180-6N, F.Cu at (207.0, 139.1)
- added U7: CAT811TTBI-GT3, KD_Package_TO_SOT_SMD:SOT-143_TO-253_M, F.Cu at (246.0, 112.5)
- C1: value 100n -> 10u; footprint KD_Capacitor:CAPC1608X90N -> KD_Capacitor:CAPC3216X150N
- C10, C13, C5, C8: value 100n -> 10n
- C11, C9: value 1u -> 10n; footprint KD_Capacitor:CAPC2012X135N -> KD_Capacitor:CAPC1608X90N
- C12, C7: value 27p -> 10n
- C16, C17: value 100n -> C_0603_100n_X7R_50V
- C18: value 1u -> C_0603_100n_X7R_50V; footprint KD_Capacitor:CAPC2012X135N -> KD_Capacitor:CAPC1608X90N
- C2: value 10u -> 100n; footprint KD_Capacitor:CAPC3216X150N -> KD_Capacitor:CAPC1608X90N
- C21: value 100n -> 1u; footprint KD_Capacitor:CAPC1608X90N -> KD_Capacitor:CAPC2012X135N
- C25, C28: value 10n -> 1u; footprint KD_Capacitor:CAPC1608X90N -> KD_Capacitor:CAPC2012X135N
- C26, C29: value 10n -> 100n
- C27, C30: value 10n -> 27p
- C3: value 100n -> 4u7; footprint KD_Capacitor:CAPC1608X90N -> KD_Capacitor:CAPAE400x540N
- C4: value 10u -> 10n; footprint KD_Capacitor:CAPC3216X150N -> KD_Capacitor:CAPC1608X90N
- C6: value 4u7 -> 10n; footprint KD_Capacitor:CAPAE400x540N -> KD_Capacitor:CAPC1608X90N
- D1: value Red -> TVS_5V5_DRTR5V0U4S-7-M; footprint KD_Diode:LEDM1608X70M -> KD_Package_TO_SOT_SMD:SOT-363_SC-70-6
- D2: value Green -> Schottky_30V_1A_PMEG3010ER_115; footprint KD_Diode:LEDM1608X70M -> KD_Diode:DIOC360X180X150_SOD123
- D3: value TVS_5V5_DRTR5V0U4S-7-M -> Schottky_30V_200mA_DCo_BAT54WS; footprint KD_Package_TO_SOT_SMD:SOT-363_SC-70-6 -> KD_Diode:D_SOD-323
- D5: value Schottky_30V_200mA_DCo_BAT54WS -> Red; footprint KD_Diode:D_SOD-323 -> KD_Diode:LEDM1608X70M
- D6: value Schottky_30V_1A_PMEG3010ER_115 -> Green; footprint KD_Diode:DIOC360X180X150_SOD123 -> KD_Diode:LEDM1608X70M
- FB2: value Ferrite_500mA_TDK_MMZ2012Y152BT000 -> Ferrite_300mA_Abracon_ACML-0805-102-T
- FB3: value Ferrite_300mA_Abracon_ACML-0805-102-T -> Ferrite_500mA_TDK_MMZ2012Y152BT000
- J2: footprint KD_Connector_Rectangular:JST_SH_BM04B-SRSS-TB_1x04-1MP_P1.00mm_Vertical -> KD_Connector_Rectangular:JST_PH_S4B-PH-SM4-TB_1x04-1MP_P2.00mm_Horizontal
- R1, R2: value R_0603_360_1% -> R_0603_5100_1%
- R10, R11, R8: value 49R9 -> 1k
- R14: value R_0603_5100_1% -> 1k
- R15: value R_0603_5100_1% -> R_0603_1k_1%
- R16: value 10k -> R_0603_1k_1%
- R17: value 1k -> R_0603_1k_1%
- R18, R19, R20, R21, R22: value 1k -> 10k
- R5: value R_0603_22k_1% -> 1k; footprint KD_Resistor:RESC1608X55N_DNP -> KD_Resistor:RESC1608X55N
- R6, R7: value R_0805_4700_5% -> 1k; footprint KD_Resistor:RESC2012X50N -> KD_Resistor:RESC1608X55N
- R9: value R_0603_360_1% -> 1k
- S1, S2: value Button_tactile_45x38_430181038816 -> 5124; footprint KD_Switch:SW_Push_1P1T_NO_Wurth_430181038816 -> KD_Switch:SWITCH_BUTTON_Kailh_mx
- S11: value 5124 -> symbol_template; footprint KD_Switch:SWITCH_BUTTON_Kailh_mx -> KD_Switch:RotaryEncoder_Bourns_Vertical_PEC11R-4x15f-Sxxxx
- S12, S13: value 5124 -> Button_tactile_45x38_430181038816; footprint KD_Switch:SWITCH_BUTTON_Kailh_mx -> KD_Switch:SW_Push_1P1T_NO_Wurth_430181038816
- TP3, TP4: value TestPoint_1.5mm_Round -> TestPoint_2.5mm_Round; footprint KD_Connector_Pads:TestPoint_Pad_D1.5mm -> KD_Connector_Pads:TestPoint_Pad_D2.5mm
- TP5: value TP D2.5 mm H0.9mm -> TestPoint_2.5mm_Round; footprint KD_Connector_Pads:TestPoint_Pad_D2.5mm_H0.9mm -> KD_Connector_Pads:TestPoint_Pad_D2.5mm
- TP9: value TP D2.5 mm H0.9mm -> TestPoint_1.5mm_Round; footprint KD_Connector_Pads:TestPoint_Pad_D2.5mm_H0.9mm -> KD_Connector_Pads:TestPoint_Pad_D1.5mm
- U1: value MCP1825T-3302E/DC -> SN74HCS365PWR; footprint KD_Package_TO_SOT_SMD:SOT127P700X180-6N -> KD_Package_SO:SOP65P600X150-16N
- U2: value CAT811TTBI-GT3 -> SN74HCS365PWR; footprint KD_Package_TO_SOT_SMD:SOT-143_TO-253_M -> KD_Package_SO:SOP65P600X150-16N
- U3: value RP2040 -> SN74HCS365PWR; footprint Package_DFN_QFN:QFN-56-1EP_7x7mm_P0.4mm_EP3.2x3.2mm -> KD_Package_SO:SOP65P600X150-16N
- U5: value SN74HCS365PWR -> RP2040; footprint KD_Package_SO:SOP65P600X150-16N -> Package_DFN_QFN:QFN-56-1EP_7x7mm_P0.4mm_EP3.2x3.2mm
- moved H1 189.3 mm to (241.1, 99.6)
- moved FD3 171.2 mm to (224.9, 103.1)
- moved FD2 170.7 mm to (222.4, 105.6)
- moved FD6 169.5 mm to (227.5, 105.6)
- moved FD4 169.5 mm to (224.9, 105.6)
- moved FD5 167.4 mm to (227.5, 103.1)
- moved FD1 166.1 mm to (222.4, 103.1)
- moved D6 87.7 mm to (235.5, 141.5), turned to -90 degrees
- moved D3 87.4 mm to (245.4, 125.0), turned to -90 degrees
- moved D5 82.8 mm to (232.9, 141.5), turned to -90 degrees
- moved TP4 65.3 mm to (233.6, 124.2), turned to -90 degrees
- moved FB3 64.7 mm to (238.5, 137.0), turned to -90 degrees
- moved TP3 64.3 mm to (233.6, 120.1), turned to -90 degrees
- moved S12 64.3 mm to (244.1, 75.1), turned to 0 degrees
- moved FB2 61.7 mm to (235.7, 137.0), turned to -90 degrees
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Connections:
- C1 pad 1: /Main/Power Supply/PWR_IN -> /Main/Neopixel LEDs/NEOPIXEL_VDD
- C10 pad 1: +3V3 -> Net-(U2-I1)
- C11 pad 1: +3V3 -> Net-(U2-I2)
- C12 pad 1: Net-(C12-Pad1) -> Net-(U2-I3)
- C13 pad 1: Net-(U3-ADC_AVDD) -> Net-(U2-I4)
- C14 pad 1: Net-(U3-ADC_AVDD) -> +3.3V
- C15 pad 1: Net-(U3-ADC_AVDD) -> +3.3V
- C16 pad 1: Net-(U3-ADC_AVDD) -> GND
- C16 pad 2: GND -> Net-(U3-I2)
- C17 pad 1: Net-(U3-ADC_AVDD) -> GND
- C17 pad 2: GND -> Net-(U3-I3)
- C18 pad 1: Net-(U3-ADC_AVDD) -> GND
- C18 pad 2: GND -> Net-(U3-I1)
- C19 pad 1: +3.3V -> +3V3
- C2 pad 1: +3V3 -> /Main/Neopixel LEDs/NEOPIXEL_VDD
- C20 pad 1: /Main/Microcontroller/1V2 -> +3V3
- C21 pad 1: /Main/Microcontroller/1V2 -> +3V3
- C22 pad 1: /Main/Microcontroller/1V2 -> +3V3
- C23 pad 1: +3V3 -> /Main/Microcontroller/1V2
- C24 pad 1: +3V3 -> /Main/Microcontroller/1V2
- C25 pad 1: Net-(U5-I1) -> Net-(U5-ADC_AVDD)
- C26 pad 1: Net-(U5-I2) -> /Main/Microcontroller/1V2
- C27 pad 1: Net-(U5-I3) -> Net-(U5-XIN)
- C28 pad 1: Net-(U5-I4) -> Net-(U5-ADC_AVDD)
- C29 pad 1: Net-(U5-I5) -> Net-(U5-ADC_AVDD)
- C3 pad 1: +3V3 -> /Main/Neopixel LEDs/NEOPIXEL_VDD
- C30 pad 1: Net-(U5-I6) -> Net-(C30-Pad1)
- C31 pad 1: +3.3V -> Net-(U5-ADC_AVDD)
- C4 pad 1: /Main/Power Supply/PWR_IN -> Net-(U1-I1)
- C5 pad 1: /Main/Power Supply/PWR_IN -> Net-(U1-I2)
- C6 pad 1: /Main/Power Supply/PWR_IN -> Net-(U1-I3)
- C7 pad 1: Net-(U3-XIN) -> Net-(U1-I4)
- C8 pad 1: Net-(U3-ADC_AVDD) -> Net-(U1-I5)
- C9 pad 1: Net-(U3-ADC_AVDD) -> Net-(U1-I6)
- D1 pad 1: Net-(D1-K) -> /Main/USB Connector/USB_D_N
- D1 pad 2: Net-(D1-A) -> GND
- D2 pad 1: GND -> Net-(D2-K)
- D2 pad 2: Net-(D2-A) -> Net-(D1-V+)
- D3 pad 1: /Main/USB Connector/USB_D_N -> Net-(D3-K)
- D3 pad 2: GND -> /Main/Memory/~{CS}_MEMORY
- D5 pad 2: /Main/Memory/~{CS}_MEMORY -> Net-(D5-A)
- D6 pad 1: Net-(D6-K) -> GND
- D6 pad 2: Net-(D3-V+) -> Net-(D6-A)
- FB1 pad 1: Net-(U1-VO) -> Net-(D2-K)
- FB1 pad 2: +3V3 -> /Main/Neopixel LEDs/NEOPIXEL_VDD
- FB2 pad 1: Net-(D6-K) -> +3V3
- FB2 pad 2: /Main/Power Supply/PWR_IN -> Net-(U5-ADC_AVDD)
- FB3 pad 1: +3V3 -> Net-(U6-VO)
- FB3 pad 2: Net-(U3-ADC_AVDD) -> +3V3
- J1 pad A4: Net-(D3-V+) -> Net-(D1-V+)
- J1 pad A9: Net-(D3-V+) -> Net-(D1-V+)
- J1 pad B4: Net-(D3-V+) -> Net-(D1-V+)
- J1 pad B9: Net-(D3-V+) -> Net-(D1-V+)
- R1 pad 1: Net-(D1-A) -> /Main/USB Connector/CC2
- R1 pad 2: +3V3 -> GND
- R10 pad 2: /Main/Microcontroller/DEBUG_LED_GREEN -> Net-(U1-I6)
- R11 pad 1: Net-(D4-RK) -> Net-(R11-Pad1)
- R11 pad 2: /Main/Microcontroller/DEBUG_LED_BLUE -> Net-(U2-I1)
- R12 pad 1: Net-(C12-Pad1) -> Net-(R12-Pad1)
- R12 pad 2: Net-(U3-XOUT) -> Net-(U2-I2)
- R13 pad 1: Net-(D5-K) -> Net-(R13-Pad1)
- R13 pad 2: /Main/Microcontroller/USBBOOT -> Net-(U2-I3)
- R14 pad 1: /Main/USB Connector/CC2 -> Net-(R14-Pad1)
- R14 pad 2: GND -> Net-(U2-I4)
- R15 pad 1: /Main/USB Connector/CC1 -> +3.3V
- R15 pad 2: GND -> Net-(R15-Pad2)
- R16 pad 1: +3V3 -> +3.3V
- R16 pad 2: /Main/Memory/~{CS}_MEMORY -> Net-(R16-Pad2)
- R17 pad 1: Net-(R17-Pad1) -> +3.3V
- R17 pad 2: Net-(U5-I1) -> Net-(R17-Pad2)
- R18 pad 1: Net-(R18-Pad1) -> Net-(R15-Pad2)
- R18 pad 2: Net-(U5-I2) -> Net-(U3-I1)
- R19 pad 1: Net-(R19-Pad1) -> Net-(R16-Pad2)
- R19 pad 2: Net-(U5-I3) -> Net-(U3-I2)
- R2 pad 1: Net-(D2-A) -> /Main/USB Connector/CC1
- R2 pad 2: PERIP_~{RESET} -> GND
- R20 pad 1: Net-(R20-Pad1) -> Net-(R17-Pad2)
- R20 pad 2: Net-(U5-I4) -> Net-(U3-I3)
- R21 pad 1: Net-(R21-Pad1) -> GND
- R21 pad 2: Net-(U5-I5) -> Net-(U3-E1)
- R22 pad 1: Net-(R22-Pad1) -> +3V3
- R22 pad 2: Net-(U5-I6) -> /Main/Memory/~{CS}_MEMORY
- R5 pad 1: /Main/Microcontroller/~{RESET} -> Net-(R5-Pad1)
- R5 pad 2: +3V3 -> Net-(U1-I1)
- R6 pad 1: +3V3 -> Net-(R6-Pad1)
- R6 pad 2: /Main/Microcontroller/SDA -> Net-(U1-I2)
- R7 pad 1: +3V3 -> Net-(R7-Pad1)
- R7 pad 2: /Main/Microcontroller/SCL -> Net-(U1-I3)
- R8 pad 1: Net-(D4-GK) -> Net-(R8-Pad1)
- R8 pad 2: Net-(R10-Pad1) -> Net-(U1-I4)
- R9 pad 1: Net-(D4-BK) -> Net-(R9-Pad1)
- R9 pad 2: /Main/Microcontroller/DEBUG_LED_RED -> Net-(U1-I5)
- S1 pad 1: unconnected-(S1-Pad1) -> +3.3V
- S1 pad 2: GND -> Net-(R5-Pad1)
- S10 pad 1: (no net) -> +3.3V
- S10 pad 2: +3.3V -> Net-(R14-Pad1)
- S12 pad 1: (no net) -> unconnected-(S12-Pad1)
- S12 pad 2: +3.3V -> GND
- S13 pad 1: (no net) -> unconnected-(S13-Pad1)
- S13 pad 2: +3.3V -> GND
- S2 pad 1: unconnected-(S2-Pad1) -> +3.3V
- S2 pad 2: GND -> Net-(R6-Pad1)
- S3 pad 1: (no net) -> +3.3V
- S3 pad 2: +3.3V -> Net-(R7-Pad1)
- S4 pad 1: (no net) -> +3.3V
- S4 pad 2: +3.3V -> Net-(R8-Pad1)
- S5 pad 1: (no net) -> +3.3V
- S5 pad 2: +3.3V -> Net-(R9-Pad1)
- S6 pad 1: (no net) -> +3.3V
- S6 pad 2: +3.3V -> Net-(R10-Pad1)
- S7 pad 1: (no net) -> +3.3V
- S7 pad 2: +3.3V -> Net-(R11-Pad1)
- S8 pad 1: (no net) -> +3.3V
- S8 pad 2: +3.3V -> Net-(R12-Pad1)
- S9 pad 1: (no net) -> +3.3V
- S9 pad 2: +3.3V -> Net-(R13-Pad1)
- TP1 pad 1: +3V3 -> Net-(U1-I1)
- TP11 pad 1: Net-(U5-I1) -> /Main/Microcontroller/SCL
- TP12 pad 1: Net-(U12-I1) -> /Main/Microcontroller/SDA
- TP13 pad 1: /Main/Buttons1/Button5 -> +3V3
- TP2 pad 1: PERIP_~{RESET} -> /Main/Buttons/Button5
- TP3 pad 1: /Main/Microcontroller/TP10 -> Net-(R15-Pad2)
- TP4 pad 1: /Main/Microcontroller/TP1 -> Net-(R17-Pad2)
- TP5 pad 1: /Main/Microcontroller/SCL -> Net-(R16-Pad2)
- TP6 pad 1: /Main/Microcontroller/SDA -> /Main/Microcontroller/1V2
- TP7 pad 1: /Main/Microcontroller/1V2 -> /Main/Microcontroller/USBBOOT
- TP8 pad 1: /Main/Microcontroller/USBBOOT -> /Main/Microcontroller/~{RESET}
- TP9 pad 1: /Main/Microcontroller/~{RESET} -> /Main/Microcontroller/TP10
- U1 pad 1: PERIP_~{RESET} -> GND
- U1 pad 2: /Main/Power Supply/PWR_IN -> Net-(U1-I1)
- U1 pad 3: GND -> /Main/Buttons/Button5
- U1 pad 4: Net-(U1-VO) -> Net-(U1-I2)
- U1 pad 5: Net-(D1-K) -> /Main/Buttons/Button4
- U1 pad 6: GND -> Net-(U1-I3)
- U2 pad 2: PERIP_~{RESET} -> Net-(U2-I1)
- U2 pad 3: +3V3 -> /Main/Buttons/Button6
- U2 pad 4: +3V3 -> Net-(U2-I2)
- U3 pad 1: Net-(U3-ADC_AVDD) -> Net-(U3-E1)
- U3 pad 10: Net-(U3-ADC_AVDD) -> unconnected-(U3-I4-Pad10)
- U3 pad 11: /Main/Buttons/Button4 -> unconnected-(U3-O5-Pad11)
- U3 pad 12: /Main/Buttons/Button5 -> unconnected-(U3-I5-Pad12)
- U3 pad 13: /Main/Microcontroller/DEBUG_LED_GREEN -> unconnected-(U3-O6-Pad13)
- U3 pad 14: /Main/Microcontroller/DEBUG_LED_RED -> unconnected-(U3-I6-Pad14)
- U3 pad 15: /Main/Microcontroller/DEBUG_LED_BLUE -> Net-(U3-E1)
- U3 pad 16: /Main/Buttons1/Button0 -> +3.3V
- U3 pad 2: /Main/Buttons/Button0 -> Net-(U3-I1)
- U3 pad 3: /Main/Buttons/Button1 -> /Main/Microcontroller/ENC_A
- U3 pad 4: /Main/Buttons/Button2 -> Net-(U3-I2)
- U3 pad 5: /Main/Microcontroller/SPI_MOSI -> /Main/Microcontroller/GPIO12
- U3 pad 6: /Main/Microcontroller/SPI_MISO -> Net-(U3-I3)
- U3 pad 7: /Main/Microcontroller/UART_RX -> /Main/Microcontroller/ENC_B
- U3 pad 8: /Main/Microcontroller/SPI_CLK -> GND
- U3 pad 9: /Main/Buttons/Button3 -> unconnected-(U3-O4-Pad9)
- U5 pad 1: GND -> Net-(U5-ADC_AVDD)
- U5 pad 10: Net-(U5-I4) -> Net-(U5-ADC_AVDD)
- U5 pad 11: /Main/Buttons1/Button1 -> /Main/Buttons/Button4
- U5 pad 12: Net-(U5-I5) -> /Main/Buttons/Button5
- U5 pad 13: /Main/Buttons1/Button0 -> unconnected-(U5-GPIO10-Pad13)
- U5 pad 14: Net-(U5-I6) -> unconnected-(U5-GPIO11-Pad14)
- U5 pad 15: GND -> unconnected-(U5-GPIO12-Pad15)
- U5 pad 16: +3.3V -> /Main/Buttons/Button6
- U5 pad 2: Net-(U5-I1) -> /Main/Buttons/Button0
- U5 pad 3: /Main/Buttons1/Button5 -> /Main/Buttons/Button1
- U5 pad 4: Net-(U5-I2) -> /Main/Buttons/Button2
- U5 pad 5: /Main/Buttons1/Button4 -> /Main/Microcontroller/SPI_MOSI
- U5 pad 6: Net-(U5-I3) -> /Main/Microcontroller/SPI_MISO
- U5 pad 7: /Main/Buttons1/Button3 -> /Main/Microcontroller/UART_RX
- U5 pad 8: GND -> /Main/Microcontroller/SPI_CLK
- U5 pad 9: /Main/Buttons1/Button2 -> /Main/Buttons/Button3
- Y1 pad 1: Net-(U3-XIN) -> Net-(U5-XIN)
- Y1 pad 3: Net-(C12-Pad1) -> Net-(C30-Pad1)
