File: PCB/Rev 02.00/000018 PGKB/000018 PGKB.kicad_pcb (KiCad board)
At the start: 2 copper layers, 112 x 73.3 mm, 132 parts, among them J1 USB Mini B, J2 BM04B-SRSS-TB, U1 SN74HCS365PWR, U2 SN74HCS365PWR, U3 SN74HCS365PWR, U4 W25Q80DVSSIG, U5 RP2040, U6 MCP1825T-3302E/DC, U7 CAT811TTBI-GT3, Y1 12 MHz

Commit message: Layout
Parts:
- removed the S11 at (181.6, 135.8)
- added C41: 10n, KD_Capacitor:CAPC1608X90N, B.Cu at (158.0, 157.6)
- added D4: Neopixel Reverse, KD_Diode:LEDM_NEO3535_REVERSE_SK6812-E, B.Cu at (120.9, 155.3)
- added H1: NPTH 3.2 M3 Clearance, KD_Mechanical_Mounting_Hole:NPTH_3.2mm_M3_clearance, F.Cu at (47.6, 108.2)
- added H2: NPTH 3.2 M3 Clearance, KD_Mechanical_Mounting_Hole:NPTH_3.2mm_M3_clearance, F.Cu at (131.2, 170.8)
- added H3: NPTH 3.2 M3 Clearance, KD_Mechanical_Mounting_Hole:NPTH_3.2mm_M3_clearance, F.Cu at (131.2, 108.2)
- added H4: NPTH 3.2 M3 Clearance, KD_Mechanical_Mounting_Hole:NPTH_3.2mm_M3_clearance, F.Cu at (47.6, 170.8)
- added H6: PTH 3.2 M3 Clearance, KD_Mechanical_Mounting_Hole:PTH_3.2mm_M3_clearance_B, F.Cu at (89.5, 128.9)
- added R28: 1k, KD_Resistor:RESC1608X55N, B.Cu at (158.0, 160.1)
- added S20: symbol_template, KD_Switch:RotaryEncoder_Bourns_Vertical_PEC11R-4x15f-Sxxxx, F.Cu at (120.9, 118.5)
- added S8: 4954, KD_Switch:SWITCH_BUTTON_Kailh_mx_socket, F.Cu at (120.9, 139.5)
- C1, C10, C11, C12, C13, C14, C15, C16, C17, C18, C19, C2, C20, C21, C22, C23, C24, C25, C26, C27, C28, C29, C3, C30, C31, C32, C33, C34, C35, C36, C37, C38, C39, C4, C40, C5, C6, C7, C8, C9, D10, D14, D7, D8, D9, FB1, FB2, FB3, FD1, FD2, FD3, FD4, FD5, FD6, J1, J2, R1, R10, R11, R12, R13, R14, R15, R16, R17, R18, R19, R2, R20, R21, R22, R23, R24, R25, R26, R27, R3, R32, R33, R4, R5, R6, R7, R8, R9, S12, S13, TP1, TP11, TP12, TP13, TP14, TP15, TP16, TP2, TP3, TP4, TP5, TP6, TP7, TP8, TP9, U1, U2, U3, U4, U5, U6, U7, Y1: moved to B.Cu
- D1: value TVS_5V5_DRTR5V0U4S-7-M -> Neopixel Reverse; footprint KD_Package_TO_SOT_SMD:SOT-363_SC-70-6 -> KD_Diode:LEDM_NEO3535_REVERSE_SK6812-E; moved to B.Cu
- D11: value Neopixel Reverse -> TVS_5V5_DRTR5V0U4S-7-M; footprint KD_Diode:LEDM_NEO3535_REVERSE_SK6812-E -> KD_Package_TO_SOT_SMD:SOT-363_SC-70-6; moved to B.Cu
- D12: value Neopixel Reverse -> Schottky_30V_1A_PMEG3010ER_115; footprint KD_Diode:LEDM_NEO3535_REVERSE_SK6812-E -> KD_Diode:DIOC360X180X150_SOD123; moved to B.Cu
- D13: value Neopixel Reverse -> Schottky_30V_200mA_DCo_BAT54WS; footprint KD_Diode:LEDM_NEO3535_REVERSE_SK6812-E -> KD_Diode:D_SOD-323; moved to B.Cu
- D15: value Neopixel Reverse -> Red; footprint KD_Diode:LEDM_NEO3535_REVERSE_SK6812-E -> KD_Diode:LEDM1608X70M; moved to B.Cu
- D16: value Neopixel Reverse -> Green; footprint KD_Diode:LEDM_NEO3535_REVERSE_SK6812-E -> KD_Diode:LEDM1608X70M; moved to B.Cu
- D2: value Schottky_30V_1A_PMEG3010ER_115 -> Neopixel Reverse; footprint KD_Diode:DIOC360X180X150_SOD123 -> KD_Diode:LEDM_NEO3535_REVERSE_SK6812-E; moved to B.Cu
- D3: value Schottky_30V_200mA_DCo_BAT54WS -> Neopixel Reverse; footprint KD_Diode:D_SOD-323 -> KD_Diode:LEDM_NEO3535_REVERSE_SK6812-E; moved to B.Cu
- D5: value Red -> Neopixel Reverse; footprint KD_Diode:LEDM1608X70M -> KD_Diode:LEDM_NEO3535_REVERSE_SK6812-E; moved to B.Cu
- D6: value Green -> Neopixel Reverse; footprint KD_Diode:LEDM1608X70M -> KD_Diode:LEDM_NEO3535_REVERSE_SK6812-E; moved to B.Cu
- H5: renamed from H1; value M2_NPTH_2.2_Minimal -> PTH 3.2 M3 Clearance; footprint KD_Mechanical_Mounting_Hole:MountingHole_2.2mm_NPTH -> KD_Mechanical_Mounting_Hole:PTH_3.2mm_M3_clearance_B
- S1: value 5124 -> 4954; footprint KD_Switch:SWITCH_BUTTON_Kailh_mx -> KD_Switch:SWITCH_BUTTON_Kailh_mx_socket
- S10: renamed from S6; value 5124 -> 4954; footprint KD_Switch:SWITCH_BUTTON_Kailh_mx -> KD_Switch:SWITCH_BUTTON_Kailh_mx_socket
- S11: renamed from S9; value 5124 -> 4954; footprint KD_Switch:SWITCH_BUTTON_Kailh_mx -> KD_Switch:SWITCH_BUTTON_Kailh_mx_socket
- S2: renamed from S4; value 5124 -> 4954; footprint KD_Switch:SWITCH_BUTTON_Kailh_mx -> KD_Switch:SWITCH_BUTTON_Kailh_mx_socket
- S3: renamed from S7; value 5124 -> 4954; footprint KD_Switch:SWITCH_BUTTON_Kailh_mx -> KD_Switch:SWITCH_BUTTON_Kailh_mx_socket
- S4: renamed from S10; value 5124 -> 4954; footprint KD_Switch:SWITCH_BUTTON_Kailh_mx -> KD_Switch:SWITCH_BUTTON_Kailh_mx_socket
- S5: renamed from S2; value 5124 -> 4954; footprint KD_Switch:SWITCH_BUTTON_Kailh_mx -> KD_Switch:SWITCH_BUTTON_Kailh_mx_socket
- S6: renamed from S5; value 5124 -> 4954; footprint KD_Switch:SWITCH_BUTTON_Kailh_mx -> KD_Switch:SWITCH_BUTTON_Kailh_mx_socket
- S7: renamed from S8; value 5124 -> 4954; footprint KD_Switch:SWITCH_BUTTON_Kailh_mx -> KD_Switch:SWITCH_BUTTON_Kailh_mx_socket
- S9: renamed from S3; value 5124 -> 4954; footprint KD_Switch:SWITCH_BUTTON_Kailh_mx -> KD_Switch:SWITCH_BUTTON_Kailh_mx_socket
- moved S12 193.2 mm to (66.1, 150.2), turned to 180 degrees
- moved D1 191.6 mm to (57.9, 155.4), turned to 0 degrees
- moved C3 189.2 mm to (56.1, 107.5), turned to 180 degrees
- moved S13 181.6 mm to (75.8, 150.2)
- moved U4 180.0 mm to (47.4, 117.4)
- moved D5 175.1 mm to (57.9, 134.4), turned to 0 degrees
- moved D2 170.7 mm to (78.9, 155.4), turned to 0 degrees
- moved Y1 165.9 mm to (69.7, 140.3), turned to 0 degrees
- moved H5 159.9 mm to (89.4, 150.2)
- moved D6 156.7 mm to (78.9, 134.5), turned to 0 degrees
- moved D3 148.7 mm to (99.9, 155.4), turned to 0 degrees
- moved U5 147.9 mm to (68.1, 129.7), turned to 180 degrees
- moved C39 146.8 mm to (100.0, 105.9), turned to 180 degrees
- moved C1 145.5 mm to (100.0, 109.1), turned to 180 degrees
- moved FB1 143.7 mm to (91.1, 114.3), turned to 90 degrees
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Connections:
- D1 pad 1: /Main/USB Connector/USB_D_N -> /Main/Neopixel LEDs/NEOPIXEL_VDD
- D1 pad 2: GND -> Net-(D1-DOUT)
- D1 pad 3: unconnected-(D1-Pad3) -> GND
- D1 pad 4: unconnected-(D1-Pad4) -> /Main/Microcontroller/NEOPIX_DRIVE
- D10 pad 2: unconnected-(D10-DOUT-Pad2) -> Net-(D10-DOUT)
- D11 pad 1: /Main/Neopixel LEDs/NEOPIXEL_VDD -> /Main/USB Connector/USB_D_N
- D11 pad 2: Net-(D11-DOUT) -> GND
- D11 pad 3: GND -> unconnected-(D11-Pad3)
- D11 pad 4: Net-(D11-DIN) -> unconnected-(D11-Pad4)
- D12 pad 1: /Main/Neopixel LEDs/NEOPIXEL_VDD -> Net-(D12-K)
- D12 pad 2: Net-(D12-DOUT) -> Net-(D11-V+)
- D13 pad 1: /Main/Neopixel LEDs/NEOPIXEL_VDD -> Net-(D13-K)
- D13 pad 2: Net-(D13-DOUT) -> /Main/Memory/~{CS}_MEMORY
- D14 pad 2: Net-(D14-DOUT) -> unconnected-(D14-DOUT-Pad2)
- D14 pad 4: Net-(D11-DOUT) -> Net-(D10-DOUT)
- D15 pad 1: /Main/Neopixel LEDs/NEOPIXEL_VDD -> Net-(D15-K)
- D15 pad 2: Net-(D15-DOUT) -> Net-(D15-A)
- D16 pad 1: /Main/Neopixel LEDs/NEOPIXEL_VDD -> GND
- D16 pad 2: Net-(D10-DIN) -> Net-(D16-A)
- D2 pad 1: Net-(D2-K) -> /Main/Neopixel LEDs/NEOPIXEL_VDD
- D2 pad 2: Net-(D1-V+) -> Net-(D2-DOUT)
- D3 pad 1: Net-(D3-K) -> /Main/Neopixel LEDs/NEOPIXEL_VDD
- D3 pad 2: /Main/Memory/~{CS}_MEMORY -> Net-(D3-DOUT)
- D5 pad 1: Net-(D5-K) -> /Main/Neopixel LEDs/NEOPIXEL_VDD
- D5 pad 2: Net-(D5-A) -> Net-(D5-DOUT)
- D6 pad 1: GND -> /Main/Neopixel LEDs/NEOPIXEL_VDD
- D6 pad 2: Net-(D6-A) -> Net-(D6-DOUT)
- D7 pad 2: Net-(D11-DIN) -> Net-(D7-DOUT)
- D7 pad 4: /Main/Microcontroller/NEOPIX_DRIVE -> Net-(D6-DOUT)
- D8 pad 2: Net-(D12-DIN) -> Net-(D8-DOUT)
- D8 pad 4: Net-(D14-DOUT) -> Net-(D7-DOUT)
- D9 pad 2: Net-(D13-DIN) -> Net-(D10-DIN)
- D9 pad 4: Net-(D15-DOUT) -> Net-(D8-DOUT)
- FB1 pad 1: Net-(D2-K) -> Net-(D12-K)
- J1 pad A4: Net-(D1-V+) -> Net-(D11-V+)
- J1 pad A9: Net-(D1-V+) -> Net-(D11-V+)
- J1 pad B4: Net-(D1-V+) -> Net-(D11-V+)
- J1 pad B9: Net-(D1-V+) -> Net-(D11-V+)
- R23 pad 1: Net-(D3-K) -> Net-(D13-K)
- R32 pad 1: Net-(D5-A) -> Net-(D15-A)
- R33 pad 1: Net-(D6-A) -> Net-(D16-A)
- S10 pad 2: Net-(R10-Pad1) -> Net-(R14-Pad1)
- S11 pad 2: Net-(R13-Pad1) -> Net-(R28-Pad1)
- S2 pad 2: Net-(R8-Pad1) -> Net-(R6-Pad1)
- S3 pad 2: Net-(R11-Pad1) -> Net-(R7-Pad1)
- S4 pad 2: Net-(R14-Pad1) -> Net-(R8-Pad1)
- S5 pad 2: Net-(R6-Pad1) -> Net-(R9-Pad1)
- S6 pad 2: Net-(R9-Pad1) -> Net-(R10-Pad1)
- S7 pad 2: Net-(R12-Pad1) -> Net-(R11-Pad1)
- S9 pad 2: Net-(R7-Pad1) -> Net-(R13-Pad1)
- TP2 pad 1: /Main/Buttons/Button5 -> /Main/Buttons/Button1
- U1 pad 11: /Main/Buttons/Button1 -> /Main/Buttons/Button5
- U1 pad 13: /Main/Buttons/Button0 -> /Main/Buttons/Button6
- U1 pad 3: /Main/Buttons/Button5 -> /Main/Buttons/Button1
- U1 pad 5: /Main/Buttons/Button4 -> /Main/Buttons/Button2
- U1 pad 9: /Main/Buttons/Button2 -> /Main/Buttons/Button4
- U2 pad 11: unconnected-(U2-O5-Pad11) -> /Main/Buttons/Button11
- U2 pad 12: GND -> Net-(U2-I5)
- U2 pad 3: /Main/Buttons/Button6 -> /Main/Buttons/Button7
- U2 pad 5: /Main/Buttons/Button7 -> /Main/Buttons/Button8
- U2 pad 7: /Main/Buttons/Button8 -> /Main/Buttons/Button9
- U2 pad 9: /Main/Buttons/Button9 -> /Main/Buttons/Button10
- U5 pad 2: /Main/Buttons/Button0 -> /Main/Microcontroller/GPIO0
- U6 pad 5: Net-(D5-K) -> Net-(D15-K)
Other:
- board size 112 x 73.3 mm -> 91.5 x 70.5 mm

Commit message: step
Parts:
- R26, R27: value R_0805_4700_5% -> 4k7; footprint KD_Resistor:RESC2012X50N -> KD_Resistor:RESC1005X40N
- moved C20 169.6 mm to (46.6, 125.2), turned to 0 degrees
- moved C19 169.3 mm to (46.4, 123.4), turned to 0 degrees
- moved C4 154.0 mm to (67.7, 167.5), turned to 0 degrees
- moved C33 153.9 mm to (61.8, 126.1), turned to 180 degrees
- moved C12 149.9 mm to (63.4, 116.2), turned to 180 degrees
- moved C8 148.1 mm to (58.5, 149.0)
- moved C24 146.8 mm to (64.4, 136.9)
- moved C28 146.6 mm to (57.3, 129.7), turned to 90 degrees
- moved C34 145.5 mm to (67.9, 120.9)
- moved R26 142.3 mm to (68.4, 117.8), turned to 0 degrees
- moved R27 139.9 mm to (68.4, 115.4), turned to 0 degrees
- moved C23 139.9 mm to (71.2, 120.1), turned to 90 degrees
- moved C26 138.8 mm to (69.4, 120.9), turned to 90 degrees
- moved C29 137.8 mm to (65.9, 136.9)
- moved C32 136.3 mm to (61.8, 124.6), turned to 180 degrees
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Routing:
- net Net-(U5-ADC_AVDD): track 0.00 -> 4.73 mm

Commit message: Update 000018 PGKB.kicad_pcb
Parts:
- moved R9 104.0 mm to (60.0, 148.9), turned to 90 degrees
- moved R13 84.9 mm to (65.6, 117.8), turned to 90 degrees
- moved R24 83.0 mm to (71.1, 150.2)
- moved R25 79.1 mm to (69.6, 136.8)
- moved R10 71.9 mm to (89.0, 142.1), turned to 90 degrees
- moved R7 67.1 mm to (110.1, 159.7), turned to 180 degrees
- moved R14 61.3 mm to (86.7, 117.8), turned to 90 degrees
- moved R8 50.2 mm to (131.4, 160.8), turned to 180 degrees
- moved R11 50.1 mm to (108.4, 139.1), turned to 0 degrees
- moved R16 49.2 mm to (117.4, 107.3), turned to 0 degrees
- moved R15 46.3 mm to (119.3, 130.1), turned to 0 degrees
- moved R17 44.4 mm to (116.2, 130.0), turned to 180 degrees
- moved R19 41.3 mm to (117.5, 109.5), turned to 180 degrees
- moved R18 38.7 mm to (119.3, 128.4), turned to 180 degrees
- moved R12 32.5 mm to (130.9, 145.7), turned to 180 degrees

Commit message: pcb
Parts:
- moved H1 2.12 mm to (46.1, 106.8)
- moved H2 2.12 mm to (132.7, 172.2)
- moved H3 2.12 mm to (132.7, 106.8)
- moved H4 2.12 mm to (46.1, 172.2)
- moved J1 0.80 mm to (86.4, 109.2)
- moved S4 0.20 mm to (120.9, 160.5)
Other:
- board size 91.5 x 70.5 mm -> 93.5 x 72.5 mm
Changed lines of the file:
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@@
   )
   (footprint "KD_Mechanical_Mounting_Hole:NPTH_3.2mm_M3_clearance" (layer "F.Cu")
-    (at 47.65 108.25)
+    (at 46.15 106.75)
     (tags "NPTH M3")
     (property "DNP" "T")
@@
   )
   (footprint "KD_Switch:SWITCH_BUTTON_Kailh_mx_socket" (layer "F.Cu")
-    (at 120.9 160.3 -90)
+    (at 120.9 160.5 -90)
     (tags "Keyboard button")
     (property "DNP" "F")
@@
         (effects (font (size 0.8 0.8) (thickness 0.15)) (justify bottom))
     )
-    (fp_text value "4954" (at 0 0 -180) (layer "F.Fab") hide
+    (fp_text value "4954" (at 0 0) (layer "F.Fab") hide
         (effects (font (size 0.8 0.8) (thickness 0.15)))
     )
-    (fp_text user "${REFERENCE}" (at 0 0 -90) (layer "F.Fab")
+    (fp_text user "${REFERENCE}" (at 0 0 90) (layer "F.Fab")
         (effects (font (size 0.44 0.44) (thickness 0.06)))
     )
@@
   )
   (footprint "KD_Mechanical_Mounting_Hole:NPTH_3.2mm_M3_clearance" (layer "F.Cu")
-    (at 47.65 170.75)
+    (at 46.15 172.25)
     (tags "NPTH M3")
     (property "DNP" "T")
@@
   )
   (footprint "KD_Mechanical_Mounting_Hole:NPTH_3.2mm_M3_clearance" (layer "F.Cu")
-    (at 131.15 108.25)
+    (at 132.65 106.75)
     (tags "NPTH M3")
     (property "DNP" "T")
@@
   )
   (footprint "KD_Mechanical_Mounting_Hole:NPTH_3.2mm_M3_clearance" (layer "F.Cu")
-    (at 131.15 170.75)
+    (at 132.65 172.25)
     (tags "NPTH M3")
     (property "DNP" "T")
@@
       (stroke (width 0.15) (type default)) (layer "B.SilkS"))
     (fp_rect (start -1.8 1.6) (end 1.8 -1.6)
-      (stroke (width 0.12) (type default)) (fill none) (layer "Eco2.User"))
+      (stroke (width 0.12) (type default)) (fill none) (layer "Edge.Cuts"))
     (fp_rect (start -3.3 -0.4) (end -1.6 -1.1)
       (stroke (width 0.1) (type solid)) (fill solid) (layer "B.Fab"))
@@
       (stroke (width 0.15) (type default)) (layer "B.SilkS"))
     (fp_rect (start -1.8 1.6) (end 1.8 -1.6)
-      (stroke (width 0.12) (type default)) (fill none) (layer "Eco2.User"))
+      (stroke (width 0.12) (type default)) (fill none) (layer "Edge.Cuts"))
     (fp_rect (start -3.3 -0.4) (end -1.6 -1.1)
       (stroke (width 0.1) (type solid)) (fill solid) (layer "B.Fab"))
@@
       (stroke (width 0.15) (type default)) (layer "B.SilkS"))
     (fp_rect (start -1.8 1.6) (end 1.8 -1.6)
-      (stroke (width 0.12) (type default)) (fill none) (layer "Eco2.User"))
+      (stroke (width 0.12) (type default)) (fill none) (layer "Edge.Cuts"))
     (fp_rect (start -3.3 -0.4) (end -1.6 -1.1)
       (stroke (width 0.1) (type solid)) (fill solid) (layer "B.Fab"))
@@
   )
   (footprint "KD_Connector_USB_HDMI_Etc:USB_C_Receptacle_GCT_USB4085" (layer "B.Cu")
-    (at 86.405 110)
+    (at 86.405 109.2)
     (descr "USB 2.0 Type C Receptacle, https://gct.co/Files/Drawings/USB4085.pdf")
     (tags "USB Type-C Receptacle Through-hole Right angle")
@@
       (stroke (width 0.15) (type default)) (layer "B.SilkS"))
     (fp_rect (start -1.8 1.6) (end 1.8 -1.6)
-      (stroke (width 0.12) (type default)) (fill none) (layer "Eco2.User"))
+      (stroke (width 0.12) (type default)) (fill none) (layer "Edge.Cuts"))
     (fp_rect (start -3.3 -0.4) (end -1.6 -1.1)
       (stroke (width 0.1) (type solid)) (fill solid) (layer "B.Fab"))
@@
       (stroke (width 0.15) (type default)) (layer "B.SilkS"))
     (fp_rect (start -1.8 1.6) (end 1.8 -1.6)
-      (stroke (width 0.12) (type default)) (fill none) (layer "Eco2.User"))
+      (stroke (width 0.12) (type default)) (fill none) (layer "Edge.Cuts"))
     (fp_rect (start -3.3 -0.4) (end -1.6 -1.1)
       (stroke (width 0.1) (type solid)) (fill solid) (layer "B.Fab"))
@@
       (stroke (width 0.15) (type default)) (layer "B.SilkS"))
     (fp_rect (start -1.8 1.6) (end 1.8 -1.6)
-      (stroke (width 0.12) (type default)) (fill none) (layer "Eco2.User"))
+      (stroke (width 0.12) (type default)) (fill none) (layer "Edge.Cuts"))
     (fp_rect (start -3.3 -0.4) (end -1.6 -1.1)
       (stroke (width 0.1) (type solid)) (fill solid) (layer "B.Fab"))
@@
       (stroke (width 0.15) (type default)) (layer "B.SilkS"))
     (fp_rect (start -1.8 1.6) (end 1.8 -1.6)
-      (stroke (width 0.12) (type default)) (fill none) (layer "Eco2.User"))
+      (stroke (width 0.12) (type default)) (fill none) (layer "Edge.Cuts"))
     (fp_rect (start -3.3 -0.4) (end -1.6 -1.1)
       (stroke (width 0.1) (type solid)) (fill solid) (layer "B.Fab"))
@@
       (stroke (width 0.15) (type default)) (layer "B.SilkS"))
     (fp_rect (start -1.8 1.6) (end 1.8 -1.6)
-      (stroke (width 0.12) (type default)) (fill none) (layer "Eco2.User"))
+      (stroke (width 0.12) (type default)) (fill none) (layer "Edge.Cuts"))
     (fp_rect (start -3.3 -0.4) (end -1.6 -1.1)
       (stroke (width 0.1) (type solid)) (fill solid) (layer "B.Fab"))
@@
       (stroke (width 0.15) (type default)) (layer "B.SilkS"))
     (fp_rect (start -1.8 1.6) (end 1.8 -1.6)
-      (stroke (width 0.12) (type default)) (fill none) (layer "Eco2.User"))
+      (stroke (width 0.12) (type default)) (fill none) (layer "Edge.Cuts"))
     (fp_rect (start -3.3 -0.4) (end -1.6 -1.1)
       (stroke (width 0.1) (type solid)) (fill solid) (layer "B.Fab"))
@@
       (stroke (width 0.15) (type default)) (layer "B.SilkS"))
     (fp_rect (start -1.8 1.6) (end 1.8 -1.6)
-      (stroke (width 0.12) (type default)) (fill none) (layer "Eco2.User"))
+      (stroke (width 0.12) (type default)) (fill none) (layer "Edge.Cuts"))
     (fp_rect (start -3.3 -0.4) (end -1.6 -1.1)
       (stroke (width 0.1) (type solid)) (fill solid) (layer "B.Fab"))
@@
       (stroke (width 0.15) (type default)) (layer "B.SilkS"))
     (fp_rect (start -1.8 1.6) (end 1.8 -1.6)
-      (stroke (width 0.12) (type default)) (fill none) (layer "Eco2.User"))
+      (stroke (width 0.12) (type default)) (fill none) (layer "Edge.Cuts"))
     (fp_rect (start -3.3 -0.4) (end -1.6 -1.1)
       (stroke (width 0.1) (type solid)) (fill solid) (layer "B.Fab"))
@@
   (gr_circle (center 99.9 139.5) (end 101.395 139.5)
     (stroke (width 0.05) (type solid)) (fill none) (layer "Cmts.User"))
-  (gr_line (start 134.15 104.25) (end 44.65 104.25)
+  (gr_line (start 43.65 175.75) (end 135.15 175.75)
     (stroke (width 0.05) (type solid)) (layer "Edge.Cuts"))
-  (gr_arc (start 43.65 105.25) (mid 43.942893 104.542894) (end 44.65 104.25)
+  (gr_arc (start 135.15 103.25) (mid 135.857108 103.542893) (end 136.15 104.25)
     (stroke (width 0.05) (type solid)) (layer "Edge.Cuts"))
-  (gr_line (start 44.65 174.75) (end 134.15 174.75)
+  (gr_line (start 135.15 103.25) (end 43.65 103.25)
     (stroke (width 0.05) (type solid)) (layer "Edge.Cuts"))
-  (gr_arc (start 135.15 173.75) (mid 134.857107 174.457106) (end 134.15 174.75)
+  (gr_line (start 42.65 104.25) (end 42.65 174.75)
     (stroke (width 0.05) (type solid)) (layer "Edge.Cuts"))
-  (gr_line (start 135.15 173.75) (end 135.15 105.25)
+  (gr_line (start 136.15 174.75) (end 136.15 104.25)
     (stroke (width 0.05) (type solid)) (layer "Edge.Cuts"))
-  (gr_line (start 43.65 105.25) (end 43.65 173.75)
+  (gr_arc (start 42.65 104.25) (mid 42.942893 103.542893) (end 43.65 103.25)
     (stroke (width 0.05) (type solid)) (layer "Edge.Cuts"))
-  (gr_arc (start 134.15 104.25) (mid 134.857106 104.542893) (end 135.15 105.25)
+  (gr_arc (start 43.65 175.75) (mid 42.942893 175.457107) (end 42.65 174.75)
     (stroke (width 0.05) (type solid)) (layer "Edge.Cuts"))
-  (gr_arc (start 44.65 174.75) (mid 43.942894 174.457107) (end 43.65 173.75)
+  (gr_arc (start 136.15 174.75) (mid 135.857107 175.457106) (end 135.15 175.75)
     (stroke (width 0.05) (type solid)) (layer "Edge.Cuts"))
   (gr_line (start 4.2 10.2) (end 62.2 10.2)

Commit message: sitte vaan routaus
Parts:
- removed C3: 4u7, KD_Capacitor:CAPAE400x540N
- FD1, FD3, FD5, TP9: moved to F.Cu
- TP3, TP4, TP5: value TestPoint_2.5mm_Round -> TP D2.5 mm H0.9mm; footprint KD_Connector_Pads:TestPoint_Pad_D2.5mm -> KD_Connector_Pads:TestPoint_Pad_D2.5mm_H0.9mm
- moved FD1 143.4 mm to (44.3, 165.6), turned to 0 degrees
- moved TP1 140.3 mm to (65.0, 170.2)
- moved FD6 138.4 mm to (44.3, 167.5)
- moved FD2 135.4 mm to (50.7, 106.5)
- moved TP6 131.2 mm to (61.2, 137.4)
- moved TP16 131.0 mm to (57.8, 106.0)
- moved FD5 130.3 mm to (50.7, 104.7), turned to 0 degrees
- moved TP7 128.1 mm to (69.1, 161.3)
- moved TP12 126.9 mm to (66.6, 107.6)
- moved TP15 126.6 mm to (64.2, 157.0)
- moved TP11 122.1 mm to (70.6, 107.8)
- moved TP8 117.7 mm to (75.8, 150.2)
- moved TP2 113.9 mm to (82.1, 137.4)
- moved C22 96.7 mm to (66.2, 115.5), turned to 180 degrees
- moved TP9 96.2 mm to (55.6, 130.7), turned to 90 degrees
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Connections:
- C10 pad 1: Net-(U2-I1) -> Net-(U2-I5)
- C11 pad 1: Net-(U2-I2) -> Net-(U2-I6)
- C12 pad 1: Net-(U2-I3) -> Net-(U1-I1)
- C13 pad 1: Net-(U2-I4) -> Net-(U1-I2)
- C4 pad 1: Net-(U1-I1) -> Net-(U2-I1)
- C41 pad 1: Net-(U2-I5) -> Net-(U1-I3)
- C5 pad 1: Net-(U1-I2) -> Net-(U2-I2)
- C6 pad 1: Net-(U1-I3) -> Net-(U2-I3)
- C7 pad 1: Net-(U1-I4) -> Net-(U2-I4)
- C8 pad 1: Net-(U1-I5) -> Net-(U1-I4)
- C9 pad 1: Net-(U1-I6) -> Net-(U1-I5)
- R10 pad 2: Net-(U1-I6) -> Net-(U1-I5)
- R11 pad 2: Net-(U2-I1) -> Net-(U2-I5)
- R12 pad 2: Net-(U2-I2) -> Net-(U2-I6)
- R13 pad 2: Net-(U2-I3) -> Net-(U1-I1)
- R14 pad 2: Net-(U2-I4) -> Net-(U1-I2)
- R28 pad 2: Net-(U2-I5) -> Net-(U1-I3)
- R5 pad 2: Net-(U1-I1) -> Net-(U2-I1)
- R6 pad 2: Net-(U1-I2) -> Net-(U2-I2)
- R7 pad 2: Net-(U1-I3) -> Net-(U2-I3)
- R8 pad 2: Net-(U1-I4) -> Net-(U2-I4)
- R9 pad 2: Net-(U1-I5) -> Net-(U1-I4)
- TP1 pad 1: Net-(U1-I1) -> Net-(U2-I1)
- U1 pad 11: /Main/Buttons/Button5 -> /Main/Buttons/Button6
- U1 pad 13: /Main/Buttons/Button6 -> unconnected-(U1-O6-Pad13)
- U1 pad 14: Net-(U1-I6) -> GND
- U1 pad 3: /Main/Buttons/Button1 -> /Main/Buttons/Button9
- U1 pad 5: /Main/Buttons/Button2 -> /Main/Buttons/Button10
- U1 pad 7: /Main/Buttons/Button3 -> /Main/Buttons/Button11
- U1 pad 9: /Main/Buttons/Button4 -> /Main/Buttons/Button5
- U2 pad 11: /Main/Buttons/Button11 -> /Main/Buttons/Button7
- U2 pad 13: unconnected-(U2-O6-Pad13) -> /Main/Buttons/Button8
- U2 pad 14: GND -> Net-(U2-I6)
- U2 pad 3: /Main/Buttons/Button7 -> /Main/Buttons/Button1
- U2 pad 5: /Main/Buttons/Button8 -> /Main/Buttons/Button2
- U2 pad 7: /Main/Buttons/Button9 -> /Main/Buttons/Button3
- U2 pad 9: /Main/Buttons/Button10 -> /Main/Buttons/Button4
Other:
- board text added: "PB"
- board text added: "PG"
