File: PCB/Rev 02.00/000018 PGKB/LEDS_Neopixel.kicad_sch (KiCad schematic)
At the start: 10 parts

Commit message: updates
Parts:
- added C2: 100n, KD_Capacitor:CAPC1608X90N, symbol KD_Capacitor:C_0603_100n_X7R_50V
- added C4: 1u, KD_Capacitor:CAPC2012X135N, symbol KD_Capacitor:C_0805_1u_X7R_25V
- added TP2 (x2): TP D2.5 mm H0.9mm, KD_Connector_Pads:TestPoint_Pad_D2.5mm_H0.9mm, symbol KD_Connector_Pads:TestPoint_2.5mm_H0.9
- D10: renamed from D16; footprint KD_Inductor:L_TDK_VLS201610CX-1 -> KD_Diode:LEDM_NEO3535_REVERSE_SK6812-E
- D11: renamed from D8; footprint KD_Inductor:L_TDK_VLS201610CX-1 -> KD_Diode:LEDM_NEO3535_REVERSE_SK6812-E
- D12: renamed from D11; footprint KD_Inductor:L_TDK_VLS201610CX-1 -> KD_Diode:LEDM_NEO3535_REVERSE_SK6812-E
- D13: renamed from D14; footprint KD_Inductor:L_TDK_VLS201610CX-1 -> KD_Diode:LEDM_NEO3535_REVERSE_SK6812-E
- D14: renamed from D9; footprint KD_Inductor:L_TDK_VLS201610CX-1 -> KD_Diode:LEDM_NEO3535_REVERSE_SK6812-E
- D15: renamed from D12; footprint KD_Inductor:L_TDK_VLS201610CX-1 -> KD_Diode:LEDM_NEO3535_REVERSE_SK6812-E
- D16: renamed from D15; footprint KD_Inductor:L_TDK_VLS201610CX-1 -> KD_Diode:LEDM_NEO3535_REVERSE_SK6812-E
- D7: footprint KD_Inductor:L_TDK_VLS201610CX-1 -> KD_Diode:LEDM_NEO3535_REVERSE_SK6812-E
- D8: renamed from D10; footprint KD_Inductor:L_TDK_VLS201610CX-1 -> KD_Diode:LEDM_NEO3535_REVERSE_SK6812-E
- D9: renamed from D13; footprint KD_Inductor:L_TDK_VLS201610CX-1 -> KD_Diode:LEDM_NEO3535_REVERSE_SK6812-E
Connections:
- net GND: now also C2.2, C4.2
- net NEOPIXEL_VDD: now also D10.1 (VDD), D12.1 (VDD), D13.1 (VDD), D15.1 (VDD), D16.1 (VDD), D8.1 (VDD), D9.1 (VDD), C2.1, C4.1, TP2.1
- net at D10.4 (DIN), D16.2 (DOUT): now also TP2.1
Other:
- moved on the sheet: D10, D11, D12, D13, D14, D15, D16, D7, D8, D9

Commit message: Layout
Parts:
- added D14: Neopixel Reverse, KD_Diode:LEDM_NEO3535_REVERSE_SK6812-E, symbol KD_Led:Neopixel_Reverse_Adafruit_4960
- renumbered D7 to D1, D11 to D2, D14 to D3, D8 to D4, D12 to D5, D15 to D6, D9 to D7, D13 to D8, D16 to D9
Connections:
- net GND: now also D14.3 (VSS)
- net NEOPIXEL_VDD: now also D14.1 (VDD)
- net at D10.2 (DOUT): now also D14.4 (DIN)

Commit message: error fixing
Parts:
- D1, D10, D14, D2, D3, D4, D5, D6, D7, D8, D9: Price 2.8 -> 0.28
Other:
- company: (none) -> Kallio Designs Oy
- title: (none) -> Programmable Keyboard
Changed lines of the file:
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@@
 (kicad_sch (version 20230121) (generator eeschema)
   (paper "A4")
+  (title_block
+    (title "Programmable Keyboard")
+    (date "2023-10-19")
+    (rev "1.0")
+    (company "Kallio Designs Oy")
+    (comment 1 "TL, NH")
+    (comment 3 "PCB_PN")
+  )
   (junction (at 127 171.45) (diameter 0) (color 0 0 0 0)
   )
@@
       (effects (font (size 1.27 1.27)) (justify left) hide)
     )
-    (property "Price" "2.8" (at 114.3 57.15 0)
+    (property "Price" "0.28" (at 114.3 57.15 0)
       (effects (font (size 1.27 1.27)) (justify left) hide)
     )
@@
       (effects (font (size 1.27 1.27)) (justify left) hide)
     )
-    (property "Price" "2.8" (at 190.5 95.25 0)
+    (property "Price" "0.28" (at 190.5 95.25 0)
       (effects (font (size 1.27 1.27)) (justify left) hide)
     )
@@
       (effects (font (size 1.27 1.27)) (justify left) hide)
     )
-    (property "Price" "2.8" (at 152.4 57.15 0)
+    (property "Price" "0.28" (at 152.4 57.15 0)
       (effects (font (size 1.27 1.27)) (justify left) hide)
     )
@@
       (effects (font (size 1.27 1.27)) (justify left) hide)
     )
-    (property "Price" "2.8" (at 114.3 95.25 0)
+    (property "Price" "0.28" (at 114.3 95.25 0)
       (effects (font (size 1.27 1.27)) (justify left) hide)
     )
@@
       (effects (font (size 1.27 1.27)) (justify left) hide)
     )
-    (property "Price" "2.8" (at 114.3 133.35 0)
+    (property "Price" "0.28" (at 114.3 133.35 0)
       (effects (font (size 1.27 1.27)) (justify left) hide)
     )
@@
       (effects (font (size 1.27 1.27)) (justify left) hide)
     )
-    (property "Price" "2.8" (at 190.5 19.05 0)
+    (property "Price" "0.28" (at 190.5 19.05 0)
       (effects (font (size 1.27 1.27)) (justify left) hide)
     )
@@
       (effects (font (size 1.27 1.27)) (justify left) hide)
     )
-    (property "Price" "2.8" (at 152.4 133.35 0)
+    (property "Price" "0.28" (at 152.4 133.35 0)
       (effects (font (size 1.27 1.27)) (justify left) hide)
     )
@@
       (effects (font (size 1.27 1.27)) (justify left) hide)
     )
-    (property "Price" "2.8" (at 114.3 19.05 0)
+    (property "Price" "0.28" (at 114.3 19.05 0)
       (effects (font (size 1.27 1.27)) (justify left) hide)
     )
@@
       (effects (font (size 1.27 1.27)) (justify left) hide)
     )
-    (property "Price" "2.8" (at 190.5 57.15 0)
+    (property "Price" "0.28" (at 190.5 57.15 0)
       (effects (font (size 1.27 1.27)) (justify left) hide)
     )
@@
       (effects (font (size 1.27 1.27)) (justify left) hide)
     )
-    (property "Price" "2.8" (at 152.4 19.05 0)
+    (property "Price" "0.28" (at 152.4 19.05 0)
       (effects (font (size 1.27 1.27)) (justify left) hide)
     )
@@
       (effects (font (size 1.27 1.27)) (justify left) hide)
     )
-    (property "Price" "2.8" (at 152.4 95.25 0)
-      (effects (font (size 1.27 1.27)) (justify left) hide)
-    )
+    (property "Price" "0.28" (at 152.4 95.25 0)
+      (effects (font (size 1.27 1.27)) (justify left) hide)
+    )
