File: PCB/Rev 02.00/000018 PGKB/Memory.kicad_sch (KiCad schematic)
At the start: 3 parts

Commit message: Schematic
Parts:
- added U4: W25Q80DVSSIG, KD_Package_SO:SOIC127P790X195-8N, symbol KD_IC_Memory:FLASH_8MBit_104MHz_W25Q80DVSSIG
Connections:
- net +3V3: now also U4.8 (VCC)
- net CLK: now also U4.6 (CLK)
- net DATA0: now also U4.5 (DI(IO0))
- net DATA1: now also U4.2 (DO(IO1))
- net DATA2: now also U4.3 (~{WP}(IO2))
- net DATA3: now also U4.7 (~{HOLD}(IO3))
- net GND: now also U4.4 (GND)
- net ~{CS}_MEMORY: now also U4.1 (~{CS})
Other:
- company: (none) -> Kallio Designs Oy
- title: (none) -> Programmable Keyboard
- moved on the sheet: C2, C4, R16
