File: PCB/Rev 02.00/000018 PGKB/controls.kicad_sch (KiCad schematic)
At the start: 15 parts, among them U11 SN74HCS365PWR

Commit message: updates
Parts:
- renumbered R24 to R15, R23 to R16, R20 to R17, R21 to R18, R22 to R20, R26 to R21, S2 to S11, U11 to U3

Commit message: Layout
Parts:
- renumbered S11 to S20
Changed lines of the file:
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@@
   (symbol (lib_id "KD_Switch:Encoder_Incremental_Bourns_PEC11R-4215K-S0012") (at 81.28 104.14 0) (unit 1)
     (in_bom yes) (on_board yes) (dnp no)
-    (property "Reference" "S11" (at 76.2 95.25 0) (do_not_autoplace)
+    (property "Reference" "S20" (at 76.2 95.25 0) (do_not_autoplace)
       (effects (font (size 1.27 1.27)) (justify left))
     )
@@
       (project "000018 PGKB"
         (path "/e63e39d7-6ac0-4ffd-8aa3-1841a4541b55/2eb44e1a-4042-4ea6-aca2-4836a6ec84e9/995d81b1-81b6-4111-907a-bbbe6e1f3b4b"
-          (reference "S11") (unit 1)
+          (reference "S20") (unit 1)
         )
       )

Commit message: sitte vaan routaus
Parts:
- TP8: value TestPoint_2.5mm_Round -> TP D2.5 mm H0.9mm; footprint KD_Connector_Pads:TestPoint_Pad_D2.5mm -> KD_Connector_Pads:TestPoint_Pad_D2.5mm_H0.9mm; symbol KD_Connector_Pads:TestPoint_2.5mm_Round -> KD_Connector_Pads:TestPoint_2.5mm_H0.9
Changed lines of the file:
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@@
     (effects (font (size 1.27 1.27)) (justify left))
   )
-  (symbol (lib_id "KD_Connector_Pads:TestPoint_2.5mm_Round") (at 101.6 114.3 0) (unit 1)
+  (symbol (lib_id "KD_Connector_Pads:TestPoint_2.5mm_H0.9") (at 101.6 114.3 0) (unit 1)
     (in_bom yes) (on_board yes) (dnp no)
     (property "Reference" "TP8" (at 99.06 107.95 0)
       (effects (font (size 1.27 1.27)) (justify left))
     )
-    (property "Value" "TestPoint_2.5mm_Round" (at 88.9 82.55 0)
-      (effects (font (size 1.27 1.27)) (justify left) hide)
-    )
-    (property "Footprint" "KD_Connector_Pads:TestPoint_Pad_D2.5mm" (at 88.9 100.33 0)
+    (property "Value" "TP D2.5 mm H0.9mm" (at 88.9 82.55 0)
+      (effects (font (size 1.27 1.27)) (justify left) hide)
+    )
+    (property "Footprint" "KD_Connector_Pads:TestPoint_Pad_D2.5mm_H0.9mm" (at 88.9 100.33 0)
       (effects (font (size 1.27 1.27)) (justify left) hide)
     )
@@
       (effects (font (size 1.27 1.27)) (justify left) hide)
     )
-    (property "Value" "TestPoint_2.5mm_Round" (at 88.9 82.55 0)
+    (property "Value" "TP D2.5 mm H0.9mm" (at 88.9 82.55 0)
       (effects (font (size 1.27 1.27)) (justify left) hide)
     )
@@
     )
   )
-  (symbol (lib_id "KD_Connector_Pads:TestPoint_2.5mm_Round") (at 96.52 87.63 0) (unit 1)
+  (symbol (lib_id "KD_Connector_Pads:TestPoint_2.5mm_H0.9") (at 96.52 87.63 0) (unit 1)
     (in_bom yes) (on_board yes) (dnp no)
     (property "Reference" "TP8" (at 93.98 81.28 0)
       (effects (font (size 1.27 1.27)) (justify left))
     )
-    (property "Value" "TestPoint_2.5mm_Round" (at 83.82 55.88 0)
-      (effects (font (size 1.27 1.27)) (justify left) hide)
-    )
-    (property "Footprint" "KD_Connector_Pads:TestPoint_Pad_D2.5mm" (at 83.82 73.66 0)
+    (property "Value" "TP D2.5 mm H0.9mm" (at 83.82 55.88 0)
+      (effects (font (size 1.27 1.27)) (justify left) hide)
+    )
+    (property "Footprint" "KD_Connector_Pads:TestPoint_Pad_D2.5mm_H0.9mm" (at 83.82 73.66 0)
       (effects (font (size 1.27 1.27)) (justify left) hide)
     )
@@
       (effects (font (size 1.27 1.27)) (justify left) hide)
     )
-    (property "Value" "TestPoint_2.5mm_Round" (at 83.82 55.88 0)
+    (property "Value" "TP D2.5 mm H0.9mm" (at 83.82 55.88 0)
       (effects (font (size 1.27 1.27)) (justify left) hide)
     )
@@
     )
   )
-  (symbol (lib_id "KD_Connector_Pads:TestPoint_2.5mm_Round") (at 105.41 99.06 0) (unit 1)
+  (symbol (lib_id "KD_Connector_Pads:TestPoint_2.5mm_H0.9") (at 105.41 99.06 0) (unit 1)
     (in_bom yes) (on_board yes) (dnp no)
     (property "Reference" "TP8" (at 102.87 92.71 0)
       (effects (font (size 1.27 1.27)) (justify left))
     )
-    (property "Value" "TestPoint_2.5mm_Round" (at 92.71 67.31 0)
-      (effects (font (size 1.27 1.27)) (justify left) hide)
-    )
-    (property "Footprint" "KD_Connector_Pads:TestPoint_Pad_D2.5mm" (at 92.71 85.09 0)
+    (property "Value" "TP D2.5 mm H0.9mm" (at 92.71 67.31 0)
+      (effects (font (size 1.27 1.27)) (justify left) hide)
+    )
+    (property "Footprint" "KD_Connector_Pads:TestPoint_Pad_D2.5mm_H0.9mm" (at 92.71 85.09 0)
       (effects (font (size 1.27 1.27)) (justify left) hide)
     )
@@
       (effects (font (size 1.27 1.27)) (justify left) hide)
     )
-    (property "Value" "TestPoint_2.5mm_Round" (at 92.71 67.31 0)
-      (effects (font (size 1.27 1.27)) (justify left) hide)
-    )
+    (property "Value" "TP D2.5 mm H0.9mm" (at 92.71 67.31 0)
+      (effects (font (size 1.27 1.27)) (justify left) hide)
+    )

Commit message: Leiskaa
Parts:
- R15, R16, R17: value R_0603_1k_1% -> 1k
Connections:
- net +3.3V renamed +3V3
Changed lines of the file:
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@@
     )
   )
-  (symbol (lib_id "power:+3.3V") (at 104.14 72.39 0) (unit 1)
+  (symbol (lib_id "power:+3V3") (at 104.14 72.39 0) (unit 1)
     (in_bom yes) (on_board yes) (dnp no) (fields_autoplaced)
     (property "Reference" "#PWR029" (at 104.14 76.2 0)
       (effects (font (size 1.27 1.27)) hide)
     )
-    (property "Value" "+3.3V" (at 104.14 68.834 0)
+    (property "Value" "+3V3" (at 104.14 68.834 0)
       (effects (font (size 1.27 1.27)))
     )
@@
   (symbol (lib_id "KD_Resistor:R_0603_1k_1%") (at 121.92 78.74 0) (unit 1)
     (in_bom yes) (on_board yes) (dnp no) (fields_autoplaced)
-    (property "Reference" "R17" (at 124.46 78.105 0)
-      (effects (font (size 1.27 1.27)) (justify left))
-    )
-    (property "Value" "R_0603_1k_1%" (at 109.22 46.99 0)
+    (property "Reference" "R17" (at 124.46 77.47 0)
+      (effects (font (size 1.27 1.27)) (justify left))
+    )
+    (property "Value" "1k" (at 109.22 46.99 0)
       (effects (font (size 1.27 1.27)) (justify left) hide)
     )
@@
       (effects (font (size 1.27 1.27)) (justify left) hide)
     )
-    (property "Code" "1k" (at 124.46 80.645 0)
+    (property "Code" "1k" (at 124.46 80.01 0)
       (effects (font (size 1.27 1.27)) (justify left))
     )
@@
     )
   )
-  (symbol (lib_id "power:+3.3V") (at 200.66 72.39 0) (unit 1)
+  (symbol (lib_id "power:+3V3") (at 200.66 72.39 0) (unit 1)
     (in_bom yes) (on_board yes) (dnp no) (fields_autoplaced)
     (property "Reference" "#PWR032" (at 200.66 76.2 0)
       (effects (font (size 1.27 1.27)) hide)
     )
-    (property "Value" "+3.3V" (at 200.66 68.834 0)
+    (property "Value" "+3V3" (at 200.66 68.834 0)
       (effects (font (size 1.27 1.27)))
     )
@@
     )
   )
-  (symbol (lib_id "power:+3.3V") (at 121.92 72.39 0) (unit 1)
+  (symbol (lib_id "power:+3V3") (at 121.92 72.39 0) (unit 1)
     (in_bom yes) (on_board yes) (dnp no) (fields_autoplaced)
     (property "Reference" "#PWR031" (at 121.92 76.2 0)
       (effects (font (size 1.27 1.27)) hide)
     )
-    (property "Value" "+3.3V" (at 121.92 68.834 0)
+    (property "Value" "+3V3" (at 121.92 68.834 0)
       (effects (font (size 1.27 1.27)))
     )
@@
   (symbol (lib_id "KD_Resistor:R_0603_1k_1%") (at 104.14 78.74 0) (unit 1)
     (in_bom yes) (on_board yes) (dnp no) (fields_autoplaced)
-    (property "Reference" "R15" (at 106.68 78.105 0)
-      (effects (font (size 1.27 1.27)) (justify left))
-    )
-    (property "Value" "R_0603_1k_1%" (at 91.44 46.99 0)
+    (property "Reference" "R15" (at 106.68 77.47 0)
+      (effects (font (size 1.27 1.27)) (justify left))
+    )
+    (property "Value" "1k" (at 91.44 46.99 0)
       (effects (font (size 1.27 1.27)) (justify left) hide)
     )
@@
       (effects (font (size 1.27 1.27)) (justify left) hide)
     )
-    (property "Code" "1k" (at 106.68 80.645 0)
+    (property "Code" "1k" (at 106.68 80.01 0)
       (effects (font (size 1.27 1.27)) (justify left))
     )
@@
     )
   )
-  (symbol (lib_id "power:+3.3V") (at 113.03 72.39 0) (unit 1)
+  (symbol (lib_id "power:+3V3") (at 113.03 72.39 0) (unit 1)
     (in_bom yes) (on_board yes) (dnp no) (fields_autoplaced)
     (property "Reference" "#PWR030" (at 113.03 76.2 0)
       (effects (font (size 1.27 1.27)) hide)
     )
-    (property "Value" "+3.3V" (at 113.03 68.834 0)
+    (property "Value" "+3V3" (at 113.03 68.834 0)
       (effects (font (size 1.27 1.27)))
     )
@@
   (symbol (lib_id "KD_Resistor:R_0603_1k_1%") (at 113.03 78.74 0) (unit 1)
     (in_bom yes) (on_board yes) (dnp no) (fields_autoplaced)
-    (property "Reference" "R16" (at 115.57 78.105 0)
-      (effects (font (size 1.27 1.27)) (justify left))
-    )
-    (property "Value" "R_0603_1k_1%" (at 100.33 46.99 0)
+    (property "Reference" "R16" (at 115.57 77.47 0)
+      (effects (font (size 1.27 1.27)) (justify left))
+    )
+    (property "Value" "1k" (at 100.33 46.99 0)
       (effects (font (size 1.27 1.27)) (justify left) hide)
     )
@@
       (effects (font (size 1.27 1.27)) (justify left) hide)
     )
-    (property "Code" "1k" (at 115.57 80.645 0)
-      (effects (font (size 1.27 1.27)) (justify left))
-    )
+    (property "Code" "1k" (at 115.57 80.01 0)
+      (effects (font (size 1.27 1.27)) (justify left))
+    )

Commit message: error fixing
Parts:
- C35: value C_0603_100n_X7R_50V -> 100n; Code 100n -> (none)
Connections:
- net GND: now also U3.10 (I4), U3.12 (I5), U3.14 (I6)
- no-connect marks 0 -> 3
Other:
- company: (none) -> Kallio Designs Oy
- title: (none) -> Programmable Keyboard
Changed lines of the file:
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@@
 (kicad_sch (version 20230121) (generator eeschema)
   (paper "A4")
+  (title_block
+    (title "Programmable Keyboard")
+    (date "2023-10-19")
+    (rev "1.0")
+    (company "Kallio Designs Oy")
+    (comment 1 "TL, NH")
+    (comment 3 "PCB_PN")
+  )
   (junction (at 113.03 101.6) (diameter 0) (color 0 0 0 0)
   )
@@
   (junction (at 139.7 101.6) (diameter 0) (color 0 0 0 0)
   )
+  (junction (at 191.77 102.87) (diameter 0) (color 0 0 0 0)
+  )
   (junction (at 200.66 82.55) (diameter 0) (color 0 0 0 0)
   )
+  (junction (at 191.77 100.33) (diameter 0) (color 0 0 0 0)
+  )
   (junction (at 105.41 101.6) (diameter 0) (color 0 0 0 0)
   )
@@
   (junction (at 166.37 90.17) (diameter 0) (color 0 0 0 0)
   )
+  (no_connect (at 228.6 102.87))
+  (no_connect (at 228.6 100.33))
+  (no_connect (at 228.6 97.79))
   (wire (pts (xy 139.7 132.08) (xy 139.7 134.62))
     (stroke (width 0) (type default))
@@
     (stroke (width 0) (type default))
   )
+  (wire (pts (xy 191.77 102.87) (xy 191.77 105.41))
+    (stroke (width 0) (type default))
+  )
   (wire (pts (xy 200.66 77.47) (xy 203.2 77.47))
     (stroke (width 0) (type default))
@@
     (stroke (width 0) (type default))
   )
+  (wire (pts (xy 203.2 102.87) (xy 191.77 102.87))
+    (stroke (width 0) (type default))
+  )
   (wire (pts (xy 92.71 106.68) (xy 92.71 109.22))
     (stroke (width 0) (type default))
@@
     (stroke (width 0) (type default))
   )
+  (wire (pts (xy 191.77 100.33) (xy 191.77 102.87))
+    (stroke (width 0) (type default))
+  )
   (wire (pts (xy 171.45 116.84) (xy 171.45 95.25))
     (stroke (width 0) (type default))
@@
     (stroke (width 0) (type default))
   )
+  (wire (pts (xy 203.2 100.33) (xy 191.77 100.33))
+    (stroke (width 0) (type default))
+  )
   (wire (pts (xy 193.04 69.85) (xy 193.04 82.55))
     (stroke (width 0) (type default))
@@
     (stroke (width 0) (type default))
   )
+  (wire (pts (xy 191.77 97.79) (xy 191.77 100.33))
+    (stroke (width 0) (type default))
+  )
   (wire (pts (xy 104.14 72.39) (xy 104.14 74.93))
     (stroke (width 0) (type default))
@@
   )
   (wire (pts (xy 69.85 101.6) (xy 69.85 90.17))
+    (stroke (width 0) (type default))
+  )
+  (wire (pts (xy 203.2 97.79) (xy 191.77 97.79))
     (stroke (width 0) (type default))
   )
@@
   (symbol (lib_id "KD_Capacitor:C_0603_100n_X7R_50V") (at 166.37 128.27 180) (unit 1)
     (in_bom yes) (on_board yes) (dnp no) (fields_autoplaced)
-    (property "Reference" "C35" (at 170.18 127.635 0)
+    (property "Reference" "C35" (at 170.18 127 0)
       (effects (font (size 1.27 1.27)) (justify right))
     )
-    (property "Value" "C_0603_100n_X7R_50V" (at 179.07 160.02 0)
-      (effects (font (size 1.27 1.27)) (justify left) hide)
+    (property "Value" "100n" (at 170.18 129.54 0)
+      (effects (font (size 1.27 1.27)) (justify right))
     )
     (property "Footprint" "KD_Capacitor:CAPC1608X90N" (at 179.07 142.24 0)
       (effects (font (size 1.27 1.27)) (justify left) hide)
     )
-    (property "Datasheet" "http://www.samsungsem.com/kr/support/product-search/mlcc/CL10B104KB8NNWC.jsp" (at 179.07 139.7 0)
-      (effects (font (size 1.27 1.27)) (justify left) hide)
-    )
-    (property "Value" "C_0603_100n_X7R_50V" (at 179.07 160.02 0)
-      (effects (font (size 1.27 1.27)) (justify left) hide)
-    )
-    (property "Code" "100n" (at 170.18 130.175 0)
-      (effects (font (size 1.27 1.27)) (justify right))
+    (property "Datasheet" "https://mm.digikey.com/Volume0/opasdata/d220001/medias/docus/658/CL10B104KB8NNWC_Spec.pdf" (at 179.07 139.7 0)
+      (effects (font (size 1.27 1.27)) (justify left) hide)
+    )
+    (property "Value" "100n" (at 170.18 130.81 0)
+      (effects (font (size 1.27 1.27)) (justify right) hide)
     )
     (property "Manufacturer" "Samsung" (at 179.07 157.48 0)
@@
   (symbol (lib_id "KD_Resistor:R_0603_10k_1%") (at 130.81 90.17 90) (unit 1)
     (in_bom yes) (on_board yes) (dnp no) (fields_autoplaced)
-    (property "Reference" "R18" (at 130.81 85.09 90)
+    (property "Reference" "R18" (at 130.81 83.82 90)
       (effects (font (size 1.27 1.27)))
     )
@@
       (effects (font (size 1.27 1.27)) (justify left) hide)
     )
-    (property "Code" "10k" (at 130.81 87.63 90)
+    (property "Code" "10k" (at 130.81 86.36 90)
       (effects (font (size 1.27 1.27)))
     )
@@
     )
   )
+  (symbol (lib_id "power:GND") (at 191.77 105.41 0) (mirror y) (unit 1)
+    (in_bom yes) (on_board yes) (dnp no)
+    (property "Reference" "#GND03" (at 191.77 111.76 0)
+      (effects (font (size 1.27 1.27)) hide)
+    )
+    (property "Value" "GND" (at 191.77 109.22 0)
+      (effects (font (size 1.27 1.27)))
+    )
+    (property "Footprint" "" (at 191.77 105.41 0)
+      (effects (font (size 1.27 1.27)) hide)
+    )
+    (property "Datasheet" "" (at 191.77 105.41 0)
+      (effects (font (size 1.27 1.27)) hide)
+    )
+    (pin "1")
+    (instances
+      (project "000052 RCCON"
+        (path "/c58960d9-4cac-4036-ad2e-1aef26946dae/f27a0928-8d32-4567-8ddf-132ea930c54d"
+          (reference "#GND03") (unit 1)
+        )
+      )
+      (project "000018 PGKB"
+        (path "/e63e39d7-6ac0-4ffd-8aa3-1841a4541b55/2eb44e1a-4042-4ea6-aca2-4836a6ec84e9/995d81b1-81b6-4111-907a-bbbe6e1f3b4b"
+          (reference "#GND039") (unit 1)
+        )
+      )
+    )
+  )
   (symbol (lib_id "KD_Resistor:R_0603_10k_1%") (at 130.81 116.84 90) (unit 1)
     (in_bom yes) (on_board yes) (dnp no) (fields_autoplaced)
-    (property "Reference" "R20" (at 130.81 111.76 90)
+    (property "Reference" "R20" (at 130.81 110.49 90)
       (effects (font (size 1.27 1.27)))
     )
@@
       (effects (font (size 1.27 1.27)) (justify left) hide)
     )
-    (property "Code" "10k" (at 130.81 114.3 90)
+    (property "Code" "10k" (at 130.81 113.03 90)
       (effects (font (size 1.27 1.27)))
     )
@@
   (symbol (lib_id "KD_Capacitor:C_0603_100n_X7R_50V") (at 153.67 128.27 180) (unit 1)
     (in_bom yes) (on_board yes) (dnp no) (fields_autoplaced)
-    (property "Reference" "C35" (at 157.48 127.635 0)
+    (property "Reference" "C35" (at 157.48 127 0)
       (effects (font (size 1.27 1.27)) (justify right))
     )
-    (property "Value" "C_0603_100n_X7R_50V" (at 166.37 160.02 0)
-      (effects (font (size 1.27 1.27)) (justify left) hide)
+    (property "Value" "100n" (at 157.48 129.54 0)
+      (effects (font (size 1.27 1.27)) (justify right))
     )
     (property "Footprint" "KD_Capacitor:CAPC1608X90N" (at 166.37 142.24 0)
       (effects (font (size 1.27 1.27)) (justify left) hide)
     )
-    (property "Datasheet" "http://www.samsungsem.com/kr/support/product-search/mlcc/CL10B104KB8NNWC.jsp" (at 166.37 139.7 0)
-      (effects (font (size 1.27 1.27)) (justify left) hide)
-    )
-    (property "Value" "C_0603_100n_X7R_50V" (at 166.37 160.02 0)
-      (effects (font (size 1.27 1.27)) (justify left) hide)
-    )
-    (property "Code" "100n" (at 157.48 130.175 0)
-      (effects (font (size 1.27 1.27)) (justify right))
+    (property "Datasheet" "https://mm.digikey.com/Volume0/opasdata/d220001/medias/docus/658/CL10B104KB8NNWC_Spec.pdf" (at 166.37 139.7 0)
+      (effects (font (size 1.27 1.27)) (justify left) hide)
+    )
+    (property "Value" "100n" (at 157.48 130.81 0)
+      (effects (font (size 1.27 1.27)) (justify right) hide)
     )
     (property "Manufacturer" "Samsung" (at 166.37 157.48 0)
@@
   (symbol (lib_id "KD_Capacitor:C_0603_100n_X7R_50V") (at 139.7 128.27 180) (unit 1)
     (in_bom yes) (on_board yes) (dnp no) (fields_autoplaced)
-    (property "Reference" "C35" (at 143.51 127.635 0)
+    (property "Reference" "C35" (at 143.51 127 0)
       (effects (font (size 1.27 1.27)) (justify right))
     )
-    (property "Value" "C_0603_100n_X7R_50V" (at 152.4 160.02 0)
-      (effects (font (size 1.27 1.27)) (justify left) hide)
+    (property "Value" "100n" (at 143.51 129.54 0)
+      (effects (font (size 1.27 1.27)) (justify right))
     )
     (property "Footprint" "KD_Capacitor:CAPC1608X90N" (at 152.4 142.24 0)
       (effects (font (size 1.27 1.27)) (justify left) hide)
     )
-    (property "Datasheet" "http://www.samsungsem.com/kr/support/product-search/mlcc/CL10B104KB8NNWC.jsp" (at 152.4 139.7 0)
-      (effects (font (size 1.27 1.27)) (justify left) hide)
-    )
-    (property "Value" "C_0603_100n_X7R_50V" (at 152.4 160.02 0)
-      (effects (font (size 1.27 1.27)) (justify left) hide)
-    )
-    (property "Code" "100n" (at 143.51 130.175 0)
-      (effects (font (size 1.27 1.27)) (justify right))
+    (property "Datasheet" "https://mm.digikey.com/Volume0/opasdata/d220001/medias/docus/658/CL10B104KB8NNWC_Spec.pdf" (at 152.4 139.7 0)
+      (effects (font (size 1.27 1.27)) (justify left) hide)
+    )
+    (property "Value" "100n" (at 143.51 130.81 0)
+      (effects (font (size 1.27 1.27)) (justify right) hide)
     )
     (property "Manufacturer" "Samsung" (at 152.4 157.48 0)
@@
   )
   (symbol (lib_id "KD_Resistor:R_0603_10k_1%") (at 130.81 101.6 90) (unit 1)
-    (in_bom yes) (on_board yes) (dnp no)
-    (property "Reference" "R19" (at 130.81 96.52 90)
+    (in_bom yes) (on_board yes) (dnp no) (fields_autoplaced)
+    (property "Reference" "R19" (at 130.81 95.25 90)
       (effects (font (size 1.27 1.27)))
     )
@@
       (effects (font (size 1.27 1.27)) (justify left) hide)
     )
-    (property "Code" "10k" (at 132.08 99.695 0)
-      (effects (font (size 1.27 1.27)) (justify left))
+    (property "Code" "10k" (at 130.81 97.79 90)
+      (effects (font (size 1.27 1.27)))
     )
     (property "Manufacturer" "Stackpole Electronics Inc" (at 101.6 114.3 0)

Commit message: MODIFICATIONS To Rev 2
Parts:
- S20: value symbol_template -> PEC11R-4215K-S0012; Code PEC11R-4215K-S0012 -> (none)
Changed lines of the file:
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@@
   (title_block
     (title "Programmable Keyboard")
-    (date "2023-10-19")
+    (date "2024-01-24")
     (rev "1.0")
     (company "Kallio Designs Oy")
@@
       (effects (font (size 1.27 1.27)) (justify left))
     )
-    (property "Value" "symbol_template" (at 68.58 59.69 0)
-      (effects (font (size 1.27 1.27)) (justify left) hide)
+    (property "Value" "PEC11R-4215K-S0012" (at 76.2 97.536 0) (do_not_autoplace)
+      (effects (font (size 1.27 1.27)) (justify left))
     )
     (property "Footprint" "KD_Switch:RotaryEncoder_Bourns_Vertical_PEC11R-4x15f-Sxxxx" (at 68.58 77.47 0)
@@
       (effects (font (size 1.27 1.27)) (justify left) hide)
     )
-    (property "Code" "PEC11R-4215K-S0012" (at 76.2 97.79 0) (do_not_autoplace)
-      (effects (font (size 1.27 1.27)) (justify left))
-    )
     (property "Manufacturer" "Bourns Inc." (at 68.58 62.23 0)
