File: PCB/Rev 02.00/000018 PGKB/mechanical.kicad_sch (KiCad schematic)
At the start: 7 parts

Commit message: Schematic
Other:
- title: TITLE -> Programmable Keyboard
Changed lines of the file:
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@@
   (paper "A4")
   (title_block
-    (title "TITLE")
-    (date "2023-05-28")
+    (title "Programmable Keyboard")
+    (date "2023-10-14")
     (rev "1.0")
     (company "Kallio Designs Oy")
-    (comment 1 "Teemu Latonen")
+    (comment 1 "TL, NH")
     (comment 2 "ASSEMBLY_PN")
     (comment 3 "PCB_PN")

Commit message: skema
Parts:
- removed H1: M2_NPTH_2.2_Minimal, KD_Mechanical_Mounting_Hole:MountingHole_2.2mm_NPTH, symbol KD_Mechanical_Mounting_Hole:M2_NPTH_2.2_Minimal
- added H1, H2, H3, H4, H5: NPTH 3.2 M3 Clearance, KD_Mechanical_Mounting_Hole:NPTH_3.2mm_M3_clearance, symbol KD_Mechanical_Mounting_Hole:NPTH_3.2_M3_Clearance
- added H6: PTH 3.2 M3 Clearance, KD_Mechanical_Mounting_Hole:PTH_3.2mm_M3_clearance_B, symbol KD_Mechanical_Mounting_Hole:PTH_3.2_M3_Clearance_B
Connections:
- new net GND: H6.1

Commit message: Layout
Parts:
- removed H1: NPTH 3.2 M3 Clearance, KD_Mechanical_Mounting_Hole:NPTH_3.2mm_M3_clearance, symbol KD_Mechanical_Mounting_Hole:NPTH_3.2_M3_Clearance
- added H5: PTH 3.2 M3 Clearance, KD_Mechanical_Mounting_Hole:PTH_3.2mm_M3_clearance_B, symbol KD_Mechanical_Mounting_Hole:PTH_3.2_M3_Clearance_B
- renumbered H5 to H1
Connections:
- net GND: now also H5.1
Other:
- moved on the sheet: H1, H2
Changed lines of the file:
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@@
     (comment 3 "PCB_PN")
+  )
+  (junction (at 57.15 69.85) (diameter 0) (color 0 0 0 0)
+  )
+  (wire (pts (xy 58.42 63.5) (xy 57.15 63.5))
+    (stroke (width 0) (type default))
   )
   (wire (pts (xy 57.15 69.85) (xy 57.15 71.12))
@@
     (stroke (width 0) (type default))
   )
-  (symbol (lib_id "KD_Mechanical_Mounting_Hole:NPTH_3.2_M3_Clearance") (at 63.5 38.1 0) (unit 1)
-    (in_bom yes) (on_board yes) (dnp no) (fields_autoplaced)
-    (property "Reference" "H2" (at 67.31 36.83 0)
-      (effects (font (size 1.27 1.27)) (justify left))
-    )
-    (property "Value" "NPTH 3.2 M3 Clearance" (at 67.31 39.37 0)
-      (effects (font (size 1.27 1.27)) (justify left))
-    )
-    (property "Footprint" "KD_Mechanical_Mounting_Hole:NPTH_3.2mm_M3_clearance" (at 50.8 24.13 0)
-      (effects (font (size 1.27 1.27)) (justify left) hide)
-    )
-    (property "Datasheet" "" (at 50.8 26.67 0)
-      (effects (font (size 1.27 1.27)) (justify left) hide)
-    )
-    (property "Manufacturer" "DNP" (at 50.8 8.89 0)
-      (effects (font (size 1.27 1.27)) (justify left) hide)
-    )
-    (property "MFG_PartNo" "DNP" (at 50.8 11.43 0)
-      (effects (font (size 1.27 1.27)) (justify left) hide)
-    )
-    (property "Supplier" "DNP" (at 50.8 13.97 0)
-      (effects (font (size 1.27 1.27)) (justify left) hide)
-    )
-    (property "Supplier_PartNo" "DNP" (at 50.8 16.51 0)
-      (effects (font (size 1.27 1.27)) (justify left) hide)
-    )
-    (property "DNP" "T" (at 50.8 19.05 0)
-      (effects (font (size 1.27 1.27)) (justify left) hide)
-    )
-    (property "Price" "0.00" (at 50.8 21.59 0)
+  (wire (pts (xy 57.15 63.5) (xy 57.15 69.85))
+    (stroke (width 0) (type default))
+  )
+  (symbol (lib_id "KD_Mechanical_Mounting_Hole:NPTH_3.2_M3_Clearance") (at 63.5 44.45 0) (unit 1)
+    (in_bom yes) (on_board yes) (dnp no) (fields_autoplaced)
+    (property "Reference" "H2" (at 67.31 43.18 0)
+      (effects (font (size 1.27 1.27)) (justify left))
+    )
+    (property "Value" "NPTH 3.2 M3 Clearance" (at 67.31 45.72 0)
+      (effects (font (size 1.27 1.27)) (justify left))
+    )
+    (property "Footprint" "KD_Mechanical_Mounting_Hole:NPTH_3.2mm_M3_clearance" (at 50.8 30.48 0)
+      (effects (font (size 1.27 1.27)) (justify left) hide)
+    )
+    (property "Datasheet" "" (at 50.8 33.02 0)
+      (effects (font (size 1.27 1.27)) (justify left) hide)
+    )
+    (property "Manufacturer" "DNP" (at 50.8 15.24 0)
+      (effects (font (size 1.27 1.27)) (justify left) hide)
+    )
+    (property "MFG_PartNo" "DNP" (at 50.8 17.78 0)
+      (effects (font (size 1.27 1.27)) (justify left) hide)
+    )
+    (property "Supplier" "DNP" (at 50.8 20.32 0)
+      (effects (font (size 1.27 1.27)) (justify left) hide)
+    )
+    (property "Supplier_PartNo" "DNP" (at 50.8 22.86 0)
+      (effects (font (size 1.27 1.27)) (justify left) hide)
+    )
+    (property "DNP" "T" (at 50.8 25.4 0)
+      (effects (font (size 1.27 1.27)) (justify left) hide)
+    )
+    (property "Price" "0.00" (at 50.8 27.94 0)
       (effects (font (size 1.27 1.27)) (justify left) hide)
     )
@@
     )
   )
-  (symbol (lib_id "KD_Mechanical_Mounting_Hole:NPTH_3.2_M3_Clearance") (at 63.5 44.45 0) (unit 1)
-    (in_bom yes) (on_board yes) (dnp no) (fields_autoplaced)
-    (property "Reference" "H1" (at 67.31 43.18 0)
-      (effects (font (size 1.27 1.27)) (justify left))
-    )
-    (property "Value" "NPTH 3.2 M3 Clearance" (at 67.31 45.72 0)
-      (effects (font (size 1.27 1.27)) (justify left))
-    )
-    (property "Footprint" "KD_Mechanical_Mounting_Hole:NPTH_3.2mm_M3_clearance" (at 50.8 30.48 0)
-      (effects (font (size 1.27 1.27)) (justify left) hide)
-    )
-    (property "Datasheet" "" (at 50.8 33.02 0)
-      (effects (font (size 1.27 1.27)) (justify left) hide)
-    )
-    (property "Manufacturer" "DNP" (at 50.8 15.24 0)
-      (effects (font (size 1.27 1.27)) (justify left) hide)
-    )
-    (property "MFG_PartNo" "DNP" (at 50.8 17.78 0)
-      (effects (font (size 1.27 1.27)) (justify left) hide)
-    )
-    (property "Supplier" "DNP" (at 50.8 20.32 0)
-      (effects (font (size 1.27 1.27)) (justify left) hide)
-    )
-    (property "Supplier_PartNo" "DNP" (at 50.8 22.86 0)
-      (effects (font (size 1.27 1.27)) (justify left) hide)
-    )
-    (property "DNP" "T" (at 50.8 25.4 0)
-      (effects (font (size 1.27 1.27)) (justify left) hide)
-    )
-    (property "Price" "0.00" (at 50.8 27.94 0)
-      (effects (font (size 1.27 1.27)) (justify left) hide)
-    )
-    (instances
-      (project "000018 PGKB"
-        (path "/e63e39d7-6ac0-4ffd-8aa3-1841a4541b55/8f5ee264-ab78-438d-b8d5-1e547e5afc7c"
-          (reference "H1") (unit 1)
-        )
-      )
-    )
-  )
   (symbol (lib_id "KD_Mechanical:Fiducial_0.5mm") (at 38.1 44.45 0) (unit 1)
     (in_bom yes) (on_board yes) (dnp no) (fields_autoplaced)
@@
         (path "/e63e39d7-6ac0-4ffd-8aa3-1841a4541b55/8f5ee264-ab78-438d-b8d5-1e547e5afc7c"
           (reference "FD4") (unit 1)
+        )
+      )
+    )
+  )
+  (symbol (lib_id "KD_Mechanical_Mounting_Hole:PTH_3.2_M3_Clearance_B") (at 63.5 63.5 0) (unit 1)
+    (in_bom yes) (on_board yes) (dnp no) (fields_autoplaced)
+    (property "Reference" "H5" (at 67.31 62.23 0)
+      (effects (font (size 1.27 1.27)) (justify left))
+    )
+    (property "Value" "PTH 3.2 M3 Clearance" (at 67.31 64.77 0)
+      (effects (font (size 1.27 1.27)) (justify left))
+    )
+    (property "Footprint" "KD_Mechanical_Mounting_Hole:PTH_3.2mm_M3_clearance_B" (at 50.8 49.53 0)
+      (effects (font (size 1.27 1.27)) (justify left) hide)
+    )
+    (property "Datasheet" "" (at 50.8 52.07 0)
+      (effects (font (size 1.27 1.27)) (justify left) hide)
+    )
+    (property "Manufacturer" "DNP" (at 50.8 34.29 0)
+      (effects (font (size 1.27 1.27)) (justify left) hide)
+    )
+    (property "MFG_PartNo" "DNP" (at 50.8 36.83 0)
+      (effects (font (size 1.27 1.27)) (justify left) hide)
+    )
+    (property "Supplier" "DNP" (at 50.8 39.37 0)
+      (effects (font (size 1.27 1.27)) (justify left) hide)
+    )
+    (property "Supplier_PartNo" "DNP" (at 50.8 41.91 0)
+      (effects (font (size 1.27 1.27)) (justify left) hide)
+    )
+    (property "DNP" "T" (at 50.8 44.45 0)
+      (effects (font (size 1.27 1.27)) (justify left) hide)
+    )
+    (property "Price" "0.00" (at 50.8 46.99 0)
+      (effects (font (size 1.27 1.27)) (justify left) hide)
+    )
+    (pin "1")
+    (instances
+      (project "000018 PGKB"
+        (path "/e63e39d7-6ac0-4ffd-8aa3-1841a4541b55/8f5ee264-ab78-438d-b8d5-1e547e5afc7c"
+          (reference "H5") (unit 1)
         )
       )
@@
     )
   )
-  (symbol (lib_id "KD_Mechanical_Mounting_Hole:NPTH_3.2_M3_Clearance") (at 63.5 63.5 0) (unit 1)
-    (in_bom yes) (on_board yes) (dnp no) (fields_autoplaced)
-    (property "Reference" "H5" (at 67.31 62.23 0)
-      (effects (font (size 1.27 1.27)) (justify left))
-    )
-    (property "Value" "NPTH 3.2 M3 Clearance" (at 67.31 64.77 0)
-      (effects (font (size 1.27 1.27)) (justify left))
-    )
-    (property "Footprint" "KD_Mechanical_Mounting_Hole:NPTH_3.2mm_M3_clearance" (at 50.8 49.53 0)
-      (effects (font (size 1.27 1.27)) (justify left) hide)
-    )
-    (property "Datasheet" "" (at 50.8 52.07 0)
-      (effects (font (size 1.27 1.27)) (justify left) hide)
-    )
-    (property "Manufacturer" "DNP" (at 50.8 34.29 0)
-      (effects (font (size 1.27 1.27)) (justify left) hide)
-    )
-    (property "MFG_PartNo" "DNP" (at 50.8 36.83 0)
-      (effects (font (size 1.27 1.27)) (justify left) hide)
-    )
-    (property "Supplier" "DNP" (at 50.8 39.37 0)
-      (effects (font (size 1.27 1.27)) (justify left) hide)
-    )
-    (property "Supplier_PartNo" "DNP" (at 50.8 41.91 0)
-      (effects (font (size 1.27 1.27)) (justify left) hide)
-    )
-    (property "DNP" "T" (at 50.8 44.45 0)
-      (effects (font (size 1.27 1.27)) (justify left) hide)
-    )
-    (property "Price" "0.00" (at 50.8 46.99 0)
-      (effects (font (size 1.27 1.27)) (justify left) hide)
-    )
-    (instances
-      (project "000018 PGKB"
-        (path "/e63e39d7-6ac0-4ffd-8aa3-1841a4541b55/8f5ee264-ab78-438d-b8d5-1e547e5afc7c"
-          (reference "H5") (unit 1)
-        )
-      )
+  (symbol (lib_id "KD_Mechanical_Mounting_Hole:NPTH_3.2_M3_Clearance") (at 63.5 38.1 0) (unit 1)
+    (in_bom yes) (on_board yes) (dnp no) (fields_autoplaced)
+    (property "Reference" "H1" (at 67.31 36.83 0)
+      (effects (font (size 1.27 1.27)) (justify left))
+    )
+    (property "Value" "NPTH 3.2 M3 Clearance" (at 67.31 39.37 0)
+      (effects (font (size 1.27 1.27)) (justify left))
+    )
+    (property "Footprint" "KD_Mechanical_Mounting_Hole:NPTH_3.2mm_M3_clearance" (at 50.8 24.13 0)
+      (effects (font (size 1.27 1.27)) (justify left) hide)
+    )
+    (property "Datasheet" "" (at 50.8 26.67 0)
+      (effects (font (size 1.27 1.27)) (justify left) hide)
+    )
+    (property "Manufacturer" "DNP" (at 50.8 8.89 0)
+      (effects (font (size 1.27 1.27)) (justify left) hide)
+    )
+    (property "MFG_PartNo" "DNP" (at 50.8 11.43 0)
+      (effects (font (size 1.27 1.27)) (justify left) hide)
+    )
+    (property "Supplier" "DNP" (at 50.8 13.97 0)
+      (effects (font (size 1.27 1.27)) (justify left) hide)
+    )
+    (property "Supplier_PartNo" "DNP" (at 50.8 16.51 0)
+      (effects (font (size 1.27 1.27)) (justify left) hide)
+    )
+    (property "DNP" "T" (at 50.8 19.05 0)
+      (effects (font (size 1.27 1.27)) (justify left) hide)
+    )
+    (property "Price" "0.00" (at 50.8 21.59 0)
+      (effects (font (size 1.27 1.27)) (justify left) hide)
+    )
+    (instances
+      (project "000018 PGKB"
+        (path "/e63e39d7-6ac0-4ffd-8aa3-1841a4541b55/8f5ee264-ab78-438d-b8d5-1e547e5afc7c"
+          (reference "H1") (unit 1)
+        )
+      )

Commit message: Leiskaa
Parts:
- added ART1: 4-Layer Marking, KD_Mechanical:ART_4-LAYER, symbol KD_Mechanical:Artwork_4-Layer_marking
- added ART2: Logo 2.5 mm Silk, KD_Mechanical:ART_LOGO_TEXT_2.5MM_SILK, symbol KD_Mechanical:Artwork_Logo_Silk_2.5mm
- H3: value NPTH 3.2 M3 Clearance -> NPTH_3.2; footprint KD_Mechanical_Mounting_Hole:NPTH_3.2mm_M3_clearance -> KD_Mechanical_Mounting_Hole:NPTH_3.2mm; symbol KD_Mechanical_Mounting_Hole:NPTH_3.2_M3_Clearance -> KD_Mechanical_Mounting_Hole:NPTH_3.2; Code (none) -> 3.2 mm hole
Other:
- moved on the sheet: FD1, FD2, FD3, FD4, FD5, FD6, H1, H2, H3, H4, H5, H6

Commit message: error fixing
Parts:
- FD1, FD2, FD3, FD4, FD5, FD6: value Fiducial_0.5mm -> Fiducial 0.5 mm; Code DNP -> (none); now left out of the parts list
Other:
- moved on the sheet: FD1, FD2, FD3, FD4, FD5, FD6, H1, H2, H3, H4, H5, H6
