File: PCB/Rev 02.00/000018 PGKB/rev_history.kicad_sch (KiCad schematic)
At the start: 0 parts

Commit message: Schematic
Other:
- note added: "1.0"
- note added: "14.10.2023"
- note added: "Niko Hämäläinen"
- note removed: "13.08.2022"
- note removed: "A"
- title: TITLE -> Programmable Keyboard
Changed lines of the file:
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@@
   (paper "A4")
   (title_block
-    (title "TITLE")
-    (date "2023-05-28")
+    (title "Programmable Keyboard")
+    (date "2023-10-14")
     (rev "1.0")
     (company "Kallio Designs Oy")
-    (comment 1 "Teemu Latonen")
+    (comment 1 "TL, NH")
     (comment 2 "ASSEMBLY_PN")
     (comment 3 "PCB_PN")
@@
     (stroke (width 0) (type solid) (color 0 0 0 1))
   )
-  (text "13.08.2022" (at 69.85 58.42 0)
+  (text "14.10.2023" (at 69.85 58.42 0)
     (effects (font (size 2 2)) (justify left bottom))
   )
@@
     (effects (font (size 2 2) (thickness 1) bold) (justify left bottom))
   )
-  (text "A" (at 58.42 58.42 0)
+  (text "1.0" (at 58.42 58.42 0)
     (effects (font (size 2 2)) (justify left bottom))
   )
@@
     (effects (font (size 2 2)) (justify left bottom))
   )
-  (text "Teemu Latonen" (at 208.28 58.42 0)
-    (effects (font (size 2 2)) (justify left bottom))
+  (text "Teemu Latonen" (at 208.026 56.515 0)
+    (effects (font (size 1.5 1.5)) (justify left bottom))
+  )
+  (text "Niko Hämäläinen" (at 208.026 59.055 0)
+    (effects (font (size 1.5 1.5)) (justify left bottom))
   )
 )

Commit message: error fixing
Other:
- note added: "19.10.2023"
- note removed: "14.10.2023"
Changed lines of the file:
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@@
   (title_block
     (title "Programmable Keyboard")
-    (date "2023-10-14")
+    (date "2023-10-19")
     (rev "1.0")
     (company "Kallio Designs Oy")
@@
     (stroke (width 0) (type solid) (color 0 0 0 1))
   )
-  (text "14.10.2023" (at 69.85 58.42 0)
+  (text "19.10.2023" (at 69.85 58.42 0)
     (effects (font (size 2 2)) (justify left bottom))
   )
