File: PCB/Rev 02.10/000018 PGKB/main.kicad_sch (KiCad schematic)
At the start: 0 parts

Commit message: Signals renamed
Other:
- sheet Microcontroller ports: added GPIO13, GPIO14, GPIO15, GPIO16, GPIO27, GPIO28, GPIO29; removed GPIO10, GPIO11, GPIO12, GPIO3, GPIO4, GPIO5, GPIO6
Changed lines of the file:
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@@
-			)
-		)
-		(pin "GPIO12" bidirectional
-			(at 189.23 111.76 0)
-			(effects
-				(font
-					(size 1.27 1.27)
-				)
-				(justify right)
 			)
 		)
@@
 				)
 				(justify left)
-			)
-		)
-		(pin "GPIO5" bidirectional
-			(at 189.23 80.01 0)
-			(effects
-				(font
-					(size 1.27 1.27)
-				)
-				(justify right)
-			)
-		)
-		(pin "GPIO4" bidirectional
-			(at 189.23 77.47 0)
-			(effects
-				(font
-					(size 1.27 1.27)
-				)
-				(justify right)
-			)
-		)
-		(pin "GPIO3" bidirectional
-			(at 189.23 74.93 0)
-			(effects
-				(font
-					(size 1.27 1.27)
-				)
-				(justify right)
-			)
-		)
-		(pin "GPIO6" bidirectional
-			(at 189.23 82.55 0)
-			(effects
-				(font
-					(size 1.27 1.27)
-				)
-				(justify right)
-			)
-		)
-		(pin "GPIO8" bidirectional
-			(at 189.23 87.63 0)
-			(effects
-				(font
-					(size 1.27 1.27)
-				)
-				(justify right)
-			)
-		)
-		(pin "GPIO7" bidirectional
-			(at 189.23 85.09 0)
-			(effects
-				(font
-					(size 1.27 1.27)
-				)
-				(justify right)
 			)
 		)
@@
 			)
 		)
-		(pin "GPIO9" bidirectional
-			(at 189.23 90.17 0)
+		(pin "GPIO8" bidirectional
+			(at 189.23 77.47 0)
 			(effects
 				(font
@@
 			)
 		)
-		(pin "GPIO11" bidirectional
+		(pin "GPIO7" bidirectional
+			(at 189.23 74.93 0)
+			(effects
+				(font
+					(size 1.27 1.27)
+				)
+				(justify right)
+			)
+		)
+		(pin "GPIO9" bidirectional
+			(at 189.23 80.01 0)
+			(effects
+				(font
+					(size 1.27 1.27)
+				)
+				(justify right)
+			)
+		)
+		(pin "GPIO29" bidirectional
+			(at 189.23 111.76 0)
+			(effects
+				(font
+					(size 1.27 1.27)
+				)
+				(justify right)
+			)
+		)
+		(pin "GPIO27" bidirectional
+			(at 189.23 92.71 0)
+			(effects
+				(font
+					(size 1.27 1.27)
+				)
+				(justify right)
+			)
+		)
+		(pin "GPIO28" bidirectional
 			(at 189.23 95.25 0)
 			(effects
@@
 			)
 		)
-		(pin "GPIO10" bidirectional
-			(at 189.23 92.71 0)
+		(pin "GPIO15" bidirectional
+			(at 189.23 87.63 0)
 			(effects
 				(font
+					(size 1.27 1.27)
+				)
+				(justify right)
+			)
+		)
+		(pin "GPIO14" bidirectional
+			(at 189.23 85.09 0)
+			(effects
+				(font
+					(size 1.27 1.27)
+				)
+				(justify right)
+			)
+		)
+		(pin "GPIO13" bidirectional
+			(at 189.23 82.55 0)
+			(effects
+				(font
+					(size 1.27 1.27)
+				)
+				(justify right)
+			)
+		)
+		(pin "GPIO16" bidirectional
+			(at 189.23 90.17 0)
+			(effects
+				(font
