File: PCB/Rev 02.10/000018 PGKB/mcu.kicad_sch (KiCad schematic)
At the start: 32 parts, among them U5 RP2040, Y1 12 MHz

Commit message: Update mcu.kicad_sch
Other:
- note added: "Place close to pin 44"
- moved on the sheet: C4
Changed lines of the file:
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@@
   (junction (at 104.14 22.86) (diameter 0) (color 0 0 0 0)
   )
+  (junction (at 147.32 40.005) (diameter 0) (color 0 0 0 0)
+  )
   (junction (at 234.95 125.73) (diameter 0) (color 0 0 0 0)
   )
@@
   )
   (junction (at 64.77 182.88) (diameter 0) (color 0 0 0 0)
-  )
-  (junction (at 59.69 22.86) (diameter 0) (color 0 0 0 0)
   )
   (junction (at 208.28 123.19) (diameter 0) (color 0 0 0 0)
@@
     (stroke (width 0) (type default))
   )
-  (wire (pts (xy 59.69 31.75) (xy 59.69 33.02))
+  (wire (pts (xy 154.305 50.8) (xy 154.305 52.07))
     (stroke (width 0) (type default))
   )
@@
     (stroke (width 0) (type default))
   )
-  (wire (pts (xy 59.69 22.86) (xy 59.69 24.13))
-    (stroke (width 0) (type default))
-  )
   (wire (pts (xy 110.49 44.45) (xy 110.49 43.18))
     (stroke (width 0) (type default))
@@
     (stroke (width 0) (type default))
   )
-  (wire (pts (xy 59.69 22.86) (xy 71.12 22.86))
-    (stroke (width 0) (type default))
-  )
   (wire (pts (xy 100.33 44.45) (xy 100.33 43.18))
     (stroke (width 0) (type default))
@@
     (stroke (width 0) (type default))
   )
+  (wire (pts (xy 154.305 43.18) (xy 154.305 40.005))
+    (stroke (width 0) (type default))
+  )
   (bus (pts (xy 251.46 130.81) (xy 251.46 133.35))
     (stroke (width 0) (type default))
@@
     (stroke (width 0) (type default))
   )
-  (wire (pts (xy 147.32 22.86) (xy 147.32 57.15))
+  (wire (pts (xy 147.32 22.86) (xy 147.32 40.005))
     (stroke (width 0) (type default))
   )
@@
     (stroke (width 0) (type default))
   )
+  (wire (pts (xy 147.32 40.005) (xy 154.305 40.005))
+    (stroke (width 0) (type default))
+  )
   (wire (pts (xy 64.77 170.18) (xy 64.77 182.88))
     (stroke (width 0) (type default))
@@
     (stroke (width 0) (type default))
   )
-  (wire (pts (xy 55.88 22.86) (xy 59.69 22.86))
+  (wire (pts (xy 55.88 22.86) (xy 71.12 22.86))
     (stroke (width 0) (type default))
   )
@@
   )
   (wire (pts (xy 187.96 85.09) (xy 162.56 85.09))
+    (stroke (width 0) (type default))
+  )
+  (wire (pts (xy 147.32 40.005) (xy 147.32 57.15))
     (stroke (width 0) (type default))
   )
@@
     (fill (type none))
     (effects (font (size 1.27 1.27)) (justify left top))
+  )
+  (text "Place close to pin 44" (at 158.75 52.705 0)
+    (effects (font (size 1.27 1.27)) (justify left bottom))
   )
   (label "USBBOOT" (at 163.83 120.65 0) (fields_autoplaced)
@@
     )
   )
-  (symbol (lib_id "KD_Capacitor:C_0805_1u_X7R_25V") (at 59.69 27.94 0) (unit 1)
+  (symbol (lib_id "KD_Capacitor:C_0805_1u_X7R_25V") (at 154.305 46.99 0) (unit 1)
     (in_bom yes) (on_board yes) (dnp no)
-    (property "Reference" "C4" (at 62.23 26.67 0)
+    (property "Reference" "C4" (at 156.845 45.72 0)
       (effects (font (size 1.27 1.27)) (justify left))
     )
-    (property "Value" "1u" (at 46.99 -3.81 0)
-      (effects (font (size 1.27 1.27)) (justify left) hide)
-    )
-    (property "Footprint" "KD_Capacitor:CAPC2012X135N" (at 46.99 13.97 0)
-      (effects (font (size 1.27 1.27)) (justify left) hide)
-    )
-    (property "Datasheet" "https://mm.digikey.com/Volume0/opasdata/d220001/medias/docus/1105/CL21B105KAFNNNE_Spec.pdf" (at 46.99 16.51 0)
-      (effects (font (size 1.27 1.27)) (justify left) hide)
-    )
-    (property "Code" "1u" (at 62.23 29.21 0)
+    (property "Value" "1u" (at 141.605 15.24 0)
+      (effects (font (size 1.27 1.27)) (justify left) hide)
+    )
+    (property "Footprint" "KD_Capacitor:CAPC2012X135N" (at 141.605 33.02 0)
+      (effects (font (size 1.27 1.27)) (justify left) hide)
+    )
+    (property "Datasheet" "https://mm.digikey.com/Volume0/opasdata/d220001/medias/docus/1105/CL21B105KAFNNNE_Spec.pdf" (at 141.605 35.56 0)
+      (effects (font (size 1.27 1.27)) (justify left) hide)
+    )
+    (property "Code" "1u" (at 156.845 48.26 0)
       (effects (font (size 1.27 1.27)) (justify left))
     )
-    (property "Manufacturer" "Samsung Electro-Mechanics" (at 46.99 -1.27 0)
-      (effects (font (size 1.27 1.27)) (justify left) hide)
-    )
-    (property "MFG_PartNo" "CL21B105KAFNNNE" (at 46.99 1.27 0)
-      (effects (font (size 1.27 1.27)) (justify left) hide)
-    )
-    (property "Supplier" "Digi-Key" (at 46.99 3.81 0)
-      (effects (font (size 1.27 1.27)) (justify left) hide)
-    )
-    (property "Supplier_PartNo" "1276-1066-1-ND" (at 46.99 6.35 0)
-      (effects (font (size 1.27 1.27)) (justify left) hide)
-    )
-    (property "DNP" "F" (at 46.99 8.89 0)
-      (effects (font (size 1.27 1.27)) (justify left) hide)
-    )
-    (property "Price" "0.03" (at 46.99 11.43 0)
+    (property "Manufacturer" "Samsung Electro-Mechanics" (at 141.605 17.78 0)
+      (effects (font (size 1.27 1.27)) (justify left) hide)
+    )
+    (property "MFG_PartNo" "CL21B105KAFNNNE" (at 141.605 20.32 0)
+      (effects (font (size 1.27 1.27)) (justify left) hide)
+    )
+    (property "Supplier" "Digi-Key" (at 141.605 22.86 0)
+      (effects (font (size 1.27 1.27)) (justify left) hide)
+    )
+    (property "Supplier_PartNo" "1276-1066-1-ND" (at 141.605 25.4 0)
+      (effects (font (size 1.27 1.27)) (justify left) hide)
+    )
+    (property "DNP" "F" (at 141.605 27.94 0)
+      (effects (font (size 1.27 1.27)) (justify left) hide)
+    )
+    (property "Price" "0.03" (at 141.605 30.48 0)
       (effects (font (size 1.27 1.27)) (justify left) hide)
     )
@@
     )
   )
-  (symbol (lib_id "power:GND") (at 59.69 33.02 0) (mirror y) (unit 1)
+  (symbol (lib_id "power:GND") (at 154.305 52.07 0) (mirror y) (unit 1)
     (in_bom yes) (on_board yes) (dnp no)
-    (property "Reference" "#GND04" (at 59.69 39.37 0)
-      (effects (font (size 1.27 1.27)) hide)
-    )
-    (property "Value" "GND" (at 59.69 36.83 0)
+    (property "Reference" "#GND04" (at 154.305 58.42 0)
+      (effects (font (size 1.27 1.27)) hide)
+    )
+    (property "Value" "GND" (at 154.305 55.88 0)
       (effects (font (size 1.27 1.27)))
     )
-    (property "Footprint" "" (at 59.69 33.02 0)
-      (effects (font (size 1.27 1.27)) hide)
-    )
-    (property "Datasheet" "" (at 59.69 33.02 0)
-      (effects (font (size 1.27 1.27)) hide)
-    )
+    (property "Footprint" "" (at 154.305 52.07 0)
+      (effects (font (size 1.27 1.27)) hide)
+    )
+    (property "Datasheet" "" (at 154.305 52.07 0)
+      (effects (font (size 1.27 1.27)) hide)
+    )

Commit message: updates
Other:
- note added: "Place C23 close to pin 45"
- note added: "Place C25 close to pin 44"
- note removed: "Place close to pin 44"
Changed lines of the file:
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@@
   (title_block
     (title "Programmable Keyboard")
-    (date "2024-01-24")
-    (rev "2.0")
+    (date "2024-04-09")
+    (rev "2.1")
     (company "Kallio Designs Oy")
     (comment 1 "TL, NH")
@@
     (stroke (width 0) (type default))
   )
-  (text_box "Notes:\nRP2040"
-    (at 207.01 156.21 0) (size 77.47 21.59)
+  (text_box "Notes:\nRP2040 Hardware design guide:\nhttps://datasheets.raspberrypi.com/rp2040/hardware-design-with-rp2040.pdf\n"
+    (at 187.96 156.21 0) (size 96.52 21.59)
     (stroke (width 0) (type default))
     (fill (type none))
-    (effects (font (size 1.27 1.27)) (justify left top))
-  )
-  (text "Place close to pin 44" (at 158.75 52.705 0)
+    (effects (font (size 1.27 1.27)) (justify left top) (href "https://datasheets.raspberrypi.com/rp2040/hardware-design-with-rp2040.pdf"))
+  )
+  (text "Place C25 close to pin 44" (at 158.75 52.705 0)
     (effects (font (size 1.27 1.27)) (justify left bottom))
   )
+  (text "Place C23 close to pin 45" (at 67.945 48.26 0)
+    (effects (font (size 1.27 1.27)) (justify left bottom))
+  )

Commit message: Bugfixes for Rev 2
Oscillator, USB reversed, USB series resistors values
Parts:
- Y1: symbol KD_Oscillator:Crystal_12M_RH100-12.000-18-2020-EXT-TR -> KD_Oscillator:Crystal_12M_ABM8-272-T3; MFG_PartNo RH100-12.000-18-2020-EXT-TR -> ABM8-272-T3; Manufacturer Raltron Electronics -> Abracon LLC; Supplier_PartNo 2151-RH100-12.000-18-2020-EXT-TRCT-ND -> 535-ABM8-272-T3CT-ND
Other:
- note added: "Place C23 near to pin 45"
- note added: "Place C25 near to pin 44"
- note removed: "Place C23 close to pin 45"
- note removed: "Place C25 close to pin 44"
- moved on the sheet: D13, R23, TP7
Changed lines of the file:
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@@
 	)
 	(junction
-		(at 57.15 182.88)
+		(at 73.66 182.88)
 		(diameter 0)
 		(color 0 0 0 0)
@@
 	)
 	(junction
-		(at 64.77 182.88)
+		(at 81.28 182.88)
 		(diameter 0)
 		(color 0 0 0 0)
@@
 	)
 	(no_connect
+		(at 111.76 135.89)
+	)
+	(no_connect
 		(at 111.76 133.35)
 	)
@@
 	)
 	(no_connect
-		(at 111.76 135.89)
-	)
-	(no_connect
 		(at 49.53 147.32)
 	)
@@
 	(wire
 		(pts
-			(xy 46.99 182.88) (xy 57.15 182.88)
+			(xy 121.92 43.18) (xy 132.08 43.18)
 		)
 		(stroke
@@
 	(wire
 		(pts
-			(xy 121.92 43.18) (xy 132.08 43.18)
+			(xy 208.28 102.87) (xy 208.28 105.41)
 		)
 		(stroke
@@
 	(wire
 		(pts
-			(xy 208.28 102.87) (xy 208.28 105.41)
+			(xy 208.28 105.41) (xy 217.17 105.41)
 		)
 		(stroke
@@
 	(wire
 		(pts
-			(xy 208.28 105.41) (xy 217.17 105.41)
+			(xy 132.08 57.15) (xy 132.08 59.69)
 		)
 		(stroke
@@
 	(wire
 		(pts
-			(xy 132.08 57.15) (xy 132.08 59.69)
+			(xy 46.99 182.88) (xy 73.66 182.88)
 		)
 		(stroke
@@
 	(wire
 		(pts
-			(xy 57.15 182.88) (xy 64.77 182.88)
+			(xy 73.66 182.88) (xy 81.28 182.88)
 		)
 		(stroke
@@
 	(wire
 		(pts
-			(xy 57.15 180.34) (xy 57.15 182.88)
+			(xy 73.66 180.34) (xy 73.66 182.88)
 		)
 		(stroke
@@
 	(wire
 		(pts
-			(xy 55.88 170.18) (xy 54.61 170.18)
+			(xy 72.39 170.18) (xy 62.23 170.18)
 		)
 		(stroke
@@
 	(wire
 		(pts
-			(xy 64.77 170.18) (xy 64.77 182.88)
+			(xy 81.28 170.18) (xy 81.28 182.88)
 		)
 		(stroke
@@
 	(wire
 		(pts
-			(xy 34.29 170.18) (xy 46.99 170.18)
+			(xy 34.29 170.18) (xy 54.61 170.18)
 		)
 		(stroke
@@
 	(wire
 		(pts
-			(xy 63.5 170.18) (xy 64.77 170.18)
+			(xy 80.01 170.18) (xy 81.28 170.18)
 		)
 		(stroke
@@
 	(wire
 		(pts
-			(xy 64.77 182.88) (xy 74.93 182.88)
+			(xy 81.28 182.88) (xy 91.44 182.88)
 		)
 		(stroke
@@
 		)
 	)
-	(text "Place C25 close to pin 44"
+	(text "Place C25 near to pin 44"
 		(exclude_from_sim no)
 		(at 158.75 52.705 0)
@@
 		)
 	)
-	(text "Place C23 close to pin 45"
+	(text "Place C23 near to pin 45"
 		(exclude_from_sim no)
 		(at 67.945 48.26 0)
@@
 	)
 	(label "USBBOOT"
-		(at 74.93 182.88 180)
+		(at 91.44 182.88 180)
 		(fields_autoplaced yes)
 		(effects
@@
 	(symbol
 		(lib_id "KD_Connector_Pads:TestPoint_2.5mm_H0.9")
-		(at 57.15 180.34 0)
+		(at 73.66 180.34 0)
 		(unit 1)
 		(exclude_from_sim no)
@@
 		(dnp no)
 		(property "Reference" "TP7"
-			(at 57.15 175.26 0)
+			(at 73.66 175.26 0)
 			(do_not_autoplace yes)
 			(effects
@@
 		)
 		(property "Value" "TP D2.5 mm H0.9mm"
-			(at 44.45 148.59 0)
+			(at 60.96 148.59 0)
 			(effects
 				(font
@@
 		)
 		(property "Footprint" "KD_Connector_Pads:TestPoint_Pad_D2.5mm_H0.9mm"
-			(at 44.45 166.37 0)
+			(at 60.96 166.37 0)
 			(effects
 				(font
@@
 		)
 		(property "Datasheet" "DNP"
-			(at 44.45 168.91 0)
+			(at 60.96 168.91 0)
 			(effects
 				(font
@@
 		)
 		(property "Description" ""
-			(at 57.15 180.34 0)
+			(at 73.66 180.34 0)
 			(effects
 				(font
@@
 		)
 		(property "Code" "DNP"
-			(at 44.45 171.45 0)
+			(at 60.96 171.45 0)
 			(effects
 				(font
@@
 		)
 		(property "Manufacturer" "DNP"
-			(at 44.45 151.13 0)
+			(at 60.96 151.13 0)
 			(effects
 				(font
@@
 		)
 		(property "MFG_PartNo" "DNP"
-			(at 44.45 153.67 0)
+			(at 60.96 153.67 0)
 			(effects
 				(font
@@
 		)
 		(property "Supplier" "DNP"
-			(at 44.45 156.21 0)
+			(at 60.96 156.21 0)
 			(effects
 				(font
@@
 		)
 		(property "Supplier_PartNo" "DNP"
-			(at 44.45 158.75 0)
+			(at 60.96 158.75 0)
 			(effects
 				(font
@@
 		)
 		(property "DNP" "T"
-			(at 44.45 161.29 0)
+			(at 60.96 161.29 0)
 			(effects
 				(font
@@
 		)
 		(property "Price" "0.00"
-			(at 44.45 163.83 0)
+			(at 60.96 163.83 0)
 			(effects
 				(font
@@
 	)
 	(symbol
-		(lib_id "KD_Oscillator:Crystal_12M_RH100-12.000-18-2020-EXT-TR")
+		(lib_id "KD_Oscillator:Crystal_12M_ABM8-272-T3")
 		(at 74.93 123.19 0)
 		(unit 1)
@@
 			)
 		)
-		(property "Datasheet" "https://www.raltron.com/webproducts/specs/CRYSTAL/RH100-12.000-18-2020-EXT-TR.pdf"
+		(property "Datasheet" "https://www.mouser.fi/datasheet/2/3/ABM8_272_T3-3392615.pdf"
 			(at 62.23 111.76 0)
 			(effects
@@
 			)
 		)
-		(property "Description" ""
-			(at 74.93 123.19 0)
+		(property "Description" "12 MHz ±30ppm Crystal 10pF 50 Ohms 4-SMD, No Lead"
+			(at 62.23 91.44 0)
 			(effects
 				(font
 					(size 1.27 1.27)
 				)
+				(justify left)
 				(hide yes)
 			)
 		)
-		(property "Manufacturer" "Raltron Electronics"
+		(property "Manufacturer" "Abracon LLC"
 			(at 62.23 93.98 0)
 			(effects
@@
 			)
 		)
-		(property "MFG_PartNo" "RH100-12.000-18-2020-EXT-TR"
+		(property "MFG_PartNo" "ABM8-272-T3"
 			(at 62.23 96.52 0)
 			(effects
@@
 			)
 		)
-		(property "Supplier_PartNo" "2151-RH100-12.000-18-2020-EXT-TRCT-ND"
+		(property "Supplier_PartNo" "535-ABM8-272-T3CT-ND"
 			(at 62.23 101.6 0)
 			(effects
@@
 	(symbol
 		(lib_id "KD_Resistor:R_0603_1k_1%")
-		(at 59.69 170.18 90)
+		(at 76.2 170.18 90)
 		(unit 1)
 		(exclude_from_sim no)
@@
 		(fields_autoplaced yes)
 		(property "Reference" "R23"
-			(at 59.69 163.83 90)
+			(at 76.2 163.83 90)
 			(effects
 				(font
@@
 		)
 		(property "Value" "1k"
-			(at 27.94 182.88 0)
+			(at 44.45 182.88 0)
 			(effects
 				(font
@@
 		)
 		(property "Footprint" "KD_Resistor:RESC1608X55N"
-			(at 45.72 182.88 0)
+			(at 62.23 182.88 0)
 			(effects
 				(font
@@
 		)
 		(property "Datasheet" "https://www.seielect.com/Catalog/SEI-RMCF_RMCP.pdf"
-			(at 48.26 182.88 0)
+			(at 64.77 182.88 0)
 			(effects
 				(font
@@
 		)
 		(property "Description" ""
-			(at 59.69 170.18 0)
+			(at 76.2 170.18 0)
 			(effects
 				(font
@@
 		)
 		(property "Code" "1k"
-			(at 59.69 166.37 90)
+			(at 76.2 166.37 90)
 			(effects
 				(font
@@
 		)
 		(property "Manufacturer" "Stackpole Electronics Inc"
-			(at 30.48 182.88 0)
+			(at 46.99 182.88 0)
 			(effects
 				(font
@@
 		)
 		(property "MFG_PartNo" "RMCF0603JT1K00"
-			(at 33.02 182.88 0)
+			(at 49.53 182.88 0)
 			(effects
 				(font
@@
 		)
 		(property "Supplier" "Digi-Key"
-			(at 35.56 182.88 0)
+			(at 52.07 182.88 0)
 			(effects
 				(font
@@
 		)
 		(property "Supplier_PartNo" "RMCF0603JT1K00CT-ND"
-			(at 38.1 182.88 0)
+			(at 54.61 182.88 0)
 			(effects
 				(font
@@
 		)
 		(property "DNP" "F"
-			(at 40.64 182.88 0)
+			(at 57.15 182.88 0)
 			(effects
 				(font
@@
 		)
 		(property "Price" "0.01"
-			(at 43.18 182.88 0)
+			(at 59.69 182.88 0)
 			(effects
 				(font
@@
 	(symbol
 		(lib_id "KD_Diode:Schottky_30V_200mA_DCo_BAT54WS")
-		(at 50.8 170.18 180)
+		(at 58.42 170.18 180)
 		(unit 1)
 		(exclude_from_sim no)
@@
 		(fields_autoplaced yes)
 		(property "Reference" "D13"
-			(at 51.1175 163.83 0)
+			(at 58.674 163.83 0)
 			(effects
 				(font
@@
 		)
 		(property "Value" "Schottky_30V_200mA_DCo_BAT54WS"
-			(at 63.5 201.93 0)
+			(at 71.12 201.93 0)
 			(effects
 				(font
@@
 		)
 		(property "Footprint" "KD_Diode:D_SOD-323"
-			(at 63.5 184.15 0)
+			(at 71.12 184.15 0)
 			(effects
 				(font
@@
 		)
 		(property "Datasheet" "https://diotec.com/tl_files/diotec/files/pdf/datasheets/bat54ws.pdf"
-			(at 63.5 181.61 0)
+			(at 71.12 181.61 0)
 			(effects
 				(font
@@
 			)
 		)
-		(property "Description" ""
-			(at 50.8 170.18 0)
+		(property "Description" "Diode Schottky 30 V 200mA Surface Mount SOD-323"
+			(at 58.42 170.18 0)
 			(effects
 				(font
@@
 		)
 		(property "Code" "BAT54WS"
-			(at 51.1175 166.37 0)
+			(at 58.674 166.37 0)
 			(effects
 				(font
@@
 		)
 		(property "Manufacturer" "DComponents"
-			(at 63.5 199.39 0)
+			(at 71.12 199.39 0)
 			(effects
 				(font
@@
 		)
 		(property "MFG_PartNo" "BAT54WS"
-			(at 63.5 196.85 0)
+			(at 71.12 196.85 0)
 			(effects
 				(font
@@
 		)
 		(property "Supplier" "Digi-Key"
-			(at 63.5 194.31 0)
+			(at 71.12 194.31 0)
 			(effects
 				(font
@@
 		)
 		(property "Supplier_PartNo" "2721-BAT54WSTR-ND"
-			(at 63.5 191.77 0)
+			(at 71.12 191.77 0)
 			(effects
 				(font
@@
 		)
 		(property "DNP" "F"
-			(at 63.5 189.23 0)
+			(at 71.12 189.23 0)
 			(effects
 				(font
@@
 		)
 		(property "Price" "0.05"
-			(at 63.5 186.69 0)
+			(at 71.12 186.69 0)
 			(effects
 				(font

Commit message: Updated layout from schematic
Connections:
- no-connect marks 9 -> 11
Changed lines of the file:
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@@
+	)
+	(no_connect
+		(at 163.83 80.01)
 	)
 	(no_connect
@@
 	)
 	(no_connect
+		(at 163.83 115.57)
+	)
+	(no_connect
