File: PCB/Rev 03.00/000018 PGKB/USBcon.kicad_sch (KiCad schematic)
At the start: 10 parts, among them J1 USB C

Commit message: Rev 3 tekemista
Parts:
- C1: Code 10u -> (none)
- D11: value TVS_5V5_DRTR5V0U4S-7-M -> DRTR5V0U4S-7; Code DRTR5V0U4S-7 -> (none)
- D12: value Schottky_30V_1A_PMEG3010ER_115 -> PMEG3010ER,115; footprint KD_Diode:DIOC360X180X150_SOD123 -> KD_Diode:DIOC360X180X150N_A; Code PMEG3010ER,115 -> (none)
- R1, R2: value R_0603_5100_1% -> 5k1; Code 5k1 -> (none)
Changed lines of the file:
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@@
 	(title_block
 		(title "Programmable Keyboard")
-		(date "2024-08-18")
+		(date "2025-01-06")
 		(rev "3.0")
 		(company "Kallio Designs Oy")
 		(comment 1 "TL, NH")
+		(comment 2 "ASSEMBLY_PN")
 		(comment 3 "000018")
 	)
@@
 			)
 		)
-		(property "Value" "R_0603_5100_1%"
-			(at 100.33 26.67 0)
-			(effects
-				(font
-					(size 1.27 1.27)
-				)
-				(justify left)
-				(hide yes)
+		(property "Value" "5k1"
+			(at 115.57 59.6899 0)
+			(effects
+				(font
+					(size 1.27 1.27)
+				)
+				(justify left)
 			)
 		)
@@
 		)
 		(property "Description" "RES 5.1K OHM 5% 1/10W 0603"
-			(at 113.03 58.42 0)
-			(effects
-				(font
-					(size 1.27 1.27)
-				)
-				(hide yes)
-			)
-		)
-		(property "Code" "5k1"
-			(at 115.57 59.6899 0)
-			(effects
-				(font
-					(size 1.27 1.27)
-				)
-				(justify left)
+			(at 100.33 26.67 0)
+			(effects
+				(font
+					(size 1.27 1.27)
+				)
+				(hide yes)
 			)
 		)
@@
 		)
 		(property "Value" "10u"
-			(at 189.23 24.13 0)
-			(effects
-				(font
-					(size 1.27 1.27)
-				)
-				(justify left)
-				(hide yes)
+			(at 205.74 57.1499 0)
+			(effects
+				(font
+					(size 1.27 1.27)
+				)
+				(justify left)
 			)
 		)
@@
 		)
 		(property "Description" "Capacitor"
-			(at 201.93 55.88 0)
+			(at 190.5 23.368 0)
 			(effects
 				(font
@@
 				(justify left)
 				(hide yes)
-			)
-		)
-		(property "Code" "10u"
-			(at 205.74 57.1499 0)
-			(effects
-				(font
-					(size 1.27 1.27)
-				)
-				(justify left)
 			)
 		)
@@
 			)
 		)
-		(property "Value" "TVS_5V5_DRTR5V0U4S-7-M"
-			(at 129.54 66.04 0)
-			(effects
-				(font
-					(size 1.27 1.27)
-				)
-				(justify left)
-				(hide yes)
+		(property "Value" "DRTR5V0U4S-7"
+			(at 144.78 99.06 0)
+			(effects
+				(font
+					(size 1.27 1.27)
+				)
 			)
 		)
@@
 		)
 		(property "Description" "TVS DIODE 5.5VWM SOT363"
-			(at 144.78 110.49 0)
-			(effects
-				(font
-					(size 1.27 1.27)
-				)
-				(hide yes)
-			)
-		)
-		(property "Code" "DRTR5V0U4S-7"
-			(at 144.78 99.06 0)
-			(effects
-				(font
-					(size 1.27 1.27)
-				)
+			(at 132.842 63.5 0)
+			(effects
+				(font
+					(size 1.27 1.27)
+				)
+				(hide yes)
 			)
 		)
@@
 			)
 		)
-		(property "Value" "Schottky_30V_1A_PMEG3010ER_115"
-			(at 158.75 82.55 0)
-			(effects
-				(font
-					(size 1.27 1.27)
-				)
-				(justify left)
-				(hide yes)
-			)
-		)
-		(property "Footprint" "KD_Diode:DIOC360X180X150_SOD123"
+		(property "Value" "PMEG3010ER,115"
+			(at 146.304 46.99 0)
+			(effects
+				(font
+					(size 1.27 1.27)
+				)
+			)
+		)
+		(property "Footprint" "KD_Diode:DIOC360X180X150N_A"
 			(at 158.75 64.77 0)
 			(effects
@@
 		)
 		(property "Description" "DIODE SCHOTTKY 30V 1A SOD123W"
-			(at 146.05 50.8 0)
-			(effects
-				(font
-					(size 1.27 1.27)
-				)
-				(hide yes)
-			)
-		)
-		(property "Code" "PMEG3010ER,115"
-			(at 146.304 46.99 0)
-			(effects
-				(font
-					(size 1.27 1.27)
-				)
+			(at 157.48 83.058 0)
+			(effects
+				(font
+					(size 1.27 1.27)
+				)
+				(hide yes)
 			)
 		)
@@
 		)
 		(property "Description" "CAP CER 0.1UF 50V X7R 0603"
-			(at 214.63 55.88 0)
+			(at 203.2 24.384 0)
 			(effects
 				(font
@@
 			)
 		)
-		(property "Value" "R_0603_5100_1%"
-			(at 109.22 26.67 0)
-			(effects
-				(font
-					(size 1.27 1.27)
-				)
-				(justify left)
-				(hide yes)
+		(property "Value" "5k1"
+			(at 124.46 59.6899 0)
+			(effects
+				(font
+					(size 1.27 1.27)
+				)
+				(justify left)
 			)
 		)
@@
 		)
 		(property "Description" "RES 5.1K OHM 5% 1/10W 0603"
-			(at 121.92 58.42 0)
-			(effects
-				(font
-					(size 1.27 1.27)
-				)
-				(hide yes)
-			)
-		)
-		(property "Code" "5k1"
-			(at 124.46 59.6899 0)
-			(effects
-				(font
-					(size 1.27 1.27)
-				)
-				(justify left)
-			)
-		)
+			(at 109.22 26.67 0)
+			(effects
+				(font
+					(size 1.27 1.27)
+				)
+				(hide yes)
+			)
+		)
