File: PCB/Rev 03.00/000018 PGKB/000018 PGKB.kicad_pcb (KiCad board)
At the start: 4 copper layers, 93.5 x 72.5 mm, 157 parts, among them J1 USB C, J2 S4B-PH-SM4-TB, J3 GND Hook, U1 SN74HCS365PWR, U2 SN74HCS365PWR, U3 SN74HCS365PWR, U4 W25Q80DVSSIG, U5 RP2040, U6 MCP1825T-3302E/DC, U7 CAT811TTBI-GT3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

Commit message: Rev3 outputs
Parts:
- moved TP12 9.38 mm to (79.9, 105.3)
- moved TP11 6.00 mm to (60.3, 106.5)
- moved TP16 2.68 mm to (55.2, 105.3)
- moved TP10 0.25 mm to (108.4, 133.4)
Routing:
- net /Main/Connectors/I2C1_SCL: track 58.7 -> 69.1 mm
- net /Main/Connectors/I2C1_SDA: track 63.5 -> 69.5 mm
- net Net-(D10-DIN): track 26.9 -> 29.0 mm
- net GND: vias 182 -> 181

Commit message: Rev 3 tekemista
Parts:
- D11: value TVS_5V5_DRTR5V0U4S-7-M -> DRTR5V0U4S-7
- D12: value Schottky_30V_1A_PMEG3010ER_115 -> PMEG3010ER,115; footprint KD_Diode:DIOC360X180X150_SOD123 -> KD_Diode:DIOC360X180X150N_A
- D13: value Schottky_30V_200mA_DCo_BAT54WS -> BAT54WS
- R1, R2, R26, R27: value R_0603_5100_1% -> 5k1
- R24: value R_0603_DNP -> DNP
- S12, S13: value 430181038816 -> PTS647SN38SMTR2 LFS; footprint KD_Switch:SW_Push_1P1T_NO_Wurth_430181038816 -> KD_Switch:SW_Push_1P1T_NO_CK_PTS647SN50SMTR2LFS
- moved R9 0.05 mm to (60.0, 149.0)
- moved C8 0.05 mm to (58.5, 149.0)
Connections:
- J3 pad 1: unconnected-(J3-Pin_1-Pad1) -> GND
- J3 pad 2: unconnected-(J3-Pin_1-Pad2) -> GND
Routing:
- net GND: track 157.9 -> 172.7 mm, vias 181 -> 180
- net /Main/Microcontroller/USBBOOT: track 39.4 -> 39.9 mm
Other:
- board text added: "${COMMENT3} ${TITLE} Rev ${REVISION} ${ISSUE_DATE},${COMMENT1}"
- board text removed: "000018 PGKB Rev 1.00"

Commit message: mfg outputs
Changed lines of the file:
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@@
 		(fp_arc
 			(start 1.372869 0.972724)
-			(mid 0.966366 0.781547)
+			(mid 0.96636 0.78155)
 			(end 0.82295 0.35584)
 			(stroke
@@
 		(tags "resistor 0603")
 		(property "Reference" "R36"
-			(at 0.566882 2.033397 360)
+			(at 0.566882 2.033397 0)
 			(layer "B.SilkS")
 			(effects
@@
 		(tags "capacitor cap 0603 1608")
 		(property "Reference" "C8"
-			(at -2.203884 -0.071209 360)
+			(at -2.203884 -0.071209 0)
 			(layer "B.SilkS")
 			(effects
