File: PCB/Rev 03.00/000018 PGKB/buttons.kicad_sch (KiCad schematic)
At the start: 50 parts, among them U1 SN74HCS365PWR, U2 SN74HCS365PWR

Commit message: mfg outputs
Parts:
- added S14, S99: 4954, KD_Switch:SWITCH_BUTTON_Kailh_mx_socket, symbol KD_Switch:Button_keyboard_no_footprint_Adafruit_4954
Other:
- note added: "Two 10-packs of switches"
