File: PCB/Rev 03.00/000018 PGKB/mcu.kicad_sch (KiCad schematic)
At the start: 32 parts, among them U5 RP2040, Y1 12 MHz

Commit message: Rev 3 tekemista
Parts:
- D13: value Schottky_30V_200mA_DCo_BAT54WS -> BAT54WS; Code BAT54WS -> (none)
- R24: value R_0603_DNP -> DNP; Code DNP -> (none)
- R37, R38: value R_0603_5100_1% -> 5k1; Code 5k1 -> (none)
- S12, S13: value 430181038816 -> PTS647SN38SMTR2 LFS; footprint KD_Switch:SW_Push_1P1T_NO_Wurth_430181038816 -> KD_Switch:SW_Push_1P1T_NO_CK_PTS647SN50SMTR2LFS; symbol KD_Switch:Button_tactile_45x38_430181038816 -> KD_Switch:Button_tactile_PTS647SN38SMTR2LFS; MFG_PartNo 430181038816 -> PTS647SN38SMTR2 LFS; Manufacturer Wurth Elektronik -> C&K; Price 0.5 -> 0.17; Supplier Mouser -> Digi-Key; Supplier_PartNo 710-430181038816 -> PTS647SN38SMTR2LFSCT-ND
Other:
- moved on the sheet: D13, R23, S12, TP7

Commit message: mfg outputs
Parts:
- D13: value BAT54WS -> BAT54WSQ-7-F; symbol KD_Diode:Schottky_30V_200mA_DCo_BAT54WS -> KD_Diode:Schottky_30V_100mA_Diodes_BAT54WSQ-7-F; MFG_PartNo BAT54WS -> BAT54WSQ-7-F; Manufacturer DComponents -> Diodes Incorporated; Supplier_PartNo 2721-BAT54WSTR-ND -> BAT54WSQ-7-FDICT-ND
Changed lines of the file:
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@@
 	)
 	(symbol
-		(lib_id "KD_Diode:Schottky_30V_200mA_DCo_BAT54WS")
+		(lib_id "KD_Diode:Schottky_30V_100mA_Diodes_BAT54WSQ-7-F")
 		(at 68.58 170.18 180)
 		(unit 1)
@@
 		(on_board yes)
 		(dnp no)
-		(fields_autoplaced yes)
 		(property "Reference" "D13"
 			(at 68.834 166.37 0)
@@
 			)
 		)
-		(property "Value" "BAT54WS"
+		(property "Value" "BAT54WSQ-7-F"
 			(at 68.58 173.99 0)
 			(do_not_autoplace yes)
@@
 			)
 		)
-		(property "Datasheet" "https://diotec.com/tl_files/diotec/files/pdf/datasheets/bat54ws.pdf"
+		(property "Datasheet" "https://www.diodes.com/assets/Datasheets/BAT54WS.pdf"
 			(at 81.28 181.61 0)
 			(effects
@@
 			)
 		)
-		(property "Description" "Diode Schottky 30 V 200mA Surface Mount SOD-323"
+		(property "Description" "Diode 30 V 100mA Surface Mount SOD-323"
 			(at 81.28 204.47 0)
 			(effects
@@
 			)
 		)
-		(property "Manufacturer" "DComponents"
+		(property "Manufacturer" "Diodes Incorporated"
 			(at 81.28 199.39 0)
 			(effects
@@
 			)
 		)
-		(property "MFG_PartNo" "BAT54WS"
+		(property "MFG_PartNo" "BAT54WSQ-7-F"
 			(at 81.28 196.85 0)
 			(effects
@@
 			)
 		)
-		(property "Supplier_PartNo" "2721-BAT54WSTR-ND"
+		(property "Supplier_PartNo" "BAT54WSQ-7-FDICT-ND"
 			(at 81.28 191.77 0)
 			(effects
