File: PCB/Rev 03.00/000018 PGKB/psu.kicad_sch (KiCad schematic)
At the start: 11 parts, among them U6 MCP1825T-3302E/DC, U7 CAT811TTBI-GT3

Commit message: Rev 3 tekemista
Parts:
- C6: Code 10u -> (none)
Changed lines of the file:
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@@
 	(title_block
 		(title "Programmable Keyboard")
-		(date "2024-08-18")
+		(date "2025-01-06")
 		(rev "3.0")
 		(company "Kallio Designs Oy")
@@
 		)
 		(property "Description" "CAP CER 0.1UF 50V X7R 0603"
-			(at 81.28 96.52 0)
+			(at 69.85 65.024 0)
 			(effects
 				(font
@@
 		)
 		(property "Value" "10u"
-			(at 121.92 66.04 0)
-			(effects
-				(font
-					(size 1.27 1.27)
-				)
-				(justify left)
-				(hide yes)
+			(at 137.16 99.06 0)
+			(effects
+				(font
+					(size 1.27 1.27)
+				)
+				(justify left)
 			)
 		)
@@
 		)
 		(property "Description" "Capacitor"
-			(at 134.62 97.79 0)
-			(effects
-				(font
-					(size 1.27 1.27)
-				)
-				(hide yes)
-			)
-		)
-		(property "Code" "10u"
-			(at 137.16 99.06 0)
-			(effects
-				(font
-					(size 1.27 1.27)
-				)
-				(justify left)
+			(at 123.19 65.278 0)
+			(effects
+				(font
+					(size 1.27 1.27)
+				)
+				(hide yes)
 			)
 		)
@@
 		)
 		(property "Description" "CAP CER 0.1UF 50V X7R 0603"
-			(at 148.59 97.79 0)
+			(at 137.16 66.294 0)
 			(effects
 				(font
@@
 		)
 		(property "Description" "IC SUPERVISOR 1 CHANNEL SOT143 3.08V"
-			(at 194.31 92.71 0)
-			(effects
-				(font
-					(size 1.27 1.27)
-				)
-				(hide yes)
-			)
+			(at 181.61 60.96 0)
+			(effects
+				(font
+					(size 1.27 1.27)
+				)
+				(justify left)
+				(hide yes)
+			)

Commit message: mfg outputs
Parts:
- U7: value CAT811TTBI-GT3 -> APX811-31UG-7; symbol KD_IC_Other:Supervisor_CAT811TTBI-GT3 -> KD_IC_Other:Supervisor_APX811-31UG-7; MFG_PartNo CAT811TTBI-GT3 -> APX811-31UG-7; Manufacturer onsemi -> Diodes Incorporated; Price 0.5 -> 0.41; Supplier_PartNo CAT811TTBI-GT3OSCT-ND -> APX811-31UG-7DICT-ND
Changed lines of the file:
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@@
 	)
 	(symbol
-		(lib_id "KD_IC_Other:Supervisor_CAT811TTBI-GT3")
+		(lib_id "KD_IC_Other:Supervisor_APX811-31UG-7")
 		(at 194.31 92.71 0)
 		(unit 1)
@@
 			)
 		)
-		(property "Value" "CAT811TTBI-GT3"
+		(property "Value" "APX811-31UG-7"
 			(at 196.85 88.9 0)
 			(do_not_autoplace yes)
@@
 			)
 		)
-		(property "Datasheet" "https://www.onsemi.com/pdf/datasheet/cat811-d.pdf"
+		(property "Datasheet" "https://www.diodes.com/assets/Datasheets/APX811_812.pdf"
 			(at 181.61 81.28 0)
 			(effects
@@
 			)
 		)
-		(property "Description" "IC SUPERVISOR 1 CHANNEL SOT143 3.08V"
+		(property "Description" "IC SUPERVISOR 1 CHANNEL SOT143"
 			(at 181.61 60.96 0)
 			(effects
@@
 			)
 		)
-		(property "Manufacturer" "onsemi"
+		(property "Manufacturer" "Diodes Incorporated"
 			(at 181.61 63.5 0)
 			(effects
@@
 			)
 		)
-		(property "MFG_PartNo" "CAT811TTBI-GT3"
+		(property "MFG_PartNo" "APX811-31UG-7"
 			(at 181.61 66.04 0)
 			(effects
@@
 			)
 		)
-		(property "Supplier_PartNo" "CAT811TTBI-GT3OSCT-ND"
+		(property "Supplier_PartNo" "APX811-31UG-7DICT-ND"
 			(at 181.61 71.12 0)
 			(effects
@@
 			)
 		)
-		(property "Price" "0.5"
+		(property "Price" "0.41"
 			(at 181.61 76.2 0)
 			(effects
