File: PCB/Rev 03.00/000018 PGKB/rev_history.kicad_sch (KiCad schematic)
At the start: 0 parts

Commit message: Rev3 outputs
Changed lines of the file:
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@@
 	(title_block
 		(title "Programmable Keyboard")
-		(date "2024-04-09")
-		(rev "2.1")
+		(date "2024-08-18")
+		(rev "3.0")
 		(company "Kallio Designs Oy")
 		(comment 1 "TL, NH")
 		(comment 2 "ASSEMBLY_PN")
-		(comment 3 "PCB_PN")
+		(comment 3 "000018")
 	)
 	(polyline
@@
 		)
 		(stroke
+			(width 0)
+			(type solid)
+			(color 0 0 0 1)
+		)
+	)
+	(polyline
+		(pts
+			(xy 57.15 77.47) (xy 243.84 77.47)
+		)
+		(stroke

Commit message: Rev 3 tekemista
Other:
- note added: "06.01.2025"
- note added: "22.10.2023"
- note added: "3.0"
- note added: "Form factor changed, connectors changed"
- note added: "LEDs added, changed key types"
- note added: "Microcontroller and surrounding circuitry changed"
- note added: "Teemu Latonen, Niko Hämäläinen"
- note removed: "14.07.2024"
Changed lines of the file:
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@@
 	(title_block
 		(title "Programmable Keyboard")
-		(date "2024-08-18")
+		(date "2025-01-06")
 		(rev "3.0")
 		(company "Kallio Designs Oy")
@@
 	(polyline
 		(pts
+			(xy 57.15 95.25) (xy 243.84 95.25)
+		)
+		(stroke
+			(width 0)
+			(type solid)
+			(color 0 0 0 1)
+		)
+	)
+	(polyline
+		(pts
 			(xy 68.58 148.59) (xy 68.58 48.26)
 		)
@@
 		)
 	)
-	(text "Teemu Latonen"
-		(exclude_from_sim no)
-		(at 208.28 64.77 0)
-		(effects
-			(font
-				(size 2 2)
-			)
-			(justify left bottom)
-		)
-	)
-	(text "14.07.2024"
+	(text "Teemu Latonen, \nNiko Hämäläinen"
+		(exclude_from_sim no)
+		(at 208.28 67.31 0)
+		(effects
+			(font
+				(size 2 2)
+			)
+			(justify left bottom)
+		)
+	)
+	(text "22.10.2023"
 		(exclude_from_sim no)
 		(at 69.85 64.77 0)
@@
 		)
 	)
+	(text "USB Signals reversed"
+		(exclude_from_sim no)
+		(at 90.17 82.55 0)
+		(effects
+			(font
+				(size 2 2)
+			)
+			(justify left bottom)
+		)
+	)
+	(text "3.0"
+		(exclude_from_sim no)
+		(at 58.42 82.55 0)
+		(effects
+			(font
+				(size 2 2)
+			)
+			(justify left bottom)
+		)
+	)
 	(text "2.0"
 		(exclude_from_sim no)
@@
 		)
 	)
+	(text "USB series resistor value changed from 10 ohm to 27 ohm"
+		(exclude_from_sim no)
+		(at 90.17 92.71 0)
+		(effects
+			(font
+				(size 2 2)
+			)
+			(justify left bottom)
+		)
+	)
 	(text "DATE"
 		(exclude_from_sim no)
@@
 		)
 	)
+	(text "Teemu Latonen"
+		(exclude_from_sim no)
+		(at 208.28 82.55 0)
+		(effects
+			(font
+				(size 2 2)
+			)
+			(justify left bottom)
+		)
+	)
+	(text "06.01.2025"
+		(exclude_from_sim no)
+		(at 69.85 82.55 0)
+		(effects
+			(font
+				(size 2 2)
+			)
+			(justify left bottom)
+		)
+	)
 	(text "Initial"
 		(exclude_from_sim no)
@@
 		)
 	)
-	(text "USB series resistor value changed from 10 ohm to 27 ohm"
+	(text "Oscillator Y1 changed"
+		(exclude_from_sim no)
+		(at 90.17 87.63 0)
+		(effects
+			(font
+				(size 2 2)
+			)
+			(justify left bottom)
+		)
+	)
+	(text "Microcontroller and surrounding circuitry changed"
 		(exclude_from_sim no)
 		(at 90.17 74.93 0)
@@
 		)
 	)
-	(text "USB Signals reversed"
+	(text "Form factor changed, connectors changed"
 		(exclude_from_sim no)
 		(at 90.17 64.77 0)
@@
 		)
 	)
-	(text "Oscillator Y1 changed"
+	(text "LEDs added, changed key types"
 		(exclude_from_sim no)
 		(at 90.17 69.85 0)

Commit message: mfg outputs
Other:
- note added: "08.01.2025"
- note added: "Diode manufacturer change, voltage supervisor type changed"
- note removed: "06.01.2025"
Changed lines of the file:
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@@
 	(polyline
 		(pts
-			(xy 57.15 95.25) (xy 243.84 95.25)
+			(xy 57.15 99.06) (xy 243.84 99.06)
 		)
 		(stroke
@@
 		)
 	)
-	(text "06.01.2025"
+	(text "08.01.2025"
 		(exclude_from_sim no)
 		(at 69.85 82.55 0)
@@
 		(effects
 			(font
+				(size 2 2)
+			)
+			(justify left bottom)
+		)
+	)
+	(text "Diode manufacturer change, voltage supervisor type changed"
+		(exclude_from_sim no)
+		(at 90.17 97.79 0)
+		(effects
+			(font
